Commit message: adiciona novas característivas físicas

File: littlebot_description/urdf/littlebot.xacro (robot description, xacro)
@@ -25,5 +25,5 @@
       <origin xyz="0 0 0.15" rpy="1.571 0 1.571"/>
       <mass value="0.100"/>
-      <inertia ixx="0"  ixy="0"  ixz="0" iyy="0" iyz="0" izz="0" />
+      <inertia ixx="1e-3"  ixy="0"  ixz="0" iyy="1e-3" iyz="0" izz="1e-3" />
     </inertial>
   </link>
@@ -88,5 +88,5 @@
       <origin xyz="0 0.0115 0" rpy="0 0 -1.571"/>
       <mass value="0.041"/>
-      <inertia ixx="0"  ixy="0"  ixz="0" iyy="0" iyz="0" izz="0" />
+      <inertia ixx="2.967e-5"  ixy="-7.675e-15"  ixz="-4.765e-14" iyy="1.616e-5" iyz="-1.121e-16" izz="1.616e-5" />
     </inertial>
   </link>

Commit message: adicionar mashe dos motores à simulação

File: littlebot_description/urdf/littlebot.xacro (robot description, xacro)
@@ -1,11 +1,8 @@
 <?xml version="1.0"?>
 <robot name="littlebot" xmlns:xacro="http://www.ros.org/wiki/xacro">
-<!-- Used for fixing robot to Gazebo 'base_link' -->
-<!--
-<link name="world"/>
-<joint name="fixed" type="fixed">
-    <parent link="world"/>
-    <child link="base_link"/>
-</joint>
+ <!--
+########################################################################################
+Modelagem do chassis2 "link" "joint"
+########################################################################################
 -->
  <link name="base_link">
@@ -24,10 +21,13 @@
     <inertial>
       <origin xyz="0 0 0.15" rpy="1.571 0 1.571"/>
-      <mass value="0.100"/>
-      <inertia ixx="1e-3"  ixy="0"  ixz="0" iyy="1e-3" iyz="0" izz="1e-3" />
-    </inertial>
-  </link>
-<!--Modelagem da roda esquerda "link" "joint"
-######################################################################################## -->
+      <mass value="0.058"/>
+      <inertia ixx="1.429e-4"  ixy="2.778e-10"  ixz="1.773e-8" iyy="1.943e-4" iyz="-2.656e-7" izz="5.361e-5" />
+    </inertial>
+  </link>
+<!--
+########################################################################################
+Modelagem da roda esquerda "link" "joint"
+########################################################################################
+-->
   <link name="roda_esquerda">
     <visual>
@@ -49,15 +49,8 @@
     </inertial>
   </link>
-  <!--
-  <joint name="base_to_roda_esquerda" type="fixed">
+  <joint name="base_to_roda_esquerda" type="continuous">
     <parent link="base_link"/>
     <child link="roda_esquerda"/>
-    <origin xyz="0 0.07393 -0.01" rpy="0 0 0" />
-  </joint>
--->
-  <joint name="base_to_roda_esquerda" type="continuous">
-    <parent link="base_link"/>
-    <child link="roda_esquerda"/>
-    <origin xyz="0 0.07393 -0.01" rpy="0 0 0" />
+    <origin xyz="0.005 0.07393 -0.014" rpy="0 0 0" />
     <axis xyz="0 1 0" />
   </joint>
@@ -70,6 +63,9 @@
     <turnGravityOff>false</turnGravityOff>
   </gazebo>
-<!--Modelagem da roda direita "link" "joint"
-######################################################################################## -->
+<!--
+########################################################################################
+Modelagem da roda direita "link" "joint"
+########################################################################################
+-->
   <link name="roda_direita">
     <visual>
@@ -91,15 +87,8 @@
     </inertial>
   </link>
-<!--
-  <joint name="base_to_roda_direita" type="fixed">
+  <joint name="base_to_roda_direita" type="continuous">
     <parent link="base_link"/>
     <child link="roda_direita"/>
-    <origin xyz="0 -0.07393 -0.01" rpy="0 0 0" />
-  </joint>
--->
-  <joint name="base_to_roda_direita" type="continuous">
-    <parent link="base_link"/>
-    <child link="roda_direita"/>
-    <origin xyz="0 -0.07393 -0.01" rpy="0 0 0" />
+    <origin xyz="0.005 -0.07393 -0.014" rpy="0 0 0" />
     <axis xyz="0 1 0" />
   </joint>
@@ -112,5 +101,7 @@
     <turnGravityOff>false</turnGravityOff>
   </gazebo>
-<!--Modelagem da rodinha "link" "joint"
+<!--
+########################################################################################
+Modelagem da rodinha "link" "joint"
 ######################################################################################## -->
   <link name="rodinha">
@@ -130,6 +121,6 @@
     <inertial>
       <origin xyz="0 0 0" rpy="3.14 0 2.141"/>
-      <mass value="0.08"/>
-      <inertia ixx="0"  ixy="0"  ixz="0" iyy="0" iyz="0" izz="0" />
+      <mass value="0.073"/>
+      <inertia ixx="5.470e-6"  ixy="4.042e-7"  ixz="3.515e-7" iyy="7.169e-6" iyz="-3.645e-7" izz="7.383e-6" />
     </inertial>
   </link>
@@ -138,4 +129,62 @@
     <child link="rodinha"/>
     <origin xyz="-0.07 0.0 -0.003" rpy="0 0 0" />
+  </joint>
+<!--
+########################################################################################
+Modelagem do motor esquerdo "link" "joint"
+########################################################################################
+-->
+  <link name="motor_esquerdo">
+    <visual>
+      <origin xyz="0 0 0" rpy="0 0 0" />
+      <geometry>
+	      <mesh filename="package://littlebot_description/meshes/motor.dae" />
+      </geometry>
+    </visual>
+    <collision>
+      <origin xyz="0 0 0" rpy="0 0 0" />
+      <geometry>
+	      <mesh filename="package://littlebot_description/meshes/motor.dae" />
+      </geometry>
+    </collision>
+    <inertial>
+      <origin xyz="0 0 0" rpy="0 0 0"/>
+      <mass value="0.09"/>
+      <inertia ixx="0"  ixy="0"  ixz="0" iyy="0" iyz="0" izz="0" />
+    </inertial>
+  </link>
+  <joint name="base_to_motor_esquerdo" type="fixed">
+    <parent link="base_link"/>
+    <child link="motor_esquerdo"/>
+    <origin xyz="-0.032 0.0387 -0.014" rpy="0 0 0" />
+  </joint>
+<!--
+########################################################################################
+Modelagem do motor direito "link" "joint"
+########################################################################################
+-->
+  <link name="motor_direito">
+    <visual>
+      <origin xyz="0 0 0" rpy="0 0 0" />
+      <geometry>
+	      <mesh filename="package://littlebot_description/meshes/motor.dae" />
+      </geometry>
+    </visual>
+    <collision>
+      <origin xyz="0 0 0" rpy="0 0 0" />
+      <geometry>
+	      <mesh filename="package://littlebot_description/meshes/motor.dae" />
+      </geometry>
+    </collision>
+    <inertial>
+      <origin xyz="0 0 0" rpy="0 0 0"/>
+      <mass value="0.09"/>
+      <inertia ixx="0"  ixy="0"  ixz="0" iyy="0" iyz="0" izz="0" />
+    </inertial>
+  </link>
+  <joint name="base_to_motor_direito" type="fixed">
+    <parent link="base_link"/>
+    <child link="motor_direito"/>
+    <origin xyz="-0.032 -0.0387 -0.014" rpy="0 0 0" />
   </joint>
 <!--
@@ -164,5 +213,5 @@
   <!--
   ******************************************************************************************
-  ros_control plugin
+  ros_control gazebo plugin
   ******************************************************************************************
   -->
@@ -172,3 +221,22 @@
     </plugin>
   </gazebo>
+  <!--
+  ******************************************************************************************
+  IMU gazebo plugin
+  ******************************************************************************************
+  -->
+  <gazebo>
+    <plugin name="imu_controller" filename="libhector_gazebo_ros_imu.so">
+      <robotNamespace>/</robotNamespace>
+      <updateRate>50.0</updateRate>
+      <bodyName>base_link</bodyName>
+      <topicName>imu/data</topicName>
+      <accelDrift>0.005 0.005 0.005</accelDrift>
+      <accelGaussianNoise>0.005 0.005 0.005</accelGaussianNoise>
+      <rateDrift>0.005 0.005 0.005 </rateDrift>
+      <rateGaussianNoise>0.005 0.005 0.005 </rateGaussianNoise>
+      <headingDrift>0.005</headingDrift>
+      <headingGaussianNoise>0.005</headingGaussianNoise>
+    </plugin>
+  </gazebo>
 </robot>

Commit message: Adicionar sonar à simulação

File: littlebot_description/urdf/littlebot.xacro (robot description, xacro)
@@ -129,5 +129,14 @@
     <child link="rodinha"/>
     <origin xyz="-0.07 0.0 -0.003" rpy="0 0 0" />
-  </joint>
+    <axis xyz="0 0 1" />
+  </joint>
+    <gazebo reference="rodinha">
+    <mu1 value="1.0"/>
+    <mu2 value="1.0"/>
+    <kp  value="10000000.0" />
+    <kd  value="1.0" />
+    <fdir1 value="1 0 0"/>
+    <turnGravityOff>false</turnGravityOff>
+  </gazebo>
 <!--
 ########################################################################################
@@ -187,4 +196,149 @@
     <child link="motor_direito"/>
     <origin xyz="-0.032 -0.0387 -0.014" rpy="0 0 0" />
+  </joint>
+<!--
+########################################################################################
+Modelagem do sonar 01 "link" "joint"
+########################################################################################
+-->
+  <link name="sonar_01">
+    <visual>
+      <origin xyz="-0.014 0 0" rpy="-1.571 1.571 -1.571" />
+      <geometry>
+	      <mesh filename="package://littlebot_description/meshes/sonar.dae" />
+      </geometry>
+    </visual>
+    <collision>
+      <origin xyz="-0.014 0 0" rpy="0 0 0" />
+      <geometry>
+	      <mesh filename="package://littlebot_description/meshes/sonar.dae" />
+      </geometry>
+    </collision>
+    <inertial>
+      <origin xyz="-0.014 0 0" rpy="0 0 0"/>
+      <mass value="0.015"/>
+      <inertia ixx="5.706e-7"  ixy="6.307e-9"  ixz="2.156e-9" iyy="2.771e-6" iyz="7.710e-9" izz="2.878e-6" />
+    </inertial>
+  </link>
+  <joint name="base_to_sonar_01" type="fixed">
+    <parent link="base_link"/>
+    <child link="sonar_01"/>
+    <origin xyz="0.077 0.0 0.044" rpy="0 0 0" />
+  </joint>
+<!--
+########################################################################################
+Modelagem do sonar 02 "link" "joint"
+########################################################################################
+-->
+  <link name="sonar_02">
+    <visual>
+      <origin xyz="-0.014 0 0" rpy="-1.571 1.571 -1.571" />
+      <geometry>
+	      <mesh filename="package://littlebot_description/meshes/sonar.dae" />
+      </geometry>
+    </visual>
+    <collision>
+      <origin xyz="-0.014 0 0" rpy="0 0 0" />
+      <geometry>
+	      <mesh filename="package://littlebot_description/meshes/sonar.dae" />
+      </geometry>
+    </collision>
+    <inertial>
+      <origin xyz="-0.014 0 0" rpy="0 0 0"/>
+      <mass value="0.015"/>
+      <inertia ixx="5.706e-7"  ixy="6.307e-9"  ixz="2.156e-9" iyy="2.771e-6" iyz="7.710e-9" izz="2.878e-6" />
+    </inertial>
+  </link>
+  <joint name="base_to_sonar_02" type="fixed">
+    <parent link="base_link"/>
+    <child link="sonar_02"/>
+    <origin xyz="0.07211 0.0248 0.044" rpy="0 0 0.3927" />
+  </joint>
+<!--
+########################################################################################
+Modelagem do sonar 03 "link" "joint"
+########################################################################################
+-->
+  <link name="sonar_03">
+    <visual>
+      <origin xyz="-0.014 0.01 0" rpy="-1.571 1.571 -1.571" />
+      <geometry>
+	      <mesh filename="package://littlebot_description/meshes/sonar.dae" />
+      </geometry>
+    </visual>
+    <collision>
+      <origin xyz="-0.014 0.01 0" rpy="0 0 0" />
+      <geometry>
+	      <mesh filename="package://littlebot_description/meshes/sonar.dae" />
+      </geometry>
+    </collision>
+    <inertial>
+      <origin xyz="-0.014 0.01 0" rpy="0 0 0"/>
+      <mass value="0.015"/>
+      <inertia ixx="5.706e-7"  ixy="6.307e-9"  ixz="2.156e-9" iyy="2.771e-6" iyz="7.710e-9" izz="2.878e-6" />
+    </inertial>
+  </link>
+  <joint name="base_to_sonar_03" type="fixed">
+    <parent link="base_link"/>
+    <child link="sonar_03"/>
+    <origin xyz="0.06522 0.038787 0.044" rpy="0 0 0.7854" />
+  </joint>
+  <!--
+########################################################################################
+Modelagem do sonar 04 "link" "joint"
+########################################################################################
+-->
+  <link name="sonar_04">
+    <visual>
+      <origin xyz="-0.014 0 0" rpy="-1.571 1.571 -1.571" />
+      <geometry>
+	      <mesh filename="package://littlebot_description/meshes/sonar.dae" />
+      </geometry>
+    </visual>
+    <collision>
+      <origin xyz="-0.014 0 0" rpy="0 0 0" />
+      <geometry>
+	      <mesh filename="package://littlebot_description/meshes/sonar.dae" />
+      </geometry>
+    </collision>
+    <inertial>
+      <origin xyz="-0.014 0 0" rpy="0 0 0"/>
+      <mass value="0.015"/>
+      <inertia ixx="5.706e-7"  ixy="6.307e-9"  ixz="2.156e-9" iyy="2.771e-6" iyz="7.710e-9" izz="2.878e-6" />
+    </inertial>
+  </link>
+  <joint name="base_to_sonar_04" type="fixed">
+    <parent link="base_link"/>
+    <child link="sonar_04"/>
+    <origin xyz="0.07211 -0.0248 0.044" rpy="0 0 -0.3927" />
+  </joint>
+<!--
+########################################################################################
+Modelagem do sonar 05 "link" "joint"
+########################################################################################
+-->
+  <link name="sonar_05">
+    <visual>
+      <origin xyz="-0.014 0.01 0" rpy="-1.571 1.571 -1.571" />
+      <geometry>
+	      <mesh filename="package://littlebot_description/meshes/sonar.dae" />
+      </geometry>
+    </visual>
+    <collision>
+      <origin xyz="-0.014 0.01 0" rpy="0 0 0" />
+      <geometry>
+	      <mesh filename="package://littlebot_description/meshes/sonar.dae" />
+      </geometry>
+    </collision>
+    <inertial>
+      <origin xyz="-0.014 0.01 0" rpy="0 0 0"/>
+      <mass value="0.015"/>
+      <inertia ixx="5.706e-7"  ixy="6.307e-9"  ixz="2.156e-9" iyy="2.771e-6" iyz="7.710e-9" izz="2.878e-6" />
+    </inertial>
+  </link>
+  <joint name="base_to_sonar_05" type="fixed">
+    <parent link="base_link"/>
+    <child link="sonar_05"/>
+    <origin xyz="0.050935 -0.052781 0.044" rpy="0 0 -0.7854" />
   </joint>
 <!--
@@ -240,3 +394,213 @@
     </plugin>
   </gazebo>
+  <!--
+  ******************************************************************************************
+  SONAR gazebo plugin
+  ******************************************************************************************
+  -->
+  <gazebo reference="sonar_01">
+   <sensor type="ray" name="TeraRanger">
+      <pose>0 0 0 0 0 0</pose>
+      <visualize>false</visualize>
+      <update_rate>50</update_rate>
+      <ray>
+         <scan>
+            <horizontal>
+               <samples>10</samples>
+               <resolution>1</resolution>
+               <min_angle>-0.14835</min_angle>
+               <max_angle>0.14835</max_angle>
+            </horizontal>
+            <vertical>
+               <samples>10</samples>
+               <resolution>1</resolution>
+               <min_angle>-0.14835</min_angle>
+               <max_angle>0.14835</max_angle>
+            </vertical>
+         </scan>
+         <range>
+            <min>0.01</min>
+            <max>2</max>
+            <resolution>0.02</resolution>
+         </range>
+      </ray>
+      <plugin filename="libgazebo_ros_range.so" name="gazebo_ros_range">
+         <gaussianNoise>0.005</gaussianNoise>
+         <alwaysOn>true</alwaysOn>
+         <updateRate>50</updateRate>
+         <topicName>sensor/sonar01</topicName>
+         <frameName>sonar_01</frameName>
+         <radiation>ULTRASOUND</radiation>
+         <fov>0.2967</fov>
+      </plugin>
+   </sensor>
+  </gazebo>
+  <!--
+  ******************************************************************************************
+  SONAR gazebo plugin
+  ******************************************************************************************
+  -->
+  <gazebo reference="sonar_02">
+   <sensor type="ray" name="TeraRanger">
+      <pose>0 0 0 0 0 0</pose>
+      <visualize>false</visualize>
+      <update_rate>50</update_rate>
+      <ray>
+         <scan>
+            <horizontal>
+               <samples>10</samples>
+               <resolution>1</resolution>
+               <min_angle>-0.14835</min_angle>
+               <max_angle>0.14835</max_angle>
+            </horizontal>
+            <vertical>
+               <samples>10</samples>
+               <resolution>1</resolution>
+               <min_angle>-0.14835</min_angle>
+               <max_angle>0.14835</max_angle>
+            </vertical>
+         </scan>
+         <range>
+            <min>0.01</min>
+            <max>2</max>
+            <resolution>0.02</resolution>
+         </range>
+      </ray>
+      <plugin filename="libgazebo_ros_range.so" name="gazebo_ros_range">
+         <gaussianNoise>0.005</gaussianNoise>
+         <alwaysOn>true</alwaysOn>
+         <updateRate>50</updateRate>
+         <topicName>sensor/sonar02</topicName>
+         <frameName>sonar_02</frameName>
+         <radiation>ULTRASOUND</radiation>
+         <fov>0.2967</fov>
+      </plugin>
+   </sensor>
+  </gazebo>
+    <!--
+  ******************************************************************************************
+  SONAR gazebo plugin
+  ******************************************************************************************
+  -->
+  <gazebo reference="sonar_03">
+   <sensor type="ray" name="TeraRanger">
+      <pose>0 0 0 0 0 0</pose>
+      <visualize>false</visualize>
+      <update_rate>50</update_rate>
+      <ray>
+         <scan>
+            <horizontal>
+               <samples>10</samples>
+               <resolution>1</resolution>
+               <min_angle>-0.14835</min_angle>
+               <max_angle>0.14835</max_angle>
+            </horizontal>
+            <vertical>
+               <samples>10</samples>
+               <resolution>1</resolution>
+               <min_angle>-0.14835</min_angle>
+               <max_angle>0.14835</max_angle>
+            </vertical>
+         </scan>
+         <range>
+            <min>0.01</min>
+            <max>2</max>
+            <resolution>0.02</resolution>
+         </range>
+      </ray>
+      <plugin filename="libgazebo_ros_range.so" name="gazebo_ros_range">
+         <gaussianNoise>0.005</gaussianNoise>
+         <alwaysOn>true</alwaysOn>
+         <updateRate>50</updateRate>
+         <topicName>sensor/sonar03</topicName>
+         <frameName>sonar_03</frameName>
+         <radiation>ULTRASOUND</radiation>
+         <fov>0.2967</fov>
+      </plugin>
+   </sensor>
+  </gazebo>
+    <!--
+  ******************************************************************************************
+  SONAR gazebo plugin
+  ******************************************************************************************
+  -->
+  <gazebo reference="sonar_04">
+   <sensor type="ray" name="TeraRanger">
+      <pose>0 0 0 0 0 0</pose>
+      <visualize>false</visualize>
+      <update_rate>50</update_rate>
+      <ray>
+         <scan>
+            <horizontal>
+               <samples>10</samples>
+               <resolution>1</resolution>
+               <min_angle>-0.14835</min_angle>
+               <max_angle>0.14835</max_angle>
+            </horizontal>
+            <vertical>
+               <samples>10</samples>
+               <resolution>1</resolution>
+               <min_angle>-0.14835</min_angle>
+               <max_angle>0.14835</max_angle>
+            </vertical>
+         </scan>
+         <range>
+            <min>0.01</min>
+            <max>2</max>
+            <resolution>0.02</resolution>
+         </range>
+      </ray>
+      <plugin filename="libgazebo_ros_range.so" name="gazebo_ros_range">
+         <gaussianNoise>0.005</gaussianNoise>
+         <alwaysOn>false</alwaysOn>
+         <updateRate>50</updateRate>
+         <topicName>sensor/sonar04</topicName>
+         <frameName>sonar_04</frameName>
+         <radiation>ULTRASOUND</radiation>
+         <fov>0.2967</fov>
+      </plugin>
+   </sensor>
+  </gazebo>
+    <!--
+  ******************************************************************************************
+  SONAR gazebo plugin
+  ******************************************************************************************
+  -->
+  <gazebo reference="sonar_05">
+   <sensor type="ray" name="TeraRanger">
+      <pose>0 0 0 0 0 0</pose>
+      <visualize>false</visualize>
+      <update_rate>50</update_rate>
+      <ray>
+         <scan>
+            <horizontal>
+               <samples>10</samples>
+               <resolution>1</resolution>
+               <min_angle>-0.14835</min_angle>
+               <max_angle>0.14835</max_angle>
+            </horizontal>
+            <vertical>
+               <samples>10</samples>
+               <resolution>1</resolution>
+               <min_angle>-0.14835</min_angle>
+               <max_angle>0.14835</max_angle>
+            </vertical>
+         </scan>
+         <range>
+            <min>0.01</min>
+            <max>2</max>
+            <resolution>0.02</resolution>
+         </range>
+      </ray>
+      <plugin filename="libgazebo_ros_range.so" name="gazebo_ros_range">
+         <gaussianNoise>0.005</gaussianNoise>
+         <alwaysOn>true</alwaysOn>
+         <updateRate>50</updateRate>
+         <topicName>sensor/sonar05</topicName>
+         <frameName>sonar_05</frameName>
+         <radiation>ULTRASOUND</radiation>
+         <fov>0.2967</fov>
+      </plugin>
+   </sensor>
+  </gazebo>
 </robot>

Commit message: atualizar URDF

File: littlebot_description/urdf/littlebot.xacro (robot description, xacro)
@@ -166,5 +166,5 @@
     <parent link="base_link"/>
     <child link="motor_esquerdo"/>
-    <origin xyz="-0.032 0.0387 -0.014" rpy="0 0 0" />
+    <origin xyz="-0.032 0.0412 -0.014" rpy="0 0 0" />
   </joint>
 <!--
@@ -195,5 +195,5 @@
     <parent link="base_link"/>
     <child link="motor_direito"/>
-    <origin xyz="-0.032 -0.0387 -0.014" rpy="0 0 0" />
+    <origin xyz="-0.032 -0.0412 -0.014" rpy="0 0 0" />
   </joint>
 <!--
