Commit message: adicionar transmission à rodinha

File: littlebot_description/urdf/littlebot.xacro (robot description, xacro)
@@ -125,5 +125,5 @@
     </inertial>
   </link>
-  <joint name="base_to_rodinha" type="fixed">
+  <joint name="base_to_rodinha" type="continuous">
     <parent link="base_link"/>
     <child link="rodinha"/>
@@ -131,5 +131,6 @@
     <axis xyz="0 0 1" />
   </joint>
-    <gazebo reference="rodinha">
+  <!--
+  <gazebo reference="rodinha">
     <mu1 value="1.0"/>
     <mu2 value="1.0"/>
@@ -139,4 +140,5 @@
     <turnGravityOff>false</turnGravityOff>
   </gazebo>
+  -->
 <!--
 ########################################################################################
@@ -347,5 +349,5 @@
 ********************************************************************************************
 -->
-  <transmission name="trans_roda_esquerda" type="SimpleTransmission">
+  <transmission name="trans_roda_esquerda">
     <type>transmission_interface/SimpleTransmission</type>
     <joint name="base_to_roda_esquerda">
@@ -362,4 +364,13 @@
     </joint>
     <actuator name="roda_direita_motor">
+      <mechanicalReduction>1</mechanicalReduction>
+    </actuator>
+  </transmission>
+  <transmission name="trans_rodinha" >
+    <type>transmission_interface/SimpleTransmission</type>
+    <joint name="base_to_rodinha">
+      <hardwareInterface>hardware_interface/EffortJointInterface</hardwareInterface>
+    </joint>
+    <actuator name="roda_esquerda_motor">
       <mechanicalReduction>1</mechanicalReduction>
     </actuator>

Commit message: adicionar movimentos da rodinha

File: littlebot_description/urdf/littlebot.xacro (robot description, xacro)
@@ -103,42 +103,89 @@
 <!--
 ########################################################################################
-Modelagem da rodinha "link" "joint"
+Modelagem da rodinha-Caster Mounting Plate "link" "joint"
 ######################################################################################## -->
-  <link name="rodinha">
-    <visual>
-      <!--<origin xyz="0 0 0" rpy="3.14 0 1.571" /> -->
-      <origin xyz="0 0 0" rpy="3.14 0 2.141" />
-      <geometry>
-	      <mesh filename="package://littlebot_description/meshes/Caster_Wheel.dae" />
-      </geometry>
-    </visual>
-    <collision>
-      <origin xyz="0 0 0" rpy="3.14 0 2.141" />
-      <geometry>
-	      <mesh filename="package://littlebot_description/meshes/Caster_Wheel.dae" />
-      </geometry>
-    </collision>
-    <inertial>
-      <origin xyz="0 0 0" rpy="3.14 0 2.141"/>
+  <link name="caster_mounting">
+    <visual>
+      <origin xyz="0 0 0" rpy="3.14 0 1.571" />
+      <geometry>
+	      <mesh filename="package://littlebot_description/meshes/Caster_Mounting_Plate.dae" />
+      </geometry>
+    </visual>
+    <collision>
+      <origin xyz="0 0 0" rpy="3.14 0 1.571" />
+      <geometry>
+	      <mesh filename="package://littlebot_description/meshes/Caster_Mounting_Plate.dae" />
+      </geometry>
+    </collision>
+    <inertial>
+      <origin xyz="0 0 0" rpy="3.14 0 1.571"/>
       <mass value="0.073"/>
       <inertia ixx="5.470e-6"  ixy="4.042e-7"  ixz="3.515e-7" iyy="7.169e-6" iyz="-3.645e-7" izz="7.383e-6" />
     </inertial>
   </link>
-  <joint name="base_to_rodinha" type="continuous">
-    <parent link="base_link"/>
-    <child link="rodinha"/>
-    <origin xyz="-0.07 0.0 -0.003" rpy="0 0 0" />
+  <joint name="base_to_caster_mounting" type="fixed">
+    <parent link="base_link"/>
+    <child link="caster_mounting"/>
+    <origin xyz="-0.0753 0.0 -0.003" rpy="0 0 0" />
+    <!--<axis xyz="0 0 1" />-->
+  </joint>
+<!--
+########################################################################################
+Modelagem da rodinha-Caster Wheel Plate "link" "joint"
+######################################################################################## -->
+  <link name="caster_wheel">
+    <visual>
+      <origin xyz="0 0 0" rpy="3.14 0 1.571" />
+      <geometry>
+	      <mesh filename="package://littlebot_description/meshes/Caster_Wheel_Plate.dae" />
+      </geometry>
+    </visual>
+    <collision>
+      <origin xyz="0 0 0" rpy="3.14 0 1.571" />
+      <geometry>
+	      <mesh filename="package://littlebot_description/meshes/Caster_Wheel_Plate.dae" />
+      </geometry>
+    </collision>
+    <inertial>
+      <origin xyz="0 0 0" rpy="3.14 0 1.571"/>
+      <mass value="0.073"/>
+      <inertia ixx="5.470e-6"  ixy="4.042e-7"  ixz="3.515e-7" iyy="7.169e-6" iyz="-3.645e-7" izz="7.383e-6" />
+    </inertial>
+  </link>
+  <joint name="caster_mounting_to_caster_wheel" type="continuous">
+    <parent link="caster_mounting"/>
+    <child link="caster_wheel"/>
+    <origin xyz="-0.0 0.0 -0.00623" rpy="0 0 0" />
     <axis xyz="0 0 1" />
   </joint>
-  <!--
-  <gazebo reference="rodinha">
-    <mu1 value="1.0"/>
-    <mu2 value="1.0"/>
-    <kp  value="10000000.0" />
-    <kd  value="1.0" />
-    <fdir1 value="1 0 0"/>
-    <turnGravityOff>false</turnGravityOff>
-  </gazebo>
-  -->
+<!--
+########################################################################################
+Modelagem da rodinha-Wheel "link" "joint"
+######################################################################################## -->
+  <link name="wheel">
+    <visual>
+      <origin xyz="0 0 0" rpy="3.14 0 1.571" />
+      <geometry>
+	      <mesh filename="package://littlebot_description/meshes/Wheel.dae" />
+      </geometry>
+    </visual>
+    <collision>
+      <origin xyz="0 0 0" rpy="3.14 0 1.571" />
+      <geometry>
+	      <mesh filename="package://littlebot_description/meshes/Wheel.dae" />
+      </geometry>
+    </collision>
+    <inertial>
+      <origin xyz="0 0 0" rpy="3.14 0 1.571"/>
+      <mass value="0.073"/>
+      <inertia ixx="5.470e-6"  ixy="4.042e-7"  ixz="3.515e-7" iyy="7.169e-6" iyz="-3.645e-7" izz="7.383e-6" />
+    </inertial>
+  </link>
+  <joint name="caster_wheel_to_wheel" type="continuous">
+    <parent link="caster_wheel"/>
+    <child link="wheel"/>
+    <origin xyz="0.0 0.0148 -0.0153" rpy="0 0 0" />
+    <axis xyz="1 0 0" />
+  </joint>
 <!--
 ########################################################################################
@@ -367,10 +414,19 @@
     </actuator>
   </transmission>
-  <transmission name="trans_rodinha" >
+  <transmission name="trans_caster" >
     <type>transmission_interface/SimpleTransmission</type>
-    <joint name="base_to_rodinha">
+    <joint name="caster_mounting_to_caster_wheel">
       <hardwareInterface>hardware_interface/EffortJointInterface</hardwareInterface>
     </joint>
-    <actuator name="roda_esquerda_motor">
+    <actuator name="act_caster">
+      <mechanicalReduction>1</mechanicalReduction>
+    </actuator>
+  </transmission>
+  <transmission name="trans_wheel" >
+    <type>transmission_interface/SimpleTransmission</type>
+    <joint name="caster_wheel_to_wheel">
+      <hardwareInterface>hardware_interface/EffortJointInterface</hardwareInterface>
+    </joint>
+    <actuator name="act_wheel">
       <mechanicalReduction>1</mechanicalReduction>
     </actuator>

Commit message: corrigir ERROR URDF

File: littlebot_description/urdf/littlebot.xacro (robot description, xacro)
@@ -1,4 +1,6 @@
 <?xml version="1.0"?>
 <robot name="littlebot" xmlns:xacro="http://www.ros.org/wiki/xacro">
+ <link name="base_link">
+ </link>
  <!--
 ########################################################################################
@@ -6,5 +8,5 @@
 ########################################################################################
 -->
- <link name="base_link">
+ <link name="chassis">
     <visual>
       <origin xyz="0 0 0" rpy="1.571 0 1.571" />
@@ -25,4 +27,9 @@
     </inertial>
   </link>
+  <joint name="base_to_chassis" type="fixed">
+    <parent link="base_link"/>
+    <child link="chassis"/>
+    <origin xyz="0.0 0.0 0.0" rpy="0 0 0" />
+  </joint>
 <!--
 ########################################################################################
@@ -440,4 +447,5 @@
     <plugin name="gazebo_ros_control" filename="libgazebo_ros_control.so">
       <robotNamespace>/</robotNamespace>
+      <legacyModeNS>true</legacyModeNS>
     </plugin>
   </gazebo>

Commit message: Valores de inertcia da rodinha

File: littlebot_description/urdf/littlebot.xacro (robot description, xacro)
@@ -127,6 +127,6 @@
     <inertial>
       <origin xyz="0 0 0" rpy="3.14 0 1.571"/>
-      <mass value="0.073"/>
-      <inertia ixx="5.470e-6"  ixy="4.042e-7"  ixz="3.515e-7" iyy="7.169e-6" iyz="-3.645e-7" izz="7.383e-6" />
+      <mass value="0.01946206"/>
+      <inertia ixx="1.561e-6"  ixy="0.000e+0"  ixz="0.000e+0" iyy="1.944e-6" iyz="0.000e+0" izz="3.350e-6" />
     </inertial>
   </link>
@@ -135,5 +135,4 @@
     <child link="caster_mounting"/>
     <origin xyz="-0.0753 0.0 -0.003" rpy="0 0 0" />
-    <!--<axis xyz="0 0 1" />-->
   </joint>
 <!--
@@ -156,6 +155,6 @@
     <inertial>
       <origin xyz="0 0 0" rpy="3.14 0 1.571"/>
-      <mass value="0.073"/>
-      <inertia ixx="5.470e-6"  ixy="4.042e-7"  ixz="3.515e-7" iyy="7.169e-6" iyz="-3.645e-7" izz="7.383e-6" />
+      <mass value="0.00982010"/>
+      <inertia ixx="8.398e-7"  ixy="-1.517e-14"  ixz="-1.601e-7" iyy="8.400e-7" iyz="1.155e-14" izz="1.340e-6" />
     </inertial>
   </link>
@@ -185,6 +184,6 @@
     <inertial>
       <origin xyz="0 0 0" rpy="3.14 0 1.571"/>
-      <mass value="0.073"/>
-      <inertia ixx="5.470e-6"  ixy="4.042e-7"  ixz="3.515e-7" iyy="7.169e-6" iyz="-3.645e-7" izz="7.383e-6" />
+      <mass value="0.007 kg"/>
+      <inertia ixx="3.569e-7"  ixy="0.000e+0"  ixz="0.000e+0" iyy="5.344e-7" iyz="0.000e+0" izz="3.569e-7" />
     </inertial>
   </link>

Commit message: Mudar link da IMU de base_link para chassis

File: littlebot_description/urdf/littlebot.xacro (robot description, xacro)
@@ -184,5 +184,5 @@
     <inertial>
       <origin xyz="0 0 0" rpy="3.14 0 1.571"/>
-      <mass value="0.007 kg"/>
+      <mass value="0.007"/>
       <inertia ixx="3.569e-7"  ixy="0.000e+0"  ixz="0.000e+0" iyy="5.344e-7" iyz="0.000e+0" izz="3.569e-7" />
     </inertial>
@@ -458,5 +458,5 @@
       <robotNamespace>/</robotNamespace>
       <updateRate>50.0</updateRate>
-      <bodyName>base_link</bodyName>
+      <bodyName>chassis</bodyName>
       <topicName>imu/data</topicName>
       <accelDrift>0.005 0.005 0.005</accelDrift>

Commit message: ajustes no URDF

File: littlebot_description/urdf/littlebot.xacro (robot description, xacro)
@@ -31,4 +31,5 @@
     <child link="chassis"/>
     <origin xyz="0.0 0.0 0.0" rpy="0 0 0" />
+    <axis xyz="0 1 0" />
   </joint>
 <!--
@@ -165,4 +166,12 @@
     <axis xyz="0 0 1" />
   </joint>
+  <gazebo reference="caster_wheel">
+    <mu1 value="1.0"/>
+    <mu2 value="1.0"/>
+    <kp  value="10000.0" />
+    <kd  value="1.0" />
+    <fdir1 value="1 0 0"/>
+    <turnGravityOff>false</turnGravityOff>
+  </gazebo>
 <!--
 ########################################################################################
@@ -194,4 +203,12 @@
     <axis xyz="1 0 0" />
   </joint>
+  <gazebo reference="wheel">
+    <mu1 value="1.0"/>
+    <mu2 value="1.0"/>
+    <kp  value="10000000.0" />
+    <kd  value="1.0" />
+    <fdir1 value="1 0 0"/>
+    <turnGravityOff>false</turnGravityOff>
+  </gazebo>
 <!--
 ########################################################################################

Commit message: Ajustar colisions para os meshs do sonar

File: littlebot_description/urdf/littlebot.xacro (robot description, xacro)
@@ -282,11 +282,11 @@
     </visual>
     <collision>
-      <origin xyz="-0.014 0 0" rpy="0 0 0" />
-      <geometry>
-	      <mesh filename="package://littlebot_description/meshes/sonar.dae" />
-      </geometry>
-    </collision>
-    <inertial>
-      <origin xyz="-0.014 0 0" rpy="0 0 0"/>
+      <origin xyz="-0.014 0 0" rpy="-1.571 1.571 -1.571" />
+      <geometry>
+	      <mesh filename="package://littlebot_description/meshes/sonar.dae" />
+      </geometry>
+    </collision>
+    <inertial>
+      <origin xyz="-0.014 0 0" rpy="-1.571 1.571 -1.571"/>
       <mass value="0.015"/>
       <inertia ixx="5.706e-7"  ixy="6.307e-9"  ixz="2.156e-9" iyy="2.771e-6" iyz="7.710e-9" izz="2.878e-6" />
@@ -311,11 +311,11 @@
     </visual>
     <collision>
-      <origin xyz="-0.014 0 0" rpy="0 0 0" />
-      <geometry>
-	      <mesh filename="package://littlebot_description/meshes/sonar.dae" />
-      </geometry>
-    </collision>
-    <inertial>
-      <origin xyz="-0.014 0 0" rpy="0 0 0"/>
+      <origin xyz="-0.014 0 0" rpy="-1.571 1.571 -1.571" />
+      <geometry>
+	      <mesh filename="package://littlebot_description/meshes/sonar.dae" />
+      </geometry>
+    </collision>
+    <inertial>
+      <origin xyz="-0.014 0 0" rpy="-1.571 1.571 -1.571"/>
       <mass value="0.015"/>
       <inertia ixx="5.706e-7"  ixy="6.307e-9"  ixz="2.156e-9" iyy="2.771e-6" iyz="7.710e-9" izz="2.878e-6" />
@@ -340,11 +340,11 @@
     </visual>
     <collision>
-      <origin xyz="-0.014 0.01 0" rpy="0 0 0" />
-      <geometry>
-	      <mesh filename="package://littlebot_description/meshes/sonar.dae" />
-      </geometry>
-    </collision>
-    <inertial>
-      <origin xyz="-0.014 0.01 0" rpy="0 0 0"/>
+      <origin xyz="-0.014 0.01 0" rpy="-1.571 1.571 -1.571" />
+      <geometry>
+	      <mesh filename="package://littlebot_description/meshes/sonar.dae" />
+      </geometry>
+    </collision>
+    <inertial>
+      <origin xyz="-0.014 0.01 0" rpy="-1.571 1.571 -1.571"/>
       <mass value="0.015"/>
       <inertia ixx="5.706e-7"  ixy="6.307e-9"  ixz="2.156e-9" iyy="2.771e-6" iyz="7.710e-9" izz="2.878e-6" />
@@ -369,11 +369,11 @@
     </visual>
     <collision>
-      <origin xyz="-0.014 0 0" rpy="0 0 0" />
-      <geometry>
-	      <mesh filename="package://littlebot_description/meshes/sonar.dae" />
-      </geometry>
-    </collision>
-    <inertial>
-      <origin xyz="-0.014 0 0" rpy="0 0 0"/>
+      <origin xyz="-0.014 0 0" rpy="-1.571 1.571 -1.571" />
+      <geometry>
+	      <mesh filename="package://littlebot_description/meshes/sonar.dae" />
+      </geometry>
+    </collision>
+    <inertial>
+      <origin xyz="-0.014 0 0" rpy="-1.571 1.571 -1.571"/>
       <mass value="0.015"/>
       <inertia ixx="5.706e-7"  ixy="6.307e-9"  ixz="2.156e-9" iyy="2.771e-6" iyz="7.710e-9" izz="2.878e-6" />
@@ -398,11 +398,11 @@
     </visual>
     <collision>
-      <origin xyz="-0.014 0.01 0" rpy="0 0 0" />
-      <geometry>
-	      <mesh filename="package://littlebot_description/meshes/sonar.dae" />
-      </geometry>
-    </collision>
-    <inertial>
-      <origin xyz="-0.014 0.01 0" rpy="0 0 0"/>
+      <origin xyz="-0.014 0.01 0" rpy="-1.571 1.571 -1.571" />
+      <geometry>
+	      <mesh filename="package://littlebot_description/meshes/sonar.dae" />
+      </geometry>
+    </collision>
+    <inertial>
+      <origin xyz="-0.014 0.01 0" rpy="-1.571 1.571 -1.571"/>
       <mass value="0.015"/>
       <inertia ixx="5.706e-7"  ixy="6.307e-9"  ixz="2.156e-9" iyy="2.771e-6" iyz="7.710e-9" izz="2.878e-6" />

Commit message: Atualizar README

File: littlebot_description/urdf/littlebot.xacro (robot description, xacro)
@@ -58,5 +58,5 @@
   </link>
   <joint name="base_to_roda_esquerda" type="continuous">
-    <parent link="base_link"/>
+    <parent link="chassis"/>
     <child link="roda_esquerda"/>
     <origin xyz="0.005 0.07393 -0.014" rpy="0 0 0" />
@@ -96,5 +96,5 @@
   </link>
   <joint name="base_to_roda_direita" type="continuous">
-    <parent link="base_link"/>
+    <parent link="chassis"/>
     <child link="roda_direita"/>
     <origin xyz="0.005 -0.07393 -0.014" rpy="0 0 0" />
@@ -133,5 +133,5 @@
   </link>
   <joint name="base_to_caster_mounting" type="fixed">
-    <parent link="base_link"/>
+    <parent link="chassis"/>
     <child link="caster_mounting"/>
     <origin xyz="-0.0753 0.0 -0.003" rpy="0 0 0" />
@@ -236,5 +236,5 @@
   </link>
   <joint name="base_to_motor_esquerdo" type="fixed">
-    <parent link="base_link"/>
+    <parent link="chassis"/>
     <child link="motor_esquerdo"/>
     <origin xyz="-0.032 0.0412 -0.014" rpy="0 0 0" />
@@ -265,5 +265,5 @@
   </link>
   <joint name="base_to_motor_direito" type="fixed">
-    <parent link="base_link"/>
+    <parent link="chassis"/>
     <child link="motor_direito"/>
     <origin xyz="-0.032 -0.0412 -0.014" rpy="0 0 0" />
@@ -294,5 +294,5 @@
   </link>
   <joint name="base_to_sonar_01" type="fixed">
-    <parent link="base_link"/>
+    <parent link="chassis"/>
     <child link="sonar_01"/>
     <origin xyz="0.077 0.0 0.044" rpy="0 0 0" />
@@ -323,5 +323,5 @@
   </link>
   <joint name="base_to_sonar_02" type="fixed">
-    <parent link="base_link"/>
+    <parent link="chassis"/>
     <child link="sonar_02"/>
     <origin xyz="0.07211 0.0248 0.044" rpy="0 0 0.3927" />
@@ -352,5 +352,5 @@
   </link>
   <joint name="base_to_sonar_03" type="fixed">
-    <parent link="base_link"/>
+    <parent link="chassis"/>
     <child link="sonar_03"/>
     <origin xyz="0.06522 0.038787 0.044" rpy="0 0 0.7854" />
@@ -381,5 +381,5 @@
   </link>
   <joint name="base_to_sonar_04" type="fixed">
-    <parent link="base_link"/>
+    <parent link="chassis"/>
     <child link="sonar_04"/>
     <origin xyz="0.07211 -0.0248 0.044" rpy="0 0 -0.3927" />
@@ -410,5 +410,5 @@
   </link>
   <joint name="base_to_sonar_05" type="fixed">
-    <parent link="base_link"/>
+    <parent link="chassis"/>
     <child link="sonar_05"/>
     <origin xyz="0.050935 -0.052781 0.044" rpy="0 0 -0.7854" />

Commit message: Incluir macros Xacro para a modelagem das rodas laterais

File: littlebot_description/urdf/littlebot.xacro (robot description, xacro)
@@ -1,4 +1,6 @@
 <?xml version="1.0"?>
 <robot name="littlebot" xmlns:xacro="http://www.ros.org/wiki/xacro">
+  <!-- Included URDF/XACRO Files -->
+  <xacro:include filename="$(find littlebot_description)/urdf/rodas.xacro" />
  <link name="base_link">
  </link>
@@ -35,78 +37,13 @@
 <!--
 ########################################################################################
-Modelagem da roda esquerda "link" "joint"
-########################################################################################
--->
-  <link name="roda_esquerda">
-    <visual>
-      <origin xyz="0 -0.0115 0" rpy="0 0 1.571" />
-      <geometry>
-	      <mesh filename="package://littlebot_description/meshes/roda.dae" />
-      </geometry>
-    </visual>
-    <collision>
-      <origin xyz="0 -0.0115 0" rpy="0 0 1.571" />
-      <geometry>
-	      <mesh filename="package://littlebot_description/meshes/roda.dae" />
-      </geometry>
-    </collision>
-    <inertial>
-      <origin xyz="0 -0.0115 0" rpy="0 0 1.571"/>
-      <mass value="0.041"/>
-      <inertia ixx="2.967e-5"  ixy="-7.675e-15"  ixz="-4.765e-14" iyy="1.616e-5" iyz="-1.121e-16" izz="1.616e-5" />
-    </inertial>
-  </link>
-  <joint name="base_to_roda_esquerda" type="continuous">
-    <parent link="chassis"/>
-    <child link="roda_esquerda"/>
+Modelagem das rodas macro Xacro
+########################################################################################
+-->
+  <xacro:littlebot_wheel lado_roda="esquerda">
     <origin xyz="0.005 0.07393 -0.014" rpy="0 0 0" />
-    <axis xyz="0 1 0" />
-  </joint>
-  <gazebo reference="roda_esquerda">
-    <mu1 value="1.0"/>
-    <mu2 value="1.0"/>
-    <kp  value="10000000.0" />
-    <kd  value="1.0" />
-    <fdir1 value="1 0 0"/>
-    <turnGravityOff>false</turnGravityOff>
-  </gazebo>
-<!--
-########################################################################################
-Modelagem da roda direita "link" "joint"
-########################################################################################
--->
-  <link name="roda_direita">
-    <visual>
-      <origin xyz="0 0.0115 0" rpy="0 0 -1.571" />
-      <geometry>
-	      <mesh filename="package://littlebot_description/meshes/roda.dae" />
-      </geometry>
-    </visual>
-    <collision>
-      <origin xyz="0 0.0115 0" rpy="0 0 -1.571 " />
-      <geometry>
-	      <mesh filename="package://littlebot_description/meshes/roda.dae" />
-      </geometry>
-    </collision>
-    <inertial>
-      <origin xyz="0 0.0115 0" rpy="0 0 -1.571"/>
-      <mass value="0.041"/>
-      <inertia ixx="2.967e-5"  ixy="-7.675e-15"  ixz="-4.765e-14" iyy="1.616e-5" iyz="-1.121e-16" izz="1.616e-5" />
-    </inertial>
-  </link>
-  <joint name="base_to_roda_direita" type="continuous">
-    <parent link="chassis"/>
-    <child link="roda_direita"/>
+  </xacro:littlebot_wheel>
+  <xacro:littlebot_wheel lado_roda="direita">
     <origin xyz="0.005 -0.07393 -0.014" rpy="0 0 0" />
-    <axis xyz="0 1 0" />
-  </joint>
-  <gazebo reference="roda_direita">
-    <mu1 value="1.0"/>
-    <mu2 value="1.0"/>
-    <kp  value="10000000.0" />
-    <kd  value="1.0" />
-    <fdir1 value="1 0 0"/>
-    <turnGravityOff>false</turnGravityOff>
-  </gazebo>
+  </xacro:littlebot_wheel>
 <!--
 ########################################################################################
@@ -419,22 +356,4 @@
 ********************************************************************************************
 -->
-  <transmission name="trans_roda_esquerda">
-    <type>transmission_interface/SimpleTransmission</type>
-    <joint name="base_to_roda_esquerda">
-      <hardwareInterface>hardware_interface/VelocityJointInterface</hardwareInterface>
-    </joint>
-    <actuator name="roda_esquerda_motor">
-      <mechanicalReduction>1</mechanicalReduction>
-    </actuator>
-  </transmission>
-  <transmission name="trans_roda_direita">
-    <type>transmission_interface/SimpleTransmission</type>
-    <joint name="base_to_roda_direita">
-      <hardwareInterface>hardware_interface/VelocityJointInterface</hardwareInterface>
-    </joint>
-    <actuator name="roda_direita_motor">
-      <mechanicalReduction>1</mechanicalReduction>
-    </actuator>
-  </transmission>
   <transmission name="trans_caster" >
     <type>transmission_interface/SimpleTransmission</type>
