Commit message: Incluir xacro paras as rodas, ajustar posicionamento das rodas para a macro

File: littlebot_description/urdf/littlebot.xacro (robot description, xacro)
@@ -3,4 +3,5 @@
   <!-- Included URDF/XACRO Files -->
   <xacro:include filename="$(find littlebot_description)/urdf/rodas.xacro" />
+  <xacro:include filename="$(find littlebot_description)/urdf/sonar.xacro" />
  <link name="base_link">
  </link>
@@ -41,8 +42,8 @@
 -->
   <xacro:littlebot_wheel lado_roda="esquerda">
-    <origin xyz="0.005 0.07393 -0.014" rpy="0 0 0" />
+    <origin xyz="0.005 0.07393 -0.014" rpy="0 0 1.571" />
   </xacro:littlebot_wheel>
   <xacro:littlebot_wheel lado_roda="direita">
-    <origin xyz="0.005 -0.07393 -0.014" rpy="0 0 0" />
+    <origin xyz="0.005 -0.07393 -0.014" rpy="0 0 -1.571" />
   </xacro:littlebot_wheel>
 <!--
@@ -141,6 +142,6 @@
   </joint>
   <gazebo reference="wheel">
-    <mu1 value="1.0"/>
-    <mu2 value="1.0"/>
+    <mu1 value="100000.0"/>
+    <mu2 value="100.0"/>
     <kp  value="10000000.0" />
     <kd  value="1.0" />
@@ -211,4 +212,5 @@
 ########################################################################################
 -->
+<!--
   <link name="sonar_01">
     <visual>
@@ -235,4 +237,8 @@
     <origin xyz="0.077 0.0 0.044" rpy="0 0 0" />
   </joint>
+-->
+  <xacro:littlebot_sonar sonar_numero="01">
+    <origin xyz="0.077 0.0 0.044" rpy="0 0 0" />
+  </xacro:littlebot_sonar>
 <!--
 ########################################################################################

File: littlebot_description/urdf/rodas.xacro (robot description, xacro)
@@ -4,5 +4,5 @@
 		<link name="roda_${lado_roda}">
 			<visual>
-				<origin xyz="0 -0.0115 0" rpy="0 0 1.571" />
+				<origin xyz="-0.01 0 0" rpy="0 0 0" />
 				<geometry>
 					<mesh filename="package://littlebot_description/meshes/roda.dae" />
@@ -10,5 +10,5 @@
 			</visual>
 			<collision>
-				<origin xyz="0 -0.0115 0" rpy="0 0 1.571" />
+				<origin xyz="-0.01 0 0" rpy="0 0 0" />
 				<geometry>
 					<mesh filename="package://littlebot_description/meshes/roda.dae" />
@@ -16,5 +16,5 @@
 			</collision>
 			<inertial>
-        <origin xyz="0 -0.0115 0" rpy="0 0 1.571"/>
+        		<origin xyz="-0.01 0 0" rpy="0 0 0"/>
 				<mass value="0.041"/>
 				<inertia ixx="2.967e-5"  ixy="-7.675e-15"  ixz="-4.765e-14" iyy="1.616e-5" iyz="-1.121e-16" izz="1.616e-5" />
@@ -32,15 +32,15 @@
 			<child link="roda_${lado_roda}"/>
 			<xacro:insert_block name="joint_pose"/>
-			<axis xyz="0 1 0" rpy="0 0 0" />
+			<axis xyz="1 0 0" rpy="0 0 0" />
 		</joint>
-    <transmission name="trans_roda_${lado_roda}">
-      <type>transmission_interface/SimpleTransmission</type>
-      <joint name="base_to_roda_${lado_roda}">
-          <hardwareInterface>hardware_interface/VelocityJointInterface</hardwareInterface>
-      </joint>
-      <actuator name="roda_${lado_roda}_motor">
-          <mechanicalReduction>1</mechanicalReduction>
-      </actuator>
-    </transmission>
+		<transmission name="trans_roda_${lado_roda}">
+			<type>transmission_interface/SimpleTransmission</type>
+			<joint name="base_to_roda_${lado_roda}">
+				<hardwareInterface>hardware_interface/VelocityJointInterface</hardwareInterface>
+			</joint>
+			<actuator name="roda_${lado_roda}_motor">
+				<mechanicalReduction>1</mechanicalReduction>
+			</actuator>
+		</transmission>
 	</xacro:macro>
 </robot>

Commit message: Incluir macro xacro para posicionamento do sonar

File: littlebot_description/urdf/littlebot.xacro (robot description, xacro)
@@ -4,4 +4,9 @@
   <xacro:include filename="$(find littlebot_description)/urdf/rodas.xacro" />
   <xacro:include filename="$(find littlebot_description)/urdf/sonar.xacro" />
+ <!--
+########################################################################################
+Modelagem base_link "link"
+########################################################################################
+-->
  <link name="base_link">
  </link>
@@ -38,5 +43,5 @@
 <!--
 ########################################################################################
-Modelagem das rodas macro Xacro
+Modelagem das rodas macro Xacro "link" "gazebo" "joint" "transmission
 ########################################################################################
 -->
@@ -49,6 +54,27 @@
 <!--
 ########################################################################################
+Modelagem do sonar "link" "joint"
+########################################################################################
+-->
+  <xacro:littlebot_sonar sonar_numero="01">
+    <origin xyz="0.077 0.0 0.044" rpy="0 0 0" />
+  </xacro:littlebot_sonar>
+  <xacro:littlebot_sonar sonar_numero="02">
+    <origin xyz="0.07211 0.0248 0.044" rpy="0 0 0.3927"/>
+  </xacro:littlebot_sonar>
+  <xacro:littlebot_sonar sonar_numero="03">
+    <origin xyz="0.06522 0.038787 0.044" rpy="0 0 0.7854" />
+  </xacro:littlebot_sonar>
+  <xacro:littlebot_sonar sonar_numero="04">
+    <origin xyz="0.07211 -0.0248 0.044" rpy="0 0 -0.3927"/>
+  </xacro:littlebot_sonar>
+  <xacro:littlebot_sonar sonar_numero="05">
+    <origin xyz="0.050935 -0.052781 0.044" rpy="0 0 -0.7854"/>
+  </xacro:littlebot_sonar>
+<!--
+########################################################################################
 Modelagem da rodinha-Caster Mounting Plate "link" "joint"
-######################################################################################## -->
+########################################################################################
+-->
   <link name="caster_mounting">
     <visual>
@@ -78,5 +104,6 @@
 ########################################################################################
 Modelagem da rodinha-Caster Wheel Plate "link" "joint"
-######################################################################################## -->
+########################################################################################
+-->
   <link name="caster_wheel">
     <visual>
@@ -104,262 +131,4 @@
     <axis xyz="0 0 1" />
   </joint>
-  <gazebo reference="caster_wheel">
-    <mu1 value="1.0"/>
-    <mu2 value="1.0"/>
-    <kp  value="10000.0" />
-    <kd  value="1.0" />
-    <fdir1 value="1 0 0"/>
-    <turnGravityOff>false</turnGravityOff>
-  </gazebo>
-<!--
-########################################################################################
-Modelagem da rodinha-Wheel "link" "joint"
-######################################################################################## -->
-  <link name="wheel">
-    <visual>
-      <origin xyz="0 0 0" rpy="3.14 0 1.571" />
-      <geometry>
-	      <mesh filename="package://littlebot_description/meshes/Wheel.dae" />
-      </geometry>
-    </visual>
-    <collision>
-      <origin xyz="0 0 0" rpy="3.14 0 1.571" />
-      <geometry>
-	      <mesh filename="package://littlebot_description/meshes/Wheel.dae" />
-      </geometry>
-    </collision>
-    <inertial>
-      <origin xyz="0 0 0" rpy="3.14 0 1.571"/>
-      <mass value="0.007"/>
-      <inertia ixx="3.569e-7"  ixy="0.000e+0"  ixz="0.000e+0" iyy="5.344e-7" iyz="0.000e+0" izz="3.569e-7" />
-    </inertial>
-  </link>
-  <joint name="caster_wheel_to_wheel" type="continuous">
-    <parent link="caster_wheel"/>
-    <child link="wheel"/>
-    <origin xyz="0.0 0.0148 -0.0153" rpy="0 0 0" />
-    <axis xyz="1 0 0" />
-  </joint>
-  <gazebo reference="wheel">
-    <mu1 value="100000.0"/>
-    <mu2 value="100.0"/>
-    <kp  value="10000000.0" />
-    <kd  value="1.0" />
-    <fdir1 value="1 0 0"/>
-    <turnGravityOff>false</turnGravityOff>
-  </gazebo>
-<!--
-########################################################################################
-Modelagem do motor esquerdo "link" "joint"
-########################################################################################
--->
-  <link name="motor_esquerdo">
-    <visual>
-      <origin xyz="0 0 0" rpy="0 0 0" />
-      <geometry>
-	      <mesh filename="package://littlebot_description/meshes/motor.dae" />
-      </geometry>
-    </visual>
-    <collision>
-      <origin xyz="0 0 0" rpy="0 0 0" />
-      <geometry>
-	      <mesh filename="package://littlebot_description/meshes/motor.dae" />
-      </geometry>
-    </collision>
-    <inertial>
-      <origin xyz="0 0 0" rpy="0 0 0"/>
-      <mass value="0.09"/>
-      <inertia ixx="0"  ixy="0"  ixz="0" iyy="0" iyz="0" izz="0" />
-    </inertial>
-  </link>
-  <joint name="base_to_motor_esquerdo" type="fixed">
-    <parent link="chassis"/>
-    <child link="motor_esquerdo"/>
-    <origin xyz="-0.032 0.0412 -0.014" rpy="0 0 0" />
-  </joint>
-<!--
-########################################################################################
-Modelagem do motor direito "link" "joint"
-########################################################################################
--->
-  <link name="motor_direito">
-    <visual>
-      <origin xyz="0 0 0" rpy="0 0 0" />
-      <geometry>
-	      <mesh filename="package://littlebot_description/meshes/motor.dae" />
-      </geometry>
-    </visual>
-    <collision>
-      <origin xyz="0 0 0" rpy="0 0 0" />
-      <geometry>
-	      <mesh filename="package://littlebot_description/meshes/motor.dae" />
-      </geometry>
-    </collision>
-    <inertial>
-      <origin xyz="0 0 0" rpy="0 0 0"/>
-      <mass value="0.09"/>
-      <inertia ixx="0"  ixy="0"  ixz="0" iyy="0" iyz="0" izz="0" />
-    </inertial>
-  </link>
-  <joint name="base_to_motor_direito" type="fixed">
-    <parent link="chassis"/>
-    <child link="motor_direito"/>
-    <origin xyz="-0.032 -0.0412 -0.014" rpy="0 0 0" />
-  </joint>
-<!--
-########################################################################################
-Modelagem do sonar 01 "link" "joint"
-########################################################################################
--->
-<!--
-  <link name="sonar_01">
-    <visual>
-      <origin xyz="-0.014 0 0" rpy="-1.571 1.571 -1.571" />
-      <geometry>
-	      <mesh filename="package://littlebot_description/meshes/sonar.dae" />
-      </geometry>
-    </visual>
-    <collision>
-      <origin xyz="-0.014 0 0" rpy="-1.571 1.571 -1.571" />
-      <geometry>
-	      <mesh filename="package://littlebot_description/meshes/sonar.dae" />
-      </geometry>
-    </collision>
-    <inertial>
-      <origin xyz="-0.014 0 0" rpy="-1.571 1.571 -1.571"/>
-      <mass value="0.015"/>
-      <inertia ixx="5.706e-7"  ixy="6.307e-9"  ixz="2.156e-9" iyy="2.771e-6" iyz="7.710e-9" izz="2.878e-6" />
-    </inertial>
-  </link>
-  <joint name="base_to_sonar_01" type="fixed">
-    <parent link="chassis"/>
-    <child link="sonar_01"/>
-    <origin xyz="0.077 0.0 0.044" rpy="0 0 0" />
-  </joint>
--->
-  <xacro:littlebot_sonar sonar_numero="01">
-    <origin xyz="0.077 0.0 0.044" rpy="0 0 0" />
-  </xacro:littlebot_sonar>
-<!--
-########################################################################################
-Modelagem do sonar 02 "link" "joint"
-########################################################################################
--->
-  <link name="sonar_02">
-    <visual>
-      <origin xyz="-0.014 0 0" rpy="-1.571 1.571 -1.571" />
-      <geometry>
-	      <mesh filename="package://littlebot_description/meshes/sonar.dae" />
-      </geometry>
-    </visual>
-    <collision>
-      <origin xyz="-0.014 0 0" rpy="-1.571 1.571 -1.571" />
-      <geometry>
-	      <mesh filename="package://littlebot_description/meshes/sonar.dae" />
-      </geometry>
-    </collision>
-    <inertial>
-      <origin xyz="-0.014 0 0" rpy="-1.571 1.571 -1.571"/>
-      <mass value="0.015"/>
-      <inertia ixx="5.706e-7"  ixy="6.307e-9"  ixz="2.156e-9" iyy="2.771e-6" iyz="7.710e-9" izz="2.878e-6" />
-    </inertial>
-  </link>
-  <joint name="base_to_sonar_02" type="fixed">
-    <parent link="chassis"/>
-    <child link="sonar_02"/>
-    <origin xyz="0.07211 0.0248 0.044" rpy="0 0 0.3927" />
-  </joint>
-<!--
-########################################################################################
-Modelagem do sonar 03 "link" "joint"
-########################################################################################
--->
-  <link name="sonar_03">
-    <visual>
-      <origin xyz="-0.014 0.01 0" rpy="-1.571 1.571 -1.571" />
-      <geometry>
-	      <mesh filename="package://littlebot_description/meshes/sonar.dae" />
-      </geometry>
-    </visual>
-    <collision>
-      <origin xyz="-0.014 0.01 0" rpy="-1.571 1.571 -1.571" />
-      <geometry>
-	      <mesh filename="package://littlebot_description/meshes/sonar.dae" />
-      </geometry>
-    </collision>
-    <inertial>
-      <origin xyz="-0.014 0.01 0" rpy="-1.571 1.571 -1.571"/>
-      <mass value="0.015"/>
-      <inertia ixx="5.706e-7"  ixy="6.307e-9"  ixz="2.156e-9" iyy="2.771e-6" iyz="7.710e-9" izz="2.878e-6" />
-    </inertial>
-  </link>
-  <joint name="base_to_sonar_03" type="fixed">
-    <parent link="chassis"/>
-    <child link="sonar_03"/>
-    <origin xyz="0.06522 0.038787 0.044" rpy="0 0 0.7854" />
-  </joint>
-  <!--
-########################################################################################
-Modelagem do sonar 04 "link" "joint"
-########################################################################################
--->
-  <link name="sonar_04">
-    <visual>
-      <origin xyz="-0.014 0 0" rpy="-1.571 1.571 -1.571" />
-      <geometry>
-	      <mesh filename="package://littlebot_description/meshes/sonar.dae" />
-      </geometry>
-    </visual>
-    <collision>
-      <origin xyz="-0.014 0 0" rpy="-1.571 1.571 -1.571" />
-      <geometry>
-	      <mesh filename="package://littlebot_description/meshes/sonar.dae" />
-      </geometry>
-    </collision>
-    <inertial>
-      <origin xyz="-0.014 0 0" rpy="-1.571 1.571 -1.571"/>
-      <mass value="0.015"/>
-      <inertia ixx="5.706e-7"  ixy="6.307e-9"  ixz="2.156e-9" iyy="2.771e-6" iyz="7.710e-9" izz="2.878e-6" />
-    </inertial>
-  </link>
-  <joint name="base_to_sonar_04" type="fixed">
-    <parent link="chassis"/>
-    <child link="sonar_04"/>
-    <origin xyz="0.07211 -0.0248 0.044" rpy="0 0 -0.3927" />
-  </joint>
-<!--
-########################################################################################
-Modelagem do sonar 05 "link" "joint"
-########################################################################################
--->
-  <link name="sonar_05">
-    <visual>
-      <origin xyz="-0.014 0.01 0" rpy="-1.571 1.571 -1.571" />
-      <geometry>
-	      <mesh filename="package://littlebot_description/meshes/sonar.dae" />
-      </geometry>
-    </visual>
-    <collision>
-      <origin xyz="-0.014 0.01 0" rpy="-1.571 1.571 -1.571" />
-      <geometry>
-	      <mesh filename="package://littlebot_description/meshes/sonar.dae" />
-      </geometry>
-    </collision>
-    <inertial>
-      <origin xyz="-0.014 0.01 0" rpy="-1.571 1.571 -1.571"/>
-      <mass value="0.015"/>
-      <inertia ixx="5.706e-7"  ixy="6.307e-9"  ixz="2.156e-9" iyy="2.771e-6" iyz="7.710e-9" izz="2.878e-6" />
-    </inertial>
-  </link>
-  <joint name="base_to_sonar_05" type="fixed">
-    <parent link="chassis"/>
-    <child link="sonar_05"/>
-    <origin xyz="0.050935 -0.052781 0.044" rpy="0 0 -0.7854" />
-  </joint>
-<!--
-********************************************************************************************
-Transmission para as rodas
-********************************************************************************************
--->
   <transmission name="trans_caster" >
     <type>transmission_interface/SimpleTransmission</type>
@@ -371,4 +140,42 @@
     </actuator>
   </transmission>
+  <gazebo reference="caster_wheel">
+    <mu1 value="1.0"/>
+    <mu2 value="1.0"/>
+    <kp  value="10000.0" />
+    <kd  value="1.0" />
+    <fdir1 value="1 0 0"/>
+    <turnGravityOff>false</turnGravityOff>
+  </gazebo>
+<!--
+########################################################################################
+Modelagem da rodinha-Wheel "link" "joint"
+########################################################################################
+-->
+  <link name="wheel">
+    <visual>
+      <origin xyz="0 0 0" rpy="3.14 0 1.571" />
+      <geometry>
+	      <mesh filename="package://littlebot_description/meshes/Wheel.dae" />
+      </geometry>
+    </visual>
+    <collision>
+      <origin xyz="0 0 0" rpy="3.14 0 1.571" />
+      <geometry>
+	      <mesh filename="package://littlebot_description/meshes/Wheel.dae" />
+      </geometry>
+    </collision>
+    <inertial>
+      <origin xyz="0 0 0" rpy="3.14 0 1.571"/>
+      <mass value="0.007"/>
+      <inertia ixx="3.569e-7"  ixy="0.000e+0"  ixz="0.000e+0" iyy="5.344e-7" iyz="0.000e+0" izz="3.569e-7" />
+    </inertial>
+  </link>
+  <joint name="caster_wheel_to_wheel" type="continuous">
+    <parent link="caster_wheel"/>
+    <child link="wheel"/>
+    <origin xyz="0.0 0.0148 -0.0153" rpy="0 0 0" />
+    <axis xyz="1 0 0" />
+  </joint>
   <transmission name="trans_wheel" >
     <type>transmission_interface/SimpleTransmission</type>
@@ -380,4 +187,70 @@
     </actuator>
   </transmission>
+  <gazebo reference="wheel">
+    <mu1 value="100000.0"/>
+    <mu2 value="100.0"/>
+    <kp  value="10000000.0" />
+    <kd  value="1.0" />
+    <fdir1 value="1 0 0"/>
+    <turnGravityOff>false</turnGravityOff>
+  </gazebo>
+<!--
+########################################################################################
+Modelagem do motor esquerdo "link" "joint"
+########################################################################################
+-->
+  <link name="motor_esquerdo">
+    <visual>
+      <origin xyz="0 0 0" rpy="0 0 0" />
+      <geometry>
+	      <mesh filename="package://littlebot_description/meshes/motor.dae" />
+      </geometry>
+    </visual>
+    <collision>
+      <origin xyz="0 0 0" rpy="0 0 0" />
+      <geometry>
+	      <mesh filename="package://littlebot_description/meshes/motor.dae" />
+      </geometry>
+    </collision>
+    <inertial>
+      <origin xyz="0 0 0" rpy="0 0 0"/>
+      <mass value="0.09"/>
+      <inertia ixx="0"  ixy="0"  ixz="0" iyy="0" iyz="0" izz="0" />
+    </inertial>
+  </link>
+  <joint name="base_to_motor_esquerdo" type="fixed">
+    <parent link="chassis"/>
+    <child link="motor_esquerdo"/>
+    <origin xyz="-0.032 0.0412 -0.014" rpy="0 0 0" />
+  </joint>
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
Commit message: Ajustar macros das rodas para posicionar as meshs

File: littlebot_description/urdf/littlebot.xacro (robot description, xacro)
@@ -1,4 +1,4 @@
 <?xml version="1.0"?>
-<robot name="littlebot" xmlns:xacro="http://www.ros.org/wiki/xacro">
+<robot name="littlebot" xmlns:xacro="http://ros.org/wiki/xacro">
   <!-- Included URDF/XACRO Files -->
   <xacro:include filename="$(find littlebot_description)/urdf/rodas.xacro" />
@@ -48,7 +48,9 @@
   <xacro:littlebot_wheel lado_roda="esquerda">
     <origin xyz="0.005 0.07393 -0.014" rpy="0 0 1.571" />
+    <origin xyz="-0.012 0 0" rpy="0 0 0"/>
   </xacro:littlebot_wheel>
   <xacro:littlebot_wheel lado_roda="direita">
-    <origin xyz="0.005 -0.07393 -0.014" rpy="0 0 -1.571" />
+    <origin xyz="0.005 -0.07393 -0.014" rpy="0 0 1.571" />
+    <origin xyz="0.012 0 0" rpy="0 0 3.142"/>
   </xacro:littlebot_wheel>
 <!--

File: littlebot_description/urdf/rodas.xacro (robot description, xacro)
@@ -1,8 +1,8 @@
 <?xml version="1.0"?>
 <robot name="littlebot_wheel" xmlns:xacro="http://ros.org/wiki/xacro" >
-	<xacro:macro name="littlebot_wheel" params="lado_roda *joint_pose">
+	<xacro:macro name="littlebot_wheel" params="lado_roda *joint_pose *mesh_pose">
 		<link name="roda_${lado_roda}">
 			<visual>
-				<origin xyz="-0.01 0 0" rpy="0 0 0" />
+				<xacro:insert_block name="mesh_pose"/>
 				<geometry>
 					<mesh filename="package://littlebot_description/meshes/roda.dae" />
@@ -10,5 +10,5 @@
 			</visual>
 			<collision>
-				<origin xyz="-0.01 0 0" rpy="0 0 0" />
+				<xacro:insert_block name="mesh_pose"/>
 				<geometry>
 					<mesh filename="package://littlebot_description/meshes/roda.dae" />
@@ -16,5 +16,5 @@
 			</collision>
 			<inertial>
-        		<origin xyz="-0.01 0 0" rpy="0 0 0"/>
+				<xacro:insert_block name="mesh_pose"/>
 				<mass value="0.041"/>
 				<inertia ixx="2.967e-5"  ixy="-7.675e-15"  ixz="-4.765e-14" iyy="1.616e-5" iyz="-1.121e-16" izz="1.616e-5" />

Commit message: Ajuste na macro das rodas

File: littlebot_description/urdf/littlebot.xacro (robot description, xacro)
@@ -47,10 +47,10 @@
 -->
   <xacro:littlebot_wheel lado_roda="esquerda">
+    <origin xyz="-0.012 0 0" rpy="0 0 0"/>
     <origin xyz="0.005 0.07393 -0.014" rpy="0 0 1.571" />
-    <origin xyz="-0.012 0 0" rpy="0 0 0"/>
   </xacro:littlebot_wheel>
   <xacro:littlebot_wheel lado_roda="direita">
+    <origin xyz="0.012 0 0" rpy="0 0 3.142"/>
     <origin xyz="0.005 -0.07393 -0.014" rpy="0 0 1.571" />
-    <origin xyz="0.012 0 0" rpy="0 0 3.142"/>
   </xacro:littlebot_wheel>
 <!--

File: littlebot_description/urdf/rodas.xacro (robot description, xacro)
@@ -1,5 +1,5 @@
 <?xml version="1.0"?>
 <robot name="littlebot_wheel" xmlns:xacro="http://ros.org/wiki/xacro" >
-	<xacro:macro name="littlebot_wheel" params="lado_roda *joint_pose *mesh_pose">
+	<xacro:macro name="littlebot_wheel" params="lado_roda *mesh_pose *joint_pose">
 		<link name="roda_${lado_roda}">
 			<visual>
@@ -21,11 +21,4 @@
 			</inertial>
 		</link>
-		<gazebo reference="roda_${lado_roda}">
-			<mu1 value="1.0"/>
-			<mu2 value="1.0"/>
-			<kp value="10000000.0" />
-			<kd value="1.0" />
-			<fdir1 value="1 0 0"/>
-		</gazebo>
 		<joint name="base_to_roda_${lado_roda}" type="continuous">
 			<parent link="chassis"/>
@@ -43,4 +36,11 @@
 			</actuator>
 		</transmission>
+		<gazebo reference="roda_${lado_roda}">
+			<mu1 value="1.0"/>
+			<mu2 value="1.0"/>
+			<kp value="10000000.0" />
+			<kd value="1.0" />
+			<fdir1 value="1 0 0"/>
+		</gazebo>
 	</xacro:macro>
 </robot>
