Commit message: Incluir motor na macro das rodas

File: littlebot_description/urdf/littlebot.xacro (robot description, xacro)
@@ -1,7 +1,7 @@
 <?xml version="1.0"?>
 <robot name="littlebot" xmlns:xacro="http://ros.org/wiki/xacro">
-  <!-- Included URDF/XACRO Files -->
-  <xacro:include filename="$(find littlebot_description)/urdf/rodas.xacro" />
-  <xacro:include filename="$(find littlebot_description)/urdf/sonar.xacro" />
+<!-- Included URDF/XACRO Files -->
+<xacro:include filename="$(find littlebot_description)/urdf/rodas.xacro" />
+<xacro:include filename="$(find littlebot_description)/urdf/sonar.xacro" />
  <!--
 ########################################################################################
@@ -49,8 +49,10 @@
     <origin xyz="-0.012 0 0" rpy="0 0 0"/>
     <origin xyz="0.005 0.07393 -0.014" rpy="0 0 1.571" />
+    <origin xyz="-0.032 0.0412 -0.014" rpy="0 0 0" />
   </xacro:littlebot_wheel>
   <xacro:littlebot_wheel lado_roda="direita">
     <origin xyz="0.012 0 0" rpy="0 0 3.142"/>
     <origin xyz="0.005 -0.07393 -0.014" rpy="0 0 1.571" />
+    <origin xyz="-0.032 -0.0412 -0.014" rpy="0 0 0" />
   </xacro:littlebot_wheel>
 <!--
@@ -197,62 +199,4 @@
     <turnGravityOff>false</turnGravityOff>
   </gazebo>
-<!--
-########################################################################################
-Modelagem do motor esquerdo "link" "joint"
-########################################################################################
--->
-  <link name="motor_esquerdo">
-    <visual>
-      <origin xyz="0 0 0" rpy="0 0 0" />
-      <geometry>
-	      <mesh filename="package://littlebot_description/meshes/motor.dae" />
-      </geometry>
-    </visual>
-    <collision>
-      <origin xyz="0 0 0" rpy="0 0 0" />
-      <geometry>
-	      <mesh filename="package://littlebot_description/meshes/motor.dae" />
-      </geometry>
-    </collision>
-    <inertial>
-      <origin xyz="0 0 0" rpy="0 0 0"/>
-      <mass value="0.09"/>
-      <inertia ixx="0"  ixy="0"  ixz="0" iyy="0" iyz="0" izz="0" />
-    </inertial>
-  </link>
-  <joint name="base_to_motor_esquerdo" type="fixed">
-    <parent link="chassis"/>
-    <child link="motor_esquerdo"/>
-    <origin xyz="-0.032 0.0412 -0.014" rpy="0 0 0" />
-  </joint>
-<!--
-########################################################################################
-Modelagem do motor direito "link" "joint"
-########################################################################################
--->
-  <link name="motor_direito">
-    <visual>
-      <origin xyz="0 0 0" rpy="0 0 0" />
-      <geometry>
-	      <mesh filename="package://littlebot_description/meshes/motor.dae" />
-      </geometry>
-    </visual>
-    <collision>
-      <origin xyz="0 0 0" rpy="0 0 0" />
-      <geometry>
-	      <mesh filename="package://littlebot_description/meshes/motor.dae" />
-      </geometry>
-    </collision>
-    <inertial>
-      <origin xyz="0 0 0" rpy="0 0 0"/>
-      <mass value="0.09"/>
-      <inertia ixx="0"  ixy="0"  ixz="0" iyy="0" iyz="0" izz="0" />
-    </inertial>
-  </link>
-  <joint name="base_to_motor_direito" type="fixed">
-    <parent link="chassis"/>
-    <child link="motor_direito"/>
-    <origin xyz="-0.032 -0.0412 -0.014" rpy="0 0 0" />
-  </joint>
   <!--
   ******************************************************************************************
@@ -369,5 +313,5 @@
    </sensor>
   </gazebo>
-    <!--
+  <!--
   ******************************************************************************************
   SONAR03 gazebo plugin
@@ -411,5 +355,5 @@
    </sensor>
   </gazebo>
-    <!--
+  <!--
   ******************************************************************************************
   SONAR04 gazebo plugin

File: littlebot_description/urdf/rodas.xacro (robot description, xacro)
@@ -1,46 +1,80 @@
 <?xml version="1.0"?>
 <robot name="littlebot_wheel" xmlns:xacro="http://ros.org/wiki/xacro" >
-	<xacro:macro name="littlebot_wheel" params="lado_roda *mesh_pose *joint_pose">
-		<link name="roda_${lado_roda}">
-			<visual>
-				<xacro:insert_block name="mesh_pose"/>
-				<geometry>
-					<mesh filename="package://littlebot_description/meshes/roda.dae" />
-				</geometry>
-			</visual>
-			<collision>
-				<xacro:insert_block name="mesh_pose"/>
-				<geometry>
-					<mesh filename="package://littlebot_description/meshes/roda.dae" />
-				</geometry>
-			</collision>
-			<inertial>
-				<xacro:insert_block name="mesh_pose"/>
-				<mass value="0.041"/>
-				<inertia ixx="2.967e-5"  ixy="-7.675e-15"  ixz="-4.765e-14" iyy="1.616e-5" iyz="-1.121e-16" izz="1.616e-5" />
-			</inertial>
-		</link>
-		<joint name="base_to_roda_${lado_roda}" type="continuous">
-			<parent link="chassis"/>
-			<child link="roda_${lado_roda}"/>
-			<xacro:insert_block name="joint_pose"/>
-			<axis xyz="1 0 0" rpy="0 0 0" />
+<xacro:macro name="littlebot_wheel" params="lado_roda *mesh_pose *joint_roda_pose *joint_motor_pose">
+<!--
+########################################################################################
+Modelagem da roda "link" "joint" "transmission" "gazebo"
+########################################################################################
+-->
+	<link name="roda_${lado_roda}">
+		<visual>
+			<xacro:insert_block name="mesh_pose"/>
+			<geometry>
+				<mesh filename="package://littlebot_description/meshes/roda.dae" />
+			</geometry>
+		</visual>
+		<collision>
+			<xacro:insert_block name="mesh_pose"/>
+			<geometry>
+				<mesh filename="package://littlebot_description/meshes/roda.dae" />
+			</geometry>
+		</collision>
+		<inertial>
+			<xacro:insert_block name="mesh_pose"/>
+			<mass value="0.041"/>
+			<inertia ixx="2.967e-5"  ixy="-7.675e-15"  ixz="-4.765e-14" iyy="1.616e-5" iyz="-1.121e-16" izz="1.616e-5" />
+		</inertial>
+	</link>
+	<joint name="base_to_roda_${lado_roda}" type="continuous">
+		<parent link="chassis"/>
+		<child link="roda_${lado_roda}"/>
+		<xacro:insert_block name="joint_roda_pose"/>
+		<axis xyz="1 0 0" rpy="0 0 0" />
+	</joint>
+	<transmission name="trans_roda_${lado_roda}">
+		<type>transmission_interface/SimpleTransmission</type>
+		<joint name="base_to_roda_${lado_roda}">
+			<hardwareInterface>hardware_interface/VelocityJointInterface</hardwareInterface>
 		</joint>
-		<transmission name="trans_roda_${lado_roda}">
-			<type>transmission_interface/SimpleTransmission</type>
-			<joint name="base_to_roda_${lado_roda}">
-				<hardwareInterface>hardware_interface/VelocityJointInterface</hardwareInterface>
-			</joint>
-			<actuator name="roda_${lado_roda}_motor">
-				<mechanicalReduction>1</mechanicalReduction>
-			</actuator>
-		</transmission>
-		<gazebo reference="roda_${lado_roda}">
-			<mu1 value="1.0"/>
-			<mu2 value="1.0"/>
-			<kp value="10000000.0" />
-			<kd value="1.0" />
-			<fdir1 value="1 0 0"/>
-		</gazebo>
-	</xacro:macro>
+		<actuator name="roda_${lado_roda}_motor">
+			<mechanicalReduction>1</mechanicalReduction>
+		</actuator>
+	</transmission>
+	<gazebo reference="roda_${lado_roda}">
+		<mu1 value="1.0"/>
+		<mu2 value="1.0"/>
+		<kp value="10000000.0" />
+		<kd value="1.0" />
+		<fdir1 value="1 0 0"/>
+	</gazebo>
+<!--
+########################################################################################
+Modelagem da roda direita "link" "joint"
+########################################################################################
+-->
+	<link name="motor_${lado_roda}">
+		<visual>
+			<origin xyz="0 0 0" rpy="0 0 0" />
+			<geometry>
+				<mesh filename="package://littlebot_description/meshes/motor.dae" />
+			</geometry>
+		</visual>
+		<collision>
+			<origin xyz="0 0 0" rpy="0 0 0" />
+			<geometry>
+				<mesh filename="package://littlebot_description/meshes/motor.dae" />
+			</geometry>
+		</collision>
+		<inertial>
+			<origin xyz="0 0 0" rpy="0 0 0"/>
+			<mass value="0.09"/>
+			<inertia ixx="0"  ixy="0"  ixz="0" iyy="0" iyz="0" izz="0" />
+		</inertial>
+	</link>
+	<joint name="base_to_motor_${lado_roda}" type="fixed">
+		<parent link="chassis"/>
+		<child link="motor_${lado_roda}"/>
+		<xacro:insert_block name="joint_motor_pose"/>
+	</joint>
+</xacro:macro>
 </robot>

Commit message: arrumar sonar em forma crescente esquerda->direita

File: littlebot_description/urdf/littlebot.xacro (robot description, xacro)
@@ -62,5 +62,5 @@
 -->
   <xacro:littlebot_sonar sonar_numero="1">
-    <origin xyz="0.077 0.0 0.044" rpy="0 0 0" />
+    <origin xyz="0.06522 0.038787 0.044" rpy="0 0 0.7854" />
   </xacro:littlebot_sonar>
   <xacro:littlebot_sonar sonar_numero="2">
@@ -68,5 +68,5 @@
   </xacro:littlebot_sonar>
   <xacro:littlebot_sonar sonar_numero="3">
-    <origin xyz="0.06522 0.038787 0.044" rpy="0 0 0.7854" />
+    <origin xyz="0.077 0.0 0.044" rpy="0 0 0" />
   </xacro:littlebot_sonar>
   <xacro:littlebot_sonar sonar_numero="4">
@@ -234,4 +234,88 @@
   ******************************************************************************************
   -->
+  <gazebo reference="sonar_3">
+   <sensor type="ray" name="TeraRanger">
+      <pose>0 0 0 0 0 0</pose>
+      <visualize>false</visualize>
+      <update_rate>50</update_rate>
+      <ray>
+         <scan>
+            <horizontal>
+               <samples>10</samples>
+               <resolution>1</resolution>
+               <min_angle>-0.14835</min_angle>
+               <max_angle>0.14835</max_angle>
+            </horizontal>
+            <vertical>
+               <samples>10</samples>
+               <resolution>1</resolution>
+               <min_angle>-0.14835</min_angle>
+               <max_angle>0.14835</max_angle>
+            </vertical>
+         </scan>
+         <range>
+            <min>0.01</min>
+            <max>2</max>
+            <resolution>0.02</resolution>
+         </range>
+      </ray>
+      <plugin filename="libgazebo_ros_range.so" name="gazebo_ros_range">
+         <gaussianNoise>0.005</gaussianNoise>
+         <alwaysOn>true</alwaysOn>
+         <updateRate>50</updateRate>
+         <topicName>sensor/sonar3</topicName>
+         <frameName>sonar_3</frameName>
+         <radiation>ULTRASOUND</radiation>
+         <fov>0.2967</fov>
+      </plugin>
+   </sensor>
+  </gazebo>
+  <!--
+  ******************************************************************************************
+  SONAR02 gazebo plugin
+  ******************************************************************************************
+  -->
+  <gazebo reference="sonar_2">
+   <sensor type="ray" name="TeraRanger">
+      <pose>0 0 0 0 0 0</pose>
+      <visualize>false</visualize>
+      <update_rate>50</update_rate>
+      <ray>
+         <scan>
+            <horizontal>
+               <samples>10</samples>
+               <resolution>1</resolution>
+               <min_angle>-0.14835</min_angle>
+               <max_angle>0.14835</max_angle>
+            </horizontal>
+            <vertical>
+               <samples>10</samples>
+               <resolution>1</resolution>
+               <min_angle>-0.14835</min_angle>
+               <max_angle>0.14835</max_angle>
+            </vertical>
+         </scan>
+         <range>
+            <min>0.01</min>
+            <max>2</max>
+            <resolution>0.02</resolution>
+         </range>
+      </ray>
+      <plugin filename="libgazebo_ros_range.so" name="gazebo_ros_range">
+         <gaussianNoise>0.005</gaussianNoise>
+         <alwaysOn>true</alwaysOn>
+         <updateRate>50</updateRate>
+         <topicName>sensor/sonar2</topicName>
+         <frameName>sonar_2</frameName>
+         <radiation>ULTRASOUND</radiation>
+         <fov>0.2967</fov>
+      </plugin>
+   </sensor>
+  </gazebo>
+  <!--
+  ******************************************************************************************
+  SONAR03 gazebo plugin
+  ******************************************************************************************
+  -->
   <gazebo reference="sonar_1">
    <sensor type="ray" name="TeraRanger">
@@ -273,88 +357,4 @@
   <!--
   ******************************************************************************************
-  SONAR02 gazebo plugin
-  ******************************************************************************************
-  -->
-  <gazebo reference="sonar_2">
-   <sensor type="ray" name="TeraRanger">
-      <pose>0 0 0 0 0 0</pose>
-      <visualize>false</visualize>
-      <update_rate>50</update_rate>
-      <ray>
-         <scan>
-            <horizontal>
-               <samples>10</samples>
-               <resolution>1</resolution>
-               <min_angle>-0.14835</min_angle>
-               <max_angle>0.14835</max_angle>
-            </horizontal>
-            <vertical>
-               <samples>10</samples>
-               <resolution>1</resolution>
-               <min_angle>-0.14835</min_angle>
-               <max_angle>0.14835</max_angle>
-            </vertical>
-         </scan>
-         <range>
-            <min>0.01</min>
-            <max>2</max>
-            <resolution>0.02</resolution>
-         </range>
-      </ray>
-      <plugin filename="libgazebo_ros_range.so" name="gazebo_ros_range">
-         <gaussianNoise>0.005</gaussianNoise>
-         <alwaysOn>true</alwaysOn>
-         <updateRate>50</updateRate>
-         <topicName>sensor/sonar2</topicName>
-         <frameName>sonar_2</frameName>
-         <radiation>ULTRASOUND</radiation>
-         <fov>0.2967</fov>
-      </plugin>
-   </sensor>
-  </gazebo>
-  <!--
-  ******************************************************************************************
-  SONAR03 gazebo plugin
-  ******************************************************************************************
-  -->
-  <gazebo reference="sonar_3">
-   <sensor type="ray" name="TeraRanger">
-      <pose>0 0 0 0 0 0</pose>
-      <visualize>false</visualize>
-      <update_rate>50</update_rate>
-      <ray>
-         <scan>
-            <horizontal>
-               <samples>10</samples>
-               <resolution>1</resolution>
-               <min_angle>-0.14835</min_angle>
-               <max_angle>0.14835</max_angle>
-            </horizontal>
-            <vertical>
-               <samples>10</samples>
-               <resolution>1</resolution>
-               <min_angle>-0.14835</min_angle>
-               <max_angle>0.14835</max_angle>
-            </vertical>
-         </scan>
-         <range>
-            <min>0.01</min>
-            <max>2</max>
-            <resolution>0.02</resolution>
-         </range>
-      </ray>
-      <plugin filename="libgazebo_ros_range.so" name="gazebo_ros_range">
-         <gaussianNoise>0.005</gaussianNoise>
-         <alwaysOn>true</alwaysOn>
-         <updateRate>50</updateRate>
-         <topicName>sensor/sonar3</topicName>
-         <frameName>sonar_3</frameName>
-         <radiation>ULTRASOUND</radiation>
-         <fov>0.2967</fov>
-      </plugin>
-   </sensor>
-  </gazebo>
-  <!--
-  ******************************************************************************************
   SONAR04 gazebo plugin
   ******************************************************************************************

Commit message: ajustar posicionamento dos sonars

File: littlebot_description/urdf/littlebot.xacro (robot description, xacro)
@@ -62,5 +62,5 @@
 -->
   <xacro:littlebot_sonar sonar_numero="1">
-    <origin xyz="0.06522 0.038787 0.044" rpy="0 0 0.7854" />
+    <origin xyz="0.05822 0.045787 0.044" rpy="0 0 0.7854" />
   </xacro:littlebot_sonar>
   <xacro:littlebot_sonar sonar_numero="2">
@@ -74,5 +74,5 @@
   </xacro:littlebot_sonar>
   <xacro:littlebot_sonar sonar_numero="5">
-    <origin xyz="0.050935 -0.052781 0.044" rpy="0 0 -0.7854"/>
+    <origin xyz="0.05822 -0.045787 0.044" rpy="0 0 -0.7854"/>
   </xacro:littlebot_sonar>
 <!--

Commit message: Aumentar altura do sonar em relação ao chassis

File: littlebot_description/urdf/littlebot.xacro (robot description, xacro)
@@ -62,17 +62,17 @@
 -->
   <xacro:littlebot_sonar sonar_numero="1">
-    <origin xyz="0.05822 0.045787 0.044" rpy="0 0 0.7854" />
+    <origin xyz="0.05822 0.045787 0.064" rpy="0 0 0.7854" />
   </xacro:littlebot_sonar>
   <xacro:littlebot_sonar sonar_numero="2">
-    <origin xyz="0.07211 0.0248 0.044" rpy="0 0 0.3927"/>
+    <origin xyz="0.07211 0.0248 0.064" rpy="0 0 0.3927"/>
   </xacro:littlebot_sonar>
   <xacro:littlebot_sonar sonar_numero="3">
-    <origin xyz="0.077 0.0 0.044" rpy="0 0 0" />
+    <origin xyz="0.077 0.0 0.064" rpy="0 0 0" />
   </xacro:littlebot_sonar>
   <xacro:littlebot_sonar sonar_numero="4">
-    <origin xyz="0.07211 -0.0248 0.044" rpy="0 0 -0.3927"/>
+    <origin xyz="0.07211 -0.0248 0.064" rpy="0 0 -0.3927"/>
   </xacro:littlebot_sonar>
   <xacro:littlebot_sonar sonar_numero="5">
-    <origin xyz="0.05822 -0.045787 0.044" rpy="0 0 -0.7854"/>
+    <origin xyz="0.05822 -0.045787 0.064" rpy="0 0 -0.7854"/>
   </xacro:littlebot_sonar>
 <!--
