Commit message: add cc-cc converters and L298 driver meshs

File: littlebot_description/urdf/littlebot.xacro (robot description, xacro)
@@ -18,17 +18,17 @@
  <link name="chassis">
     <visual>
-      <origin xyz="0 0 0" rpy="1.571 0 1.571" />
-      <geometry>
-	      <mesh filename="package://littlebot_description/meshes/chassis2.dae" />
-      </geometry>
-    </visual>
-    <collision>
-      <origin xyz="0 0 0" rpy="1.571 0 1.571" />
-      <geometry>
-	      <mesh filename="package://littlebot_description/meshes/chassis2.dae" />
-      </geometry>
-    </collision>
-    <inertial>
-      <origin xyz="0 0 0.15" rpy="1.571 0 1.571"/>
+      <origin xyz="0 0 0" rpy="0 0 0" />
+      <geometry>
+	      <mesh filename="package://littlebot_description/meshes/chassis.dae" />
+      </geometry>
+    </visual>
+    <collision>
+      <origin xyz="0 0 0" rpy="0 0 0" />
+      <geometry>
+	      <mesh filename="package://littlebot_description/meshes/chassis.dae" />
+      </geometry>
+    </collision>
+    <inertial>
+      <origin xyz="0 0 0.15" rpy="0 0 0"/>
       <mass value="0.058"/>
       <inertia ixx="1.429e-4"  ixy="2.778e-10"  ixz="1.773e-8" iyy="1.943e-4" iyz="-2.656e-7" izz="5.361e-5" />
@@ -58,8 +58,37 @@
 <!--
 ########################################################################################
+Modelagem do suporte do sonar "link" "joint"
+########################################################################################
+-->
+ <link name="suporte_sonar">
+    <visual>
+      <origin xyz="0 0 0" rpy="0 0 0" />
+      <geometry>
+	      <mesh filename="package://littlebot_description/meshes/suporte_sonar.dae" />
+      </geometry>
+    </visual>
+    <collision>
+      <origin xyz="0 0 0" rpy="0 0 0" />
+      <geometry>
+	      <mesh filename="package://littlebot_description/meshes/suporte_sonar.dae" />
+      </geometry>
+    </collision>
+    <inertial>
+      <origin xyz="0 0 0.15" rpy="0 0 0"/>
+      <mass value="0.058"/>
+      <inertia ixx="1.429e-4"  ixy="2.778e-10"  ixz="1.773e-8" iyy="1.943e-4" iyz="-2.656e-7" izz="5.361e-5" />
+    </inertial>
+  </link>
+  <joint name="chassis_to_suporte" type="fixed">
+    <parent link="chassis"/>
+    <child link="suporte_sonar"/>
+    <origin xyz="0.094 0.0 0.0" rpy="0 0 0" />
+    <axis xyz="0 1 0" />
+  </joint>
+<!--
+########################################################################################
 Modelagem do sonar "link" "joint"
 ########################################################################################
 -->
-<!--
   <xacro:littlebot_sonar sonar_numero="1">
     <origin xyz="0.05822 0.045787 0.064" rpy="0 0 0.7854" />
@@ -69,5 +98,5 @@
   </xacro:littlebot_sonar>
   <xacro:littlebot_sonar sonar_numero="3">
-    <origin xyz="0.077 0.0 0.064" rpy="0 0 0" />
+    <origin xyz="0.092279 0.0 0.004733" rpy="0 0 0" />
   </xacro:littlebot_sonar>
   <xacro:littlebot_sonar sonar_numero="4">
@@ -77,5 +106,91 @@
     <origin xyz="0.05822 -0.045787 0.064" rpy="0 0 -0.7854"/>
   </xacro:littlebot_sonar>
-  -->
+<!--
+########################################################################################
+Modelagem da conversor1 "link" "joint"
+########################################################################################
+-->
+  <link name="conversor1">
+    <visual>
+      <origin xyz="0 0 0" rpy="0 0 0" />
+      <geometry>
+	      <mesh filename="package://littlebot_description/meshes/CC-converter.dae" />
+      </geometry>
+    </visual>
+    <collision>
+      <origin xyz="0 0 0" rpy="3.14 0 1.571" />
+      <geometry>
+	      <mesh filename="package://littlebot_description/meshes/CC-converter.dae" />
+      </geometry>
+    </collision>
+    <inertial>
+      <origin xyz="0 0 0" rpy="3.14 0 1.571"/>
+      <mass value="0.01946206"/>
+      <inertia ixx="1.561e-6"  ixy="0.000e+0"  ixz="0.000e+0" iyy="1.944e-6" iyz="0.000e+0" izz="3.350e-6" />
+    </inertial>
+  </link>
+  <joint name="base_to_conversor1" type="fixed">
+    <parent link="chassis"/>
+    <child link="conversor1"/>
+    <origin xyz="-0.0285 -0.0185 0.00165" rpy="0 0 0" />
+  </joint>
+<!--
+########################################################################################
+Modelagem da conversor2 "link" "joint"
+########################################################################################
+-->
+  <link name="conversor2">
+    <visual>
+      <origin xyz="0 0 0" rpy="0 0 0" />
+      <geometry>
+	      <mesh filename="package://littlebot_description/meshes/CC-converter.dae" />
+      </geometry>
+    </visual>
+    <collision>
+      <origin xyz="0 0 0" rpy="3.14 0 1.571" />
+      <geometry>
+	      <mesh filename="package://littlebot_description/meshes/CC-converter.dae" />
+      </geometry>
+    </collision>
+    <inertial>
+      <origin xyz="0 0 0" rpy="3.14 0 1.571"/>
+      <mass value="0.01946206"/>
+      <inertia ixx="1.561e-6"  ixy="0.000e+0"  ixz="0.000e+0" iyy="1.944e-6" iyz="0.000e+0" izz="3.350e-6" />
+    </inertial>
+  </link>
+  <joint name="base_to_conversor2" type="fixed">
+    <parent link="chassis"/>
+    <child link="conversor2"/>
+    <origin xyz="-0.0285 -0.0445 0.00165" rpy="0 0 0" />
+  </joint>
+<!--
+########################################################################################
+Modelagem da pont_h "link" "joint"
+########################################################################################
+-->
+  <link name="pont_h">
+    <visual>
+      <origin xyz="0 0 0" rpy="0 0 0" />
+      <geometry>
+	      <mesh filename="package://littlebot_description/meshes/L298_Driver.dae" />
+      </geometry>
+    </visual>
+    <collision>
+      <origin xyz="0 0 0" rpy="3.14 0 1.571" />
+      <geometry>
+	      <mesh filename="package://littlebot_description/meshes/L298_Driver.dae" />
+      </geometry>
+    </collision>
+    <inertial>
+      <origin xyz="0 0 0" rpy="3.14 0 1.571"/>
+      <mass value="0.01946206"/>
+      <inertia ixx="1.561e-6"  ixy="0.000e+0"  ixz="0.000e+0" iyy="1.944e-6" iyz="0.000e+0" izz="3.350e-6" />
+    </inertial>
+  </link>
+  <joint name="base_to_pont_h" type="fixed">
+    <parent link="chassis"/>
+    <child link="pont_h"/>
+    <origin xyz="-0.0745 0.046 0.0015 " rpy="0 0 0" />
+  </joint>
 <!--
 ########################################################################################

File: littlebot_description/urdf/sonar.xacro (robot description, xacro)
@@ -4,17 +4,17 @@
         <link name="sonar_${sonar_numero}">
             <visual>
-                <origin xyz="-0.014 0 0" rpy="-1.571 1.571 -1.571" />
+                <origin xyz="0 0 0" rpy="0 0 0" />
                 <geometry>
-                    <mesh filename="package://littlebot_description/meshes/sonar.dae" />
+                    <mesh filename="package://littlebot_description/meshes/HC-SR04.dae" />
                 </geometry>
             </visual>
             <collision>
-                <origin xyz="-0.014 0 0" rpy="-1.571 1.571 -1.571" />
+                <origin xyz="0 0 0" rpy="0 0 0" />
                 <geometry>
-                    <mesh filename="package://littlebot_description/meshes/sonar.dae" />
+                    <mesh filename="package://littlebot_description/meshes/HC-SR04.dae" />
                 </geometry>
             </collision>
             <inertial>
-                <origin xyz="-0.014 0 0" rpy="-1.571 1.571 -1.571"/>
+                <origin xyz="0 0 0" rpy="0 0 0"/>
                 <mass value="0.015"/>
                 <inertia ixx="5.706e-7"  ixy="6.307e-9"  ixz="2.156e-9" iyy="2.771e-6" iyz="7.710e-9" izz="2.878e-6" />

Commit message: Add well mesh left

File: littlebot_description/urdf/littlebot.xacro (robot description, xacro)
@@ -47,12 +47,14 @@
 -->
   <xacro:littlebot_wheel lado_roda="esquerda">
-    <origin xyz="-0.012 0 0" rpy="0 0 0"/>
-    <origin xyz="0.005 0.07393 -0.014" rpy="0 0 1.571" />
-    <origin xyz="-0.032 0.0412 -0.014" rpy="0 0 0" />
+    <origin xyz="0.0 0 0" rpy="0 0 0"/>
+    <origin xyz="0.0263 0.055 -0.01425" rpy="0 0 0" />
+    <origin xyz="0.0 0.0 0.0" rpy="0 0 0" />
+    <origin xyz="0.0015 0.0479 -0.003" rpy="0 0 0" />
   </xacro:littlebot_wheel>
   <xacro:littlebot_wheel lado_roda="direita">
-    <origin xyz="0.012 0 0" rpy="0 0 3.142"/>
-    <origin xyz="0.005 -0.07393 -0.014" rpy="0 0 1.571" />
-    <origin xyz="-0.032 -0.0412 -0.014" rpy="0 0 0" />
+    <origin xyz="0 0 0" rpy="0 0 0"/>
+    <origin xyz="0.0263 -0.055 -0.01425" rpy="0 0 0" />
+    <origin xyz="0 -0.0178 -0.0225" rpy="3.142 0 0" />
+    <origin xyz="0.0015 -0.0301 -0.003" rpy="0 0 0" />
   </xacro:littlebot_wheel>
 <!--

File: littlebot_description/urdf/rodas.xacro (robot description, xacro)
@@ -1,5 +1,5 @@
 <?xml version="1.0"?>
 <robot name="littlebot_wheel" xmlns:xacro="http://ros.org/wiki/xacro" >
-<xacro:macro name="littlebot_wheel" params="lado_roda *mesh_pose *joint_roda_pose *joint_motor_pose">
+<xacro:macro name="littlebot_wheel" params="lado_roda *mesh_roda_pose *joint_roda_pose *mesh_motor_pose *joint_motor_pose">
 <!--
 ########################################################################################
@@ -9,5 +9,5 @@
 	<link name="roda_${lado_roda}">
 		<visual>
-			<xacro:insert_block name="mesh_pose"/>
+			<xacro:insert_block name="mesh_roda_pose"/>
 			<geometry>
 				<mesh filename="package://littlebot_description/meshes/roda.dae" />
@@ -15,5 +15,5 @@
 		</visual>
 		<collision>
-			<xacro:insert_block name="mesh_pose"/>
+			<xacro:insert_block name="mesh_roda_pose"/>
 			<geometry>
 				<mesh filename="package://littlebot_description/meshes/roda.dae" />
@@ -21,5 +21,5 @@
 		</collision>
 		<inertial>
-			<xacro:insert_block name="mesh_pose"/>
+			<xacro:insert_block name="mesh_roda_pose"/>
 			<mass value="0.041"/>
 			<inertia ixx="2.967e-5"  ixy="-7.675e-15"  ixz="-4.765e-14" iyy="1.616e-5" iyz="-1.121e-16" izz="1.616e-5" />
@@ -30,5 +30,5 @@
 		<child link="roda_${lado_roda}"/>
 		<xacro:insert_block name="joint_roda_pose"/>
-		<axis xyz="1 0 0" rpy="0 0 0" />
+		<axis xyz="0 1 0" rpy="0 0 0" />
 	</joint>
 	<transmission name="trans_roda_${lado_roda}">
@@ -50,10 +50,10 @@
 <!--
 ########################################################################################
-Modelagem da roda direita "link" "joint"
+Modelagem do motor direita "link" "joint"
 ########################################################################################
 -->
 	<link name="motor_${lado_roda}">
 		<visual>
-			<origin xyz="0 0 0" rpy="0 0 0" />
+			<xacro:insert_block name="mesh_motor_pose"/>
 			<geometry>
 				<mesh filename="package://littlebot_description/meshes/motor.dae" />
@@ -61,5 +61,5 @@
 		</visual>
 		<collision>
-			<origin xyz="0 0 0" rpy="0 0 0" />
+			<xacro:insert_block name="mesh_motor_pose"/>
 			<geometry>
 				<mesh filename="package://littlebot_description/meshes/motor.dae" />
@@ -67,5 +67,5 @@
 		</collision>
 		<inertial>
-			<origin xyz="0 0 0" rpy="0 0 0"/>
+			<xacro:insert_block name="mesh_motor_pose"/>>
 			<mass value="0.09"/>
 			<inertia ixx="0"  ixy="0"  ixz="0" iyy="0" iyz="0" izz="0" />

Commit message: add well mesh right

File: littlebot_description/urdf/littlebot.xacro (robot description, xacro)
@@ -53,5 +53,5 @@
   </xacro:littlebot_wheel>
   <xacro:littlebot_wheel lado_roda="direita">
-    <origin xyz="0 0 0" rpy="0 0 0"/>
+    <origin xyz="0 0 0" rpy="0 0 3.142"/>
     <origin xyz="0.0263 -0.055 -0.01425" rpy="0 0 0" />
     <origin xyz="0 -0.0178 -0.0225" rpy="3.142 0 0" />

Commit message: add meshe of the chassis with all fixed joints

File: littlebot_description/urdf/littlebot.xacro (robot description, xacro)
@@ -20,5 +20,6 @@
       <origin xyz="0 0 0" rpy="0 0 0" />
       <geometry>
-	      <mesh filename="package://littlebot_description/meshes/chassis.dae" />
+	      <!-- <mesh filename="package://littlebot_description/meshes/chassis.dae" /> -->
+        <mesh filename="package://littlebot_description/meshes/littlebot.dae" />
       </geometry>
     </visual>
@@ -49,12 +50,12 @@
     <origin xyz="0.0 0 0" rpy="0 0 0"/>
     <origin xyz="0.0263 0.055 -0.01425" rpy="0 0 0" />
-    <origin xyz="0.0 0.0 0.0" rpy="0 0 0" />
-    <origin xyz="0.0015 0.0479 -0.003" rpy="0 0 0" />
+    <!-- <origin xyz="0.0 0.0 0.0" rpy="0 0 0" />
+    <origin xyz="0.0015 0.0479 -0.003" rpy="0 0 0" /> -->
   </xacro:littlebot_wheel>
   <xacro:littlebot_wheel lado_roda="direita">
     <origin xyz="0 0 0" rpy="0 0 3.142"/>
     <origin xyz="0.0263 -0.055 -0.01425" rpy="0 0 0" />
-    <origin xyz="0 -0.0178 -0.0225" rpy="3.142 0 0" />
-    <origin xyz="0.0015 -0.0301 -0.003" rpy="0 0 0" />
+    <!-- <origin xyz="0 -0.0178 -0.0225" rpy="3.142 0 0" />
+    <origin xyz="0.0015 -0.0301 -0.003" rpy="0 0 0" /> -->
   </xacro:littlebot_wheel>
 <!--
@@ -63,5 +64,5 @@
 ########################################################################################
 -->
- <link name="suporte_sonar">
+ <!-- <link name="suporte_sonar">
     <visual>
       <origin xyz="0 0 0" rpy="0 0 0" />
@@ -87,5 +88,5 @@
     <origin xyz="0.094 0.0 0.0" rpy="0 0 0" />
     <axis xyz="0 1 0" />
-  </joint>
+  </joint> -->
 <!--
 ########################################################################################
@@ -113,5 +114,5 @@
 ########################################################################################
 -->
-  <link name="conversor1">
+  <!-- <link name="conversor1">
     <visual>
       <origin xyz="0 0 0" rpy="0 0 0" />
@@ -136,5 +137,5 @@
     <child link="conversor1"/>
     <origin xyz="-0.0285 -0.0185 0.00165" rpy="0 0 0" />
-  </joint>
+  </joint> -->
 <!--
 ########################################################################################
@@ -142,5 +143,5 @@
 ########################################################################################
 -->
-  <link name="conversor2">
+  <!-- <link name="conversor2">
     <visual>
       <origin xyz="0 0 0" rpy="0 0 0" />
@@ -165,5 +166,5 @@
     <child link="conversor2"/>
     <origin xyz="-0.0285 -0.0445 0.00165" rpy="0 0 0" />
-  </joint>
+  </joint> -->
 <!--
 ########################################################################################
@@ -171,5 +172,5 @@
 ########################################################################################
 -->
-  <link name="pont_h">
+  <!-- <link name="pont_h">
     <visual>
       <origin xyz="0 0 0" rpy="0 0 0" />
@@ -194,5 +195,5 @@
     <child link="pont_h"/>
     <origin xyz="-0.0745 0.046 0.0015 " rpy="0 0 0" />
-  </joint>
+  </joint> -->
 <!--
 ########################################################################################
@@ -200,5 +201,5 @@
 ########################################################################################
 -->
-  <link name="caster_mounting">
+  <!-- <link name="caster_mounting">
     <visual>
       <origin xyz="0 0 0" rpy="3.14 0 1.571" />
@@ -223,5 +224,5 @@
     <child link="caster_mounting"/>
     <origin xyz="-0.0753 0.0 -0.003" rpy="0 0 0" />
-  </joint>
+  </joint> -->
 <!--
 ########################################################################################
@@ -249,5 +250,6 @@
   </link>
   <joint name="caster_mounting_to_caster_wheel" type="continuous">
-    <parent link="caster_mounting"/>
+    <!-- <parent link="caster_mounting"/> -->
+    <parent link="chassis"/>
     <child link="caster_wheel"/>
     <origin xyz="-0.0 0.0 -0.00623" rpy="0 0 0" />

File: littlebot_description/urdf/rodas.xacro (robot description, xacro)
@@ -1,5 +1,6 @@
 <?xml version="1.0"?>
 <robot name="littlebot_wheel" xmlns:xacro="http://ros.org/wiki/xacro" >
-<xacro:macro name="littlebot_wheel" params="lado_roda *mesh_roda_pose *joint_roda_pose *mesh_motor_pose *joint_motor_pose">
+<!-- <xacro:macro name="littlebot_wheel" params="lado_roda *mesh_roda_pose *joint_roda_pose *mesh_motor_pose *joint_motor_pose"> -->
+<xacro:macro name="littlebot_wheel" params="lado_roda *mesh_roda_pose *joint_roda_pose">
 <!--
 ########################################################################################
@@ -53,5 +54,5 @@
 ########################################################################################
 -->
-	<link name="motor_${lado_roda}">
+	<!-- <link name="motor_${lado_roda}">
 		<visual>
 			<xacro:insert_block name="mesh_motor_pose"/>
@@ -76,5 +77,5 @@
 		<child link="motor_${lado_roda}"/>
 		<xacro:insert_block name="joint_motor_pose"/>
-	</joint>
+	</joint> -->
 </xacro:macro>
 </robot>

Commit message: finished cc-cc converter mesh, adjuste wheels positions

File: littlebot_description/urdf/littlebot.xacro (robot description, xacro)
@@ -49,5 +49,5 @@
   <xacro:littlebot_wheel lado_roda="esquerda">
     <origin xyz="0.0 0 0" rpy="0 0 0"/>
-    <origin xyz="0.0263 0.055 -0.01425" rpy="0 0 0" />
+    <origin xyz="0.0281 0.057 -0.01425" rpy="0 0 0" />
     <!-- <origin xyz="0.0 0.0 0.0" rpy="0 0 0" />
     <origin xyz="0.0015 0.0479 -0.003" rpy="0 0 0" /> -->
@@ -55,5 +55,5 @@
   <xacro:littlebot_wheel lado_roda="direita">
     <origin xyz="0 0 0" rpy="0 0 3.142"/>
-    <origin xyz="0.0263 -0.055 -0.01425" rpy="0 0 0" />
+    <origin xyz="0.0281 -0.057 -0.01425" rpy="0 0 0" />
     <!-- <origin xyz="0 -0.0178 -0.0225" rpy="3.142 0 0" />
     <origin xyz="0.0015 -0.0301 -0.003" rpy="0 0 0" /> -->

Commit message: correct position of all sonar meshes

File: littlebot_description/urdf/littlebot.xacro (robot description, xacro)
@@ -95,8 +95,8 @@
 -->
   <xacro:littlebot_sonar sonar_numero="1">
-    <origin xyz="0.05822 0.045787 0.064" rpy="0 0 0.7854" />
+    <origin xyz="0.07879836 0.03772198 0.004733" rpy="0 0 0.686455448" />
   </xacro:littlebot_sonar>
   <xacro:littlebot_sonar sonar_numero="2">
-    <origin xyz="0.07211 0.0248 0.064" rpy="0 0 0.3927"/>
+    <origin xyz="0.08880761 0.02002920 0.004733" rpy="0 0 0.343218997"/>
   </xacro:littlebot_sonar>
   <xacro:littlebot_sonar sonar_numero="3">
@@ -104,8 +104,8 @@
   </xacro:littlebot_sonar>
   <xacro:littlebot_sonar sonar_numero="4">
-    <origin xyz="0.07211 -0.0248 0.064" rpy="0 0 -0.3927"/>
+    <origin xyz="0.08880761 -0.02002920 0.004733" rpy="0 0 -0.343218997"/>
   </xacro:littlebot_sonar>
   <xacro:littlebot_sonar sonar_numero="5">
-    <origin xyz="0.05822 -0.045787 0.064" rpy="0 0 -0.7854"/>
+    <origin xyz="0.07879836 -0.03772198 0.004733" rpy="0 0 -0.686455448"/>
   </xacro:littlebot_sonar>
 <!--
@@ -253,5 +253,5 @@
     <parent link="chassis"/>
     <child link="caster_wheel"/>
-    <origin xyz="-0.0 0.0 -0.00623" rpy="0 0 0" />
+    <origin xyz="-0.087 0.0 -0.00623" rpy="0 0 0" />
     <axis xyz="0 0 1" />
   </joint>

Commit message: Adjust inertia of the chassis meshe

File: littlebot_description/urdf/littlebot.xacro (robot description, xacro)
@@ -31,7 +31,9 @@
     </collision>
     <inertial>
-      <origin xyz="0 0 0.15" rpy="0 0 0"/>
-      <mass value="0.058"/>
-      <inertia ixx="1.429e-4"  ixy="2.778e-10"  ixz="1.773e-8" iyy="1.943e-4" iyz="-2.656e-7" izz="5.361e-5" />
+      <origin xyz="0 0 0" rpy="1.571 0 1.571"/>
+      <!-- <mass value="0.058"/> -->
+      <mass value="0.19357368"/>
+      <!-- <inertia ixx="1.429e-4"  ixy="2.778e-10"  ixz="1.773e-8" iyy="1.943e-4" iyz="-2.656e-7" izz="5.361e-5" /> -->
+      <inertia ixx="1.84569610e-4"  ixy="-4.09475462e-6"  ixz="-2.91063667e-5" iyy="7.65700035e-4" iyz="2.32776537e-8" izz="9.00861891e-4" />
     </inertial>
   </link>
@@ -40,5 +42,4 @@
     <child link="chassis"/>
     <origin xyz="0.0 0.0 0.0" rpy="0 0 0" />
-    <axis xyz="0 1 0" />
   </joint>
 <!--
@@ -245,6 +246,6 @@
     <inertial>
       <origin xyz="0 0 0" rpy="3.14 0 1.571"/>
-      <mass value="0.00982010"/>
-      <inertia ixx="8.398e-7"  ixy="-1.517e-14"  ixz="-1.601e-7" iyy="8.400e-7" iyz="1.155e-14" izz="1.340e-6" />
+      <mass value="0.01290279"/>
+      <inertia ixx="1.23004519e-6"  ixy="-4.54832220e-14"  ixz="-4.88841255e-7" iyy="1.51454374e-6" iyz="-1.45133258e-14" izz="1.82945276e-6" />
     </inertial>
   </link>

Commit message: adjust ultrasonic sensor link position

File: littlebot_description/urdf/littlebot.xacro (robot description, xacro)
@@ -96,17 +96,22 @@
 -->
   <xacro:littlebot_sonar sonar_numero="1">
-    <origin xyz="0.07879836 0.03772198 0.004733" rpy="0 0 0.686455448" />
+    <origin xyz="0 0 -0.020267" rpy="0 0 0" />
+    <origin xyz="0.07879836 0.03772198 0.02500000" rpy="0 0 0.686455448" />
   </xacro:littlebot_sonar>
   <xacro:littlebot_sonar sonar_numero="2">
-    <origin xyz="0.08880761 0.02002920 0.004733" rpy="0 0 0.343218997"/>
+    <origin xyz="0 0 -0.020267" rpy="0 0 0" />
+    <origin xyz="0.08880761 0.02002920 0.02500000" rpy="0 0 0.343218997"/>
   </xacro:littlebot_sonar>
   <xacro:littlebot_sonar sonar_numero="3">
-    <origin xyz="0.092279 0.0 0.004733" rpy="0 0 0" />
+    <origin xyz="0 0 -0.020267" rpy="0 0 0" />
+    <origin xyz="0.092279 0.0 0.02500000" rpy="0 0 0" />
   </xacro:littlebot_sonar>
   <xacro:littlebot_sonar sonar_numero="4">
-    <origin xyz="0.08880761 -0.02002920 0.004733" rpy="0 0 -0.343218997"/>
+    <origin xyz="0 0 -0.020267" rpy="0 0 0" />
+    <origin xyz="0.08880761 -0.02002920 0.02500000" rpy="0 0 -0.343218997"/>
   </xacro:littlebot_sonar>
   <xacro:littlebot_sonar sonar_numero="5">
-    <origin xyz="0.07879836 -0.03772198 0.004733" rpy="0 0 -0.686455448"/>
+    <origin xyz="0 0 -0.020267" rpy="0 0 0" />
+    <origin xyz="0.07879836 -0.03772198 0.02500000" rpy="0 0 -0.686455448"/>
   </xacro:littlebot_sonar>
 <!--

File: littlebot_description/urdf/sonar.xacro (robot description, xacro)
@@ -1,8 +1,8 @@
 <?xml version="1.0"?>
 <robot name="littlebot_sonar" xmlns:xacro="http://ros.org/wiki/xacro" >
-	<xacro:macro name="littlebot_sonar" params="sonar_numero *joint_pose">
+	<xacro:macro name="littlebot_sonar" params="sonar_numero *meshe_pose *joint_pose">
         <link name="sonar_${sonar_numero}">
             <visual>
-                <origin xyz="0 0 0" rpy="0 0 0" />
+                <xacro:insert_block name="meshe_pose"/>
                 <geometry>
                     <mesh filename="package://littlebot_description/meshes/HC-SR04.dae" />
@@ -10,5 +10,5 @@
             </visual>
             <collision>
-                <origin xyz="0 0 0" rpy="0 0 0" />
+                <xacro:insert_block name="meshe_pose"/>
                 <geometry>
                     <mesh filename="package://littlebot_description/meshes/HC-SR04.dae" />
@@ -16,5 +16,5 @@
             </collision>
             <inertial>
-                <origin xyz="0 0 0" rpy="0 0 0"/>
+                <xacro:insert_block name="meshe_pose"/>
                 <mass value="0.015"/>
                 <inertia ixx="5.706e-7"  ixy="6.307e-9"  ixz="2.156e-9" iyy="2.771e-6" iyz="7.710e-9" izz="2.878e-6" />
