Commit message: adjust wheel link position

File: littlebot_description/urdf/littlebot.xacro (robot description, xacro)
@@ -50,5 +50,5 @@
   <xacro:littlebot_wheel lado_roda="esquerda">
     <origin xyz="0.0 0 0" rpy="0 0 0"/>
-    <origin xyz="0.0281 0.057 -0.01425" rpy="0 0 0" />
+    <origin xyz="0.0281 0.067 -0.01425" rpy="0 0 0" />
     <!-- <origin xyz="0.0 0.0 0.0" rpy="0 0 0" />
     <origin xyz="0.0015 0.0479 -0.003" rpy="0 0 0" /> -->
@@ -56,5 +56,5 @@
   <xacro:littlebot_wheel lado_roda="direita">
     <origin xyz="0 0 0" rpy="0 0 3.142"/>
-    <origin xyz="0.0281 -0.057 -0.01425" rpy="0 0 0" />
+    <origin xyz="0.0281 -0.067 -0.01425" rpy="0 0 0" />
     <!-- <origin xyz="0 -0.0178 -0.0225" rpy="3.142 0 0" />
     <origin xyz="0.0015 -0.0301 -0.003" rpy="0 0 0" /> -->

Commit message: add imu link in URDF file

File: littlebot_description/urdf/littlebot.xacro (robot description, xacro)
@@ -31,5 +31,5 @@
     </collision>
     <inertial>
-      <origin xyz="0 0 0" rpy="1.571 0 1.571"/>
+      <origin xyz="0 0 0" rpy="0 0 0"/>
       <!-- <mass value="0.058"/> -->
       <mass value="0.19357368"/>
@@ -115,4 +115,33 @@
     <origin xyz="0.07879836 -0.03772198 0.02500000" rpy="0 0 -0.686455448"/>
   </xacro:littlebot_sonar>
+ <!--
+########################################################################################
+Modelagem da IMU MPU-6050 "link" "joint"
+########################################################################################
+-->
+ <link name="imu_link">
+    <visual>
+      <origin xyz="0 0 0" rpy="0 0 0" />
+      <geometry>
+        <mesh filename="package://littlebot_description/meshes/MPU_6050.dae" />
+      </geometry>
+    </visual>
+    <collision>
+      <origin xyz="0 0 0" rpy="0 0 0" />
+      <geometry>
+	      <mesh filename="package://littlebot_description/meshes/MPU_6050.dae" />
+      </geometry>
+    </collision>
+    <inertial>
+      <origin xyz="0 0 0" rpy="0 0 0"/>
+      <mass value="0.00142672"/>
+      <inertia ixx="4.54052487e-8"  ixy="1.07305074e-10"  ixz="-2.17782593e-10" iyy="2.70451174e-8" iyz="-4.58999382e-11" izz="7.14041804e-8" />
+    </inertial>
+  </link>
+  <joint name="chassis_to_imu" type="fixed">
+    <parent link="chassis"/>
+    <child link="imu_link"/>
+    <origin xyz="0.028 0.0 0.005" rpy="0 0 0" />
+  </joint>
 <!--
 ########################################################################################
@@ -346,5 +375,5 @@
       <robotNamespace>/</robotNamespace>
       <updateRate>50.0</updateRate>
-      <bodyName>chassis</bodyName>
+      <bodyName>imu_link</bodyName>
       <topicName>imu/data</topicName>
       <accelDrift>0.005 0.005 0.005</accelDrift>

Commit message: use macro for sonars in littlebot.xacro

File: littlebot_description/urdf/littlebot.xacro (robot description, xacro)
@@ -231,44 +231,52 @@
   <!--
   ******************************************************************************************
+  SONAR_macro gazebo plugin
+  ******************************************************************************************
+  -->
+  <xacro:macro name="sonar" params="reference topic_name">
+    <gazebo reference="${reference}">
+      <sensor type="ray" name="TeraRanger">
+          <pose>0 0 0 0 0 0</pose>
+          <visualize>false</visualize>
+          <update_rate>50</update_rate>
+          <ray>
+            <scan>
+                <horizontal>
+                  <samples>10</samples>
+                  <resolution>1</resolution>
+                  <min_angle>-0.14835</min_angle>
+                  <max_angle>0.14835</max_angle>
+                </horizontal>
+                <vertical>
+                  <samples>10</samples>
+                  <resolution>1</resolution>
+                  <min_angle>-0.14835</min_angle>
+                  <max_angle>0.14835</max_angle>
+                </vertical>
+            </scan>
+            <range>
+                <min>0.01</min>
+                <max>2</max>
+                <resolution>0.02</resolution>
+            </range>
+          </ray>
+          <plugin filename="libgazebo_ros_range.so" name="gazebo_ros_range">
+            <gaussianNoise>0.005</gaussianNoise>
+            <alwaysOn>true</alwaysOn>
+            <updateRate>50</updateRate>
+            <topicName>sensor/${topic_name}</topicName>
+            <frameName>${reference}</frameName>
+            <radiation>ULTRASOUND</radiation>
+            <fov>0.2967</fov>
+          </plugin>
+        </sensor>
+      </gazebo>
+  </xacro:macro>
+  <!--
+  ******************************************************************************************
   SONAR_01 gazebo plugin
   ******************************************************************************************
   -->
-  <gazebo reference="sonar_3">
-   <sensor type="ray" name="TeraRanger">
-      <pose>0 0 0 0 0 0</pose>
-      <visualize>false</visualize>
-      <update_rate>50</update_rate>
-      <ray>
-         <scan>
-            <horizontal>
-               <samples>10</samples>
-               <resolution>1</resolution>
-               <min_angle>-0.14835</min_angle>
-               <max_angle>0.14835</max_angle>
-            </horizontal>
-            <vertical>
-               <samples>10</samples>
-               <resolution>1</resolution>
-               <min_angle>-0.14835</min_angle>
-               <max_angle>0.14835</max_angle>
-            </vertical>
-         </scan>
-         <range>
-            <min>0.01</min>
-            <max>2</max>
-            <resolution>0.02</resolution>
-         </range>
-      </ray>
-      <plugin filename="libgazebo_ros_range.so" name="gazebo_ros_range">
-         <gaussianNoise>0.005</gaussianNoise>
-         <alwaysOn>true</alwaysOn>
-         <updateRate>50</updateRate>
-         <topicName>sensor/sonar3</topicName>
-         <frameName>sonar_3</frameName>
-         <radiation>ULTRASOUND</radiation>
-         <fov>0.2967</fov>
-      </plugin>
-    </sensor>
-  </gazebo>
+  <xacro:sonar reference="sonar_1" topic_name="sonar1" />
   <!--
   ******************************************************************************************
@@ -276,41 +284,5 @@
   ******************************************************************************************
   -->
-  <gazebo reference="sonar_2">
-   <sensor type="ray" name="TeraRanger">
-      <pose>0 0 0 0 0 0</pose>
-      <visualize>false</visualize>
-      <update_rate>50</update_rate>
-      <ray>
-         <scan>
-            <horizontal>
-               <samples>10</samples>
-               <resolution>1</resolution>
-               <min_angle>-0.14835</min_angle>
-               <max_angle>0.14835</max_angle>
-            </horizontal>
-            <vertical>
-               <samples>10</samples>
-               <resolution>1</resolution>
-               <min_angle>-0.14835</min_angle>
-               <max_angle>0.14835</max_angle>
-            </vertical>
-         </scan>
-         <range>
-            <min>0.01</min>
-            <max>2</max>
-            <resolution>0.02</resolution>
-         </range>
-      </ray>
-      <plugin filename="libgazebo_ros_range.so" name="gazebo_ros_range">
-         <gaussianNoise>0.005</gaussianNoise>
-         <alwaysOn>true</alwaysOn>
-         <updateRate>50</updateRate>
-         <topicName>sensor/sonar2</topicName>
-         <frameName>sonar_2</frameName>
-         <radiation>ULTRASOUND</radiation>
-         <fov>0.2967</fov>
-      </plugin>
-   </sensor>
-  </gazebo>
+  <xacro:sonar reference="sonar_2" topic_name="sonar2" />
   <!--
   ******************************************************************************************
@@ -318,41 +290,5 @@
   ******************************************************************************************
   -->
-  <gazebo reference="sonar_1">
-   <sensor type="ray" name="TeraRanger">
-      <pose>0 0 0 0 0 0</pose>
-      <visualize>false</visualize>
-      <update_rate>50</update_rate>
-      <ray>
-         <scan>
-            <horizontal>
-               <samples>10</samples>
-               <resolution>1</resolution>
-               <min_angle>-0.14835</min_angle>
-               <max_angle>0.14835</max_angle>
-            </horizontal>
-            <vertical>
-               <samples>10</samples>
-               <resolution>1</resolution>
-               <min_angle>-0.14835</min_angle>
-               <max_angle>0.14835</max_angle>
-            </vertical>
-         </scan>
-         <range>
-            <min>0.01</min>
-            <max>2</max>
-            <resolution>0.02</resolution>
-         </range>
-      </ray>
-      <plugin filename="libgazebo_ros_range.so" name="gazebo_ros_range">
-         <gaussianNoise>0.005</gaussianNoise>
-         <alwaysOn>true</alwaysOn>
-         <updateRate>50</updateRate>
-         <topicName>sensor/sonar1</topicName>
-         <frameName>sonar_1</frameName>
-         <radiation>ULTRASOUND</radiation>
-         <fov>0.2967</fov>
-      </plugin>
-   </sensor>
-  </gazebo>
+  <xacro:sonar reference="sonar_3" topic_name="sonar3" />
   <!--
   ******************************************************************************************
@@ -360,41 +296,5 @@
   ******************************************************************************************
   -->
-  <gazebo reference="sonar_4">
-   <sensor type="ray" name="TeraRanger">
-      <pose>0 0 0 0 0 0</pose>
-      <visualize>false</visualize>
-      <update_rate>50</update_rate>
-      <ray>
-         <scan>
-            <horizontal>
-               <samples>10</samples>
-               <resolution>1</resolution>
-               <min_angle>-0.14835</min_angle>
-               <max_angle>0.14835</max_angle>
-            </horizontal>
-            <vertical>
-               <samples>10</samples>
-               <resolution>1</resolution>
-               <min_angle>-0.14835</min_angle>
-               <max_angle>0.14835</max_angle>
-            </vertical>
-         </scan>
-         <range>
-            <min>0.01</min>
-            <max>2</max>
-            <resolution>0.02</resolution>
-         </range>
-      </ray>
-      <plugin filename="libgazebo_ros_range.so" name="gazebo_ros_range">
-         <gaussianNoise>0.005</gaussianNoise>
-         <alwaysOn>false</alwaysOn>
-         <updateRate>50</updateRate>
-         <topicName>sensor/sonar4</topicName>
-         <frameName>sonar_4</frameName>
-         <radiation>ULTRASOUND</radiation>
-         <fov>0.2967</fov>
-      </plugin>
-   </sensor>
-  </gazebo>
+  <xacro:sonar reference="sonar_4" topic_name="sonar4" />
   <!--
   ******************************************************************************************
@@ -402,40 +302,4 @@
   ******************************************************************************************
   -->
-  <gazebo reference="sonar_5">
-   <sensor type="ray" name="TeraRanger">
-      <pose>0 0 0 0 0 0</pose>
-      <visualize>false</visualize>
-      <update_rate>50</update_rate>
-      <ray>
-         <scan>
-            <horizontal>
-               <samples>10</samples>
-               <resolution>1</resolution>
-               <min_angle>-0.14835</min_angle>
-               <max_angle>0.14835</max_angle>
-            </horizontal>
-            <vertical>
-               <samples>10</samples>
-               <resolution>1</resolution>
-               <min_angle>-0.14835</min_angle>
-               <max_angle>0.14835</max_angle>
-            </vertical>
-         </scan>
-         <range>
-            <min>0.01</min>
-            <max>2</max>
-            <resolution>0.02</resolution>
-         </range>
-      </ray>
-      <plugin filename="libgazebo_ros_range.so" name="gazebo_ros_range">
-         <gaussianNoise>0.005</gaussianNoise>
-         <alwaysOn>true</alwaysOn>
-         <updateRate>50</updateRate>
-         <topicName>sensor/sonar5</topicName>
-         <frameName>sonar_5</frameName>
-         <radiation>ULTRASOUND</radiation>
-         <fov>0.2967</fov>
-      </plugin>
-   </sensor>
-  </gazebo>
+  <xacro:sonar reference="sonar_5" topic_name="sonar5" />
 </robot>

Commit message: adjust caster_whell origin

File: littlebot_description/urdf/littlebot.xacro (robot description, xacro)
@@ -262,10 +262,11 @@
 <!--
 ########################################################################################
-Modelagem da rodinha-Caster Wheel Plate "link" "joint"
+Modelagem da rodinha-Caster Wheel Plate "link" "joint" "transmission"
 ########################################################################################
 -->
   <link name="caster_wheel">
     <visual>
-      <origin xyz="0 0 0" rpy="3.14 0 1.571" />
+      <!-- <origin xyz="0 0 0" rpy="3.14 0 1.571" /> -->
+      <origin xyz="0 0 0" rpy="3.14 0 0" />
       <geometry>
 	      <mesh filename="package://littlebot_description/meshes/Caster_Wheel_Plate.dae" />
@@ -273,5 +274,5 @@
     </visual>
     <collision>
-      <origin xyz="0 0 0" rpy="3.14 0 1.571" />
+      <origin xyz="0 0 0" rpy="3.14 0 0" />
       <geometry>
 	      <mesh filename="package://littlebot_description/meshes/Caster_Wheel_Plate.dae" />
@@ -279,5 +280,5 @@
     </collision>
     <inertial>
-      <origin xyz="0 0 0" rpy="3.14 0 1.571"/>
+      <origin xyz="0 0 0" rpy="3.14 0 0" />
       <mass value="0.01290279"/>
       <inertia ixx="1.23004519e-6"  ixy="-4.54832220e-14"  ixz="-4.88841255e-7" iyy="1.51454374e-6" iyz="-1.45133258e-14" izz="1.82945276e-6" />
@@ -288,5 +289,5 @@
     <parent link="chassis"/>
     <child link="caster_wheel"/>
-    <origin xyz="-0.087 0.0 -0.00623" rpy="0 0 0" />
+    <origin xyz="-0.087 0.0 -0.0092" rpy="0 0 0" />
     <axis xyz="0 0 1" />
   </joint>
@@ -310,10 +311,10 @@
 <!--
 ########################################################################################
-Modelagem da rodinha-Wheel "link" "joint"
+Modelagem da rodinha-Wheel "link" "joint" "transmission"
 ########################################################################################
 -->
   <link name="wheel">
     <visual>
-      <origin xyz="0 0 0" rpy="3.14 0 1.571" />
+      <origin xyz="0 0 0" rpy="0 0 0" />
       <geometry>
 	      <mesh filename="package://littlebot_description/meshes/Wheel.dae" />
@@ -321,5 +322,5 @@
     </visual>
     <collision>
-      <origin xyz="0 0 0" rpy="3.14 0 1.571" />
+      <origin xyz="0 0 0" rpy="0 0 0" />
       <geometry>
 	      <mesh filename="package://littlebot_description/meshes/Wheel.dae" />
@@ -327,5 +328,5 @@
     </collision>
     <inertial>
-      <origin xyz="0 0 0" rpy="3.14 0 1.571"/>
+      <origin xyz="0 0 0" rpy="0 0 0"/>
       <mass value="0.007"/>
       <inertia ixx="3.569e-7"  ixy="0.000e+0"  ixz="0.000e+0" iyy="5.344e-7" iyz="0.000e+0" izz="3.569e-7" />
@@ -335,6 +336,6 @@
     <parent link="caster_wheel"/>
     <child link="wheel"/>
-    <origin xyz="0.0 0.0148 -0.0153" rpy="0 0 0" />
-    <axis xyz="1 0 0" />
+    <origin xyz="0.0149 0 -0.0151" rpy="0 0 0" />
+    <axis xyz="0 1 0" />
   </joint>
   <transmission name="trans_wheel" >
