Commit message: add wheel in description file

File: littlebot_description/urdf/littlebot_description.urdf.xacro (robot description, xacro)
@@ -2,12 +2,12 @@
 <robot name="littlebot">
 <!-- Included URDF XACRO Files -->
-<!-- <xacro:include filename="$(find littlebot_description)/urdf/rodas.xacro" />
-<xacro:include filename="$(find littlebot_description)/urdf/sonar.xacro" /> -->
- <!--
-Modelagem base_link "link"
--->
- <link name="base_link">
- </link>
- <link name="chassis">
+<!-- <xacro:include filename="$(find littlebot_description)/urdf/littlebot_wheel.urdf.xacro" /> -->
+<!-- <xacro:include filename="$(find littlebot_description)/urdf/sonar.xacro" /> -->
+  <!-- Modelagem base_link "link" -->
+  <link name="base_link">
+  </link>
+  <!-- Modelagem chassis "link" and "joint"-->
+  <!-- ========================================================================== -->
+  <link name="chassis">
     <visual>
       <origin xyz="0 0 0" rpy="0 0 0" />
@@ -33,3 +33,57 @@
     <origin xyz="0.0 0.0 0.0" rpy="0 0 0" />
   </joint>
+  <!-- Left whell model "link" "joint" "transmission" "gazebo" -->
+  <!-- ========================================================================== -->
+	<link name="left_wheel">
+		<visual>
+			<origin xyz="0.0 0 0" rpy="0 0 0"/>
+			<geometry>
+				<mesh filename="package://littlebot_description/meshes/roda.dae" />
+			</geometry>
+		</visual>
+		<collision>
+			<origin xyz="0.0 0 0" rpy="0 0 0"/>
+			<geometry>
+				<mesh filename="package://littlebot_description/meshes/roda.dae" />
+			</geometry>
+		</collision>
+		<inertial>
+			<origin xyz="0.0 0 0" rpy="0 0 0"/>
+			<mass value="0.041"/>
+			<inertia ixx="2.967e-5"  ixy="-7.675e-15"  ixz="-4.765e-14" iyy="1.616e-5" iyz="-1.121e-16" izz="1.616e-5" />
+    	</inertial>
+	</link>
+	<joint name="base_to_left_wheel" type="continuous">
+		<parent link="chassis"/>
+		<child link="left_wheel"/>
+		<origin xyz="0.0281 0.067 -0.01425" rpy="0 0 0" />
+		<axis xyz="0 1 0" rpy="0 0 0" />
+	</joint>
+  <!-- Right wheel model "link" "joint" "transmission" "gazebo" -->
+  <!-- ========================================================================== -->
+	<link name="right_wheel">
+		<visual>
+			<origin xyz="0 0 0" rpy="0 0 3.142"/>
+			<geometry>
+				<mesh filename="package://littlebot_description/meshes/roda.dae" />
+			</geometry>
+		</visual>
+		<collision>
+			<origin xyz="0 0 0" rpy="0 0 3.142"/>
+			<geometry>
+				<mesh filename="package://littlebot_description/meshes/roda.dae" />
+			</geometry>
+		</collision>
+		<inertial>
+			<origin xyz="0 0 0" rpy="0 0 3.142"/>
+			<mass value="0.041"/>
+			<inertia ixx="2.967e-5"  ixy="-7.675e-15"  ixz="-4.765e-14" iyy="1.616e-5" iyz="-1.121e-16" izz="1.616e-5" />
+    	</inertial>
+	</link>
+	<joint name="base_to_right_wheel" type="continuous">
+		<parent link="chassis"/>
+		<child link="right_wheel"/>
+		<origin xyz="0.0281 -0.067 -0.01425" rpy="0 0 0" />
+		<axis xyz="0 1 0" rpy="0 0 0" />
+	</joint>
 </robot>

Commit message: create control package

File: littlebot_description/urdf/littlebot_description.urdf.xacro (robot description, xacro)
@@ -1,4 +1,4 @@
 <?xml version="1.0"?>
-<robot name="littlebot">
+<robot xmlns:xacro="http://ros.org/wiki/xacro"  name="littlebot">
 <!-- Included URDF XACRO Files -->
 <!-- <xacro:include filename="$(find littlebot_description)/urdf/littlebot_wheel.urdf.xacro" /> -->
@@ -13,5 +13,5 @@
       <origin xyz="0 0 0" rpy="0 0 0" />
       <geometry>
-        <mesh filename="package://littlebot_description/meshes/littlebot.dae" />
+        <mesh filename="/home/nestor/Documents/littlebot/littlebot_ws/src/littlebot/littlebot_description/meshes/littlebot.dae" />
       </geometry>
     </visual>
@@ -19,5 +19,5 @@
       <origin xyz="0 0 0" rpy="0 0 0" />
       <geometry>
-	      <mesh filename="package://littlebot_description/meshes/chassis.dae" />
+	      <mesh filename="/home/nestor/Documents/littlebot/littlebot_ws/src/littlebot/littlebot_description/meshes/chassis.dae" />
       </geometry>
     </collision>
@@ -39,5 +39,5 @@
 			<origin xyz="0.0 0 0" rpy="0 0 0"/>
 			<geometry>
-				<mesh filename="package://littlebot_description/meshes/roda.dae" />
+				<mesh filename="/home/nestor/Documents/littlebot/littlebot_ws/src/littlebot/littlebot_description/meshes/roda.dae" />
 			</geometry>
 		</visual>
@@ -45,5 +45,5 @@
 			<origin xyz="0.0 0 0" rpy="0 0 0"/>
 			<geometry>
-				<mesh filename="package://littlebot_description/meshes/roda.dae" />
+				<mesh filename="/home/nestor/Documents/littlebot/littlebot_ws/src/littlebot/littlebot_description/meshes/roda.dae" />
 			</geometry>
 		</collision>
@@ -60,4 +60,11 @@
 		<axis xyz="0 1 0" rpy="0 0 0" />
 	</joint>
+	<gazebo reference="left_wheel">
+      <mu1 value="1.0"/>
+      <mu2 value="0.5"/>
+      <kp value="10000000.0" />
+      <kd value="1.0" />
+      <fdir1 value="1 0 0"/>
+    </gazebo>
   <!-- Right wheel model "link" "joint" "transmission" "gazebo" -->
   <!-- ========================================================================== -->
@@ -66,5 +73,5 @@
 			<origin xyz="0 0 0" rpy="0 0 3.142"/>
 			<geometry>
-				<mesh filename="package://littlebot_description/meshes/roda.dae" />
+				<mesh filename="/home/nestor/Documents/littlebot/littlebot_ws/src/littlebot/littlebot_description/meshes/roda.dae" />
 			</geometry>
 		</visual>
@@ -72,5 +79,5 @@
 			<origin xyz="0 0 0" rpy="0 0 3.142"/>
 			<geometry>
-				<mesh filename="package://littlebot_description/meshes/roda.dae" />
+				<mesh filename="/home/nestor/Documents/littlebot/littlebot_ws/src/littlebot/littlebot_description/meshes/roda.dae" />
 			</geometry>
 		</collision>
@@ -87,3 +94,37 @@
 		<axis xyz="0 1 0" rpy="0 0 0" />
 	</joint>
+  <gazebo reference="right_wheel">
+    <mu1 value="1.0"/>
+    <mu2 value="0.5"/>
+    <kp value="10000000.0" />
+    <kd value="1.0" />
+    <fdir1 value="1 0 0"/>
+  </gazebo>
+<!-- ============================================================================= -->
+	<gazebo>
+    <plugin name="gazebo_ros2_control" filename="libgazebo_ros2_control.so">
+      <parameters>"$(find littlebot_control)/config/control.yaml"</parameters>
+    </plugin>
+  </gazebo>
+	<ros2_control name="littlebot_hardware" type="system">
+    <hardware>
+      <plugin>gazebo_ros2_control/GazeboSystem</plugin>
+    </hardware>
+    <joint name="base_to_left_wheel">
+      <command_interface name="velocity">
+        <param name="min">-1</param>
+        <param name="max">1</param>
+      </command_interface>
+      <state_interface name="position"/>
+      <state_interface name="velocity"/>
+    </joint>
+    <joint name="base_to_right_wheel">
+      <command_interface name="velocity">
+        <param name="min">-1</param>
+        <param name="max">1</param>
+      </command_interface>
+      <state_interface name="position"/>
+      <state_interface name="velocity"/>
+    </joint>
+  </ros2_control>
 </robot>

Commit message: included IMU in simulation

File: littlebot_description/urdf/littlebot_description.urdf.xacro (robot description, xacro)
@@ -32,4 +32,30 @@
     <child link="chassis"/>
     <origin xyz="0.0 0.0 0.0" rpy="0 0 0" />
+  </joint>
+ <!-- Modelagem da IMU MPU-6050 "link" "joint" -->
+ <!-- ========================================================================== -->
+ <link name="imu_link">
+    <visual>
+      <origin xyz="0 0 0" rpy="0 0 0" />
+      <geometry>
+        <mesh filename="file://$(find littlebot_description)/meshes/MPU_6050.dae" />
+      </geometry>
+    </visual>
+    <collision>
+      <origin xyz="0 0 0" rpy="0 0 0" />
+      <geometry>
+	      <mesh filename="file://$(find littlebot_description)/meshes/MPU_6050.dae" />
+      </geometry>
+    </collision>
+    <inertial>
+      <origin xyz="0 0 0" rpy="0 0 0"/>
+      <mass value="0.00142672"/>
+      <inertia ixx="4.54052487e-8"  ixy="1.07305074e-10"  ixz="-2.17782593e-10" iyy="2.70451174e-8" iyz="-4.58999382e-11" izz="7.14041804e-8" />
+    </inertial>
+  </link>
+  <joint name="chassis_to_imu" type="fixed">
+    <parent link="chassis"/>
+    <child link="imu_link"/>
+    <origin xyz="0.028 0.0 0.005" rpy="0 0 0" />
   </joint>
   <!-- Left whell model "link" "joint" "transmission" "gazebo" -->
@@ -128,3 +154,17 @@
     </joint>
   </ros2_control>
+  <gazebo reference="imu_link">
+    <sensor name="imu_sensor" type="imu">
+      <plugin filename="libgazebo_ros_imu_sensor.so" name="imu_plugin">
+        <ros>
+          <namespace>/</namespace>
+          <remapping>~/out:=imu/data_raw</remapping>
+        </ros>
+        <initial_orientation_as_reference>false</initial_orientation_as_reference>
+      </plugin>
+      <always_on>true</always_on>
+      <update_rate>100</update_rate>
+      <visualize>true</visualize>
+    </sensor>
+  </gazebo>
 </robot>

Commit message: find comand in URDF file

File: littlebot_description/urdf/littlebot_description.urdf.xacro (robot description, xacro)
@@ -13,5 +13,5 @@
       <origin xyz="0 0 0" rpy="0 0 0" />
       <geometry>
-        <mesh filename="/home/nestor/Documents/littlebot/littlebot_ws/src/littlebot/littlebot_description/meshes/littlebot.dae" />
+        <mesh filename="file://$(find littlebot_description)/meshes/littlebot.dae" />
       </geometry>
     </visual>
@@ -19,5 +19,5 @@
       <origin xyz="0 0 0" rpy="0 0 0" />
       <geometry>
-	      <mesh filename="/home/nestor/Documents/littlebot/littlebot_ws/src/littlebot/littlebot_description/meshes/chassis.dae" />
+	      <mesh filename="file://$(find littlebot_description)/meshes/chassis.dae" />
       </geometry>
     </collision>
@@ -65,5 +65,5 @@
 			<origin xyz="0.0 0 0" rpy="0 0 0"/>
 			<geometry>
-				<mesh filename="/home/nestor/Documents/littlebot/littlebot_ws/src/littlebot/littlebot_description/meshes/roda.dae" />
+				<mesh filename="file://$(find littlebot_description)/meshes/roda.dae" />
 			</geometry>
 		</visual>
@@ -71,5 +71,5 @@
 			<origin xyz="0.0 0 0" rpy="0 0 0"/>
 			<geometry>
-				<mesh filename="/home/nestor/Documents/littlebot/littlebot_ws/src/littlebot/littlebot_description/meshes/roda.dae" />
+				<mesh filename="file://$(find littlebot_description)/meshes/roda.dae" />
 			</geometry>
 		</collision>
@@ -99,5 +99,5 @@
 			<origin xyz="0 0 0" rpy="0 0 3.142"/>
 			<geometry>
-				<mesh filename="/home/nestor/Documents/littlebot/littlebot_ws/src/littlebot/littlebot_description/meshes/roda.dae" />
+				<mesh filename="file://$(find littlebot_description)/meshes/roda.dae" />
 			</geometry>
 		</visual>
@@ -105,5 +105,5 @@
 			<origin xyz="0 0 0" rpy="0 0 3.142"/>
 			<geometry>
-				<mesh filename="/home/nestor/Documents/littlebot/littlebot_ws/src/littlebot/littlebot_description/meshes/roda.dae" />
+				<mesh filename="file://$(find littlebot_description)/meshes/roda.dae" />
 			</geometry>
 		</collision>

Commit message: created the sonar xacro file

File: littlebot_description/urdf/littlebot_description.urdf.xacro (robot description, xacro)
@@ -3,5 +3,5 @@
 <!-- Included URDF XACRO Files -->
 <!-- <xacro:include filename="$(find littlebot_description)/urdf/littlebot_wheel.urdf.xacro" /> -->
-<!-- <xacro:include filename="$(find littlebot_description)/urdf/sonar.xacro" /> -->
+<xacro:include filename="$(find littlebot_description)/urdf/littlebot_sonar.urdf.xacro" />
   <!-- Modelagem base_link "link" -->
   <link name="base_link">
@@ -127,5 +127,28 @@
     <fdir1 value="1 0 0"/>
   </gazebo>
-<!-- ============================================================================= -->
+<!-- Modelagem do sonar "link" "joint" -->
+<!-- ========================================================================== -->
+  <xacro:littlebot_sonar sonar_numero="1">
+    <origin xyz="0 0 -0.020267" rpy="0 0 0" />
+    <origin xyz="0.07879836 0.03772198 0.02500000" rpy="0 0 0.686455448" />
+  </xacro:littlebot_sonar>
+  <xacro:littlebot_sonar sonar_numero="2">
+    <origin xyz="0 0 -0.020267" rpy="0 0 0" />
+    <origin xyz="0.08880761 0.02002920 0.02500000" rpy="0 0 0.343218997"/>
+  </xacro:littlebot_sonar>
+  <xacro:littlebot_sonar sonar_numero="3">
+    <origin xyz="0 0 -0.020267" rpy="0 0 0" />
+    <origin xyz="0.092279 0.0 0.02500000" rpy="0 0 0" />
+  </xacro:littlebot_sonar>
+  <xacro:littlebot_sonar sonar_numero="4">
+    <origin xyz="0 0 -0.020267" rpy="0 0 0" />
+    <origin xyz="0.08880761 -0.02002920 0.02500000" rpy="0 0 -0.343218997"/>
+  </xacro:littlebot_sonar>
+  <xacro:littlebot_sonar sonar_numero="5">
+    <origin xyz="0 0 -0.020267" rpy="0 0 0" />
+    <origin xyz="0.07879836 -0.03772198 0.02500000" rpy="0 0 -0.686455448"/>
+  </xacro:littlebot_sonar>
+<!-- Plugin control -->
+<!-- ***************************************************************************** -->
 	<gazebo>
     <plugin name="gazebo_ros2_control" filename="libgazebo_ros2_control.so">
@@ -154,4 +177,6 @@
     </joint>
   </ros2_control>
+<!-- Plugin IMU -->
+<!-- ***************************************************************************** -->
   <gazebo reference="imu_link">
     <sensor name="imu_sensor" type="imu">

Commit message: added sensor range plugin

File: littlebot_description/urdf/littlebot_description.urdf.xacro (robot description, xacro)
@@ -149,5 +149,5 @@
     <origin xyz="0.07879836 -0.03772198 0.02500000" rpy="0 0 -0.686455448"/>
   </xacro:littlebot_sonar>
-<!-- Plugin control -->
+<!-- Plugin CONTROLER -->
 <!-- ***************************************************************************** -->
 	<gazebo>
@@ -193,3 +193,87 @@
     </sensor>
   </gazebo>
+<!-- Plugin SONAR -->
+<!-- ***************************************************************************** -->
+  <xacro:macro name="sonar" params="reference topic_name">
+    <gazebo reference="${reference}">
+      <sensor type="ray" name="TeraRanger">
+        <pose>0 0 0 0 0 0</pose>
+        <visualize>false</visualize>
+        <update_rate>50</update_rate>
+        <ray>
+          <scan>
+              <horizontal>
+                <samples>10</samples>
+                <resolution>1</resolution>
+                <min_angle>-0.14835</min_angle>
+                <max_angle>0.14835</max_angle>
+              </horizontal>
+              <vertical>
+                <samples>10</samples>
+                <resolution>1</resolution>
+                <min_angle>-0.14835</min_angle>
+                <max_angle>0.14835</max_angle>
+              </vertical>
+          </scan>
+          <range>
+              <min>0.01</min>
+              <max>2</max>
+              <resolution>0.02</resolution>
+          </range>
+          <noise>
+            <type>gaussian</type>
+            <mean>0.0</mean>
+            <stddev>0.005</stddev>
+          </noise>
+        </ray>
+        <plugin name="gazebo_ros_range_controller" filename="libgazebo_ros_ray_sensor.so">
+          <ros>
+            <!-- <namespace>/</namespace> -->
+            <remapping>~/out:=sensor/${topic_name}</remapping>
+          </ros>
+          <output_type>sensor_msgs/Range</output_type>
+          <frame_name> ${reference} </frame_name>
+        </plugin>
+        <!-- <plugin filename="libgazebo_ros_range.so" name="gazebo_ros_range">
+          <topicName>sensor/${topic_name}</topicName>
+          <frameName>${reference}</frameName>
+          <gaussianNoise>0.005</gaussianNoise>
+          <updateRate>50</updateRate>
+          <fov>0.2967</fov>
+          <alwaysOn>true</alwaysOn>
+          <radiation>ULTRASOUND</radiation>
+        </plugin> -->
+      </sensor>
+    </gazebo>
+  </xacro:macro>
+  <!--
+  ******************************************************************************************
+  SONAR_01 gazebo plugin
+  ******************************************************************************************
+  -->
+  <xacro:sonar reference="sonar_1" topic_name="sonar1" />
+  <!--
+  ******************************************************************************************
+  SONAR02 gazebo plugin
+  ******************************************************************************************
+  -->
+  <xacro:sonar reference="sonar_2" topic_name="sonar2" />
+  <!--
+  ******************************************************************************************
+  SONAR03 gazebo plugin
+  ******************************************************************************************
+  -->
+  <xacro:sonar reference="sonar_3" topic_name="sonar3" />
+  <!--
+  ******************************************************************************************
+  SONAR04 gazebo plugin
+  ******************************************************************************************
+  -->
+  <xacro:sonar reference="sonar_4" topic_name="sonar4" />
+  <!--
+  ******************************************************************************************
+  SONAR05 gazebo plugin
+  ******************************************************************************************
+  -->
+  <xacro:sonar reference="sonar_5" topic_name="sonar5" />
 </robot>

Commit message: wheel xacro done

File: littlebot_description/urdf/littlebot_description.urdf.xacro (robot description, xacro)
@@ -2,5 +2,5 @@
 <robot xmlns:xacro="http://ros.org/wiki/xacro"  name="littlebot">
 <!-- Included URDF XACRO Files -->
-<!-- <xacro:include filename="$(find littlebot_description)/urdf/littlebot_wheel.urdf.xacro" /> -->
+<xacro:include filename="$(find littlebot_description)/urdf/littlebot_wheel.urdf.xacro" />
 <xacro:include filename="$(find littlebot_description)/urdf/littlebot_sonar.urdf.xacro" />
   <!-- Modelagem base_link "link" -->
@@ -25,5 +25,7 @@
       <origin xyz="0 0 0" rpy="0 0 0"/>
       <mass value="0.19357368"/>
-      <inertia ixx="1.84569610e-4"  ixy="-4.09475462e-6"  ixz="-2.91063667e-5" iyy="7.65700035e-4" iyz="2.32776537e-8" izz="9.00861891e-4" />
+      <inertia ixx="1.84569610e-4"  ixy="-4.09475462e-6"  ixz="-2.91063667e-5"
+                                    iyy="7.65700035e-4"   iyz="2.32776537e-8"
+                                                          izz="9.00861891e-4" />
     </inertial>
   </link>
@@ -51,5 +53,7 @@
       <origin xyz="0 0 0" rpy="0 0 0"/>
       <mass value="0.00142672"/>
-      <inertia ixx="4.54052487e-8"  ixy="1.07305074e-10"  ixz="-2.17782593e-10" iyy="2.70451174e-8" iyz="-4.58999382e-11" izz="7.14041804e-8" />
+      <inertia ixx="4.54052487e-8"  ixy="1.07305074e-10"  ixz="-2.17782593e-10"
+                                    iyy="2.70451174e-8"   iyz="-4.58999382e-11"
+                                                          izz="7.14041804e-8" />
     </inertial>
   </link>
@@ -59,72 +63,14 @@
     <origin xyz="0.028 0.0 0.005" rpy="0 0 0" />
   </joint>
-  <!-- Left whell model "link" "joint" "transmission" "gazebo" -->
+  <!-- Whells model "link" "joint" "transmission" "gazebo" -->
   <!-- ========================================================================== -->
-	<link name="left_wheel">
-		<visual>
-			<origin xyz="0.0 0 0" rpy="0 0 0"/>
-			<geometry>
-				<mesh filename="file://$(find littlebot_description)/meshes/roda.dae" />
-			</geometry>
-		</visual>
-		<collision>
-			<origin xyz="0.0 0 0" rpy="0 0 0"/>
-			<geometry>
-				<mesh filename="file://$(find littlebot_description)/meshes/roda.dae" />
-			</geometry>
-		</collision>
-		<inertial>
-			<origin xyz="0.0 0 0" rpy="0 0 0"/>
-			<mass value="0.041"/>
-			<inertia ixx="2.967e-5"  ixy="-7.675e-15"  ixz="-4.765e-14" iyy="1.616e-5" iyz="-1.121e-16" izz="1.616e-5" />
-    	</inertial>
-	</link>
-	<joint name="base_to_left_wheel" type="continuous">
-		<parent link="chassis"/>
-		<child link="left_wheel"/>
-		<origin xyz="0.0281 0.067 -0.01425" rpy="0 0 0" />
-		<axis xyz="0 1 0" rpy="0 0 0" />
-	</joint>
-	<gazebo reference="left_wheel">
-      <mu1 value="1.0"/>
-      <mu2 value="0.5"/>
-      <kp value="10000000.0" />
-      <kd value="1.0" />
-      <fdir1 value="1 0 0"/>
-    </gazebo>
-  <!-- Right wheel model "link" "joint" "transmission" "gazebo" -->
-  <!-- ========================================================================== -->
-	<link name="right_wheel">
-		<visual>
-			<origin xyz="0 0 0" rpy="0 0 3.142"/>
-			<geometry>
-				<mesh filename="file://$(find littlebot_description)/meshes/roda.dae" />
-			</geometry>
-		</visual>
-		<collision>
-			<origin xyz="0 0 0" rpy="0 0 3.142"/>
-			<geometry>
-				<mesh filename="file://$(find littlebot_description)/meshes/roda.dae" />
-			</geometry>
-		</collision>
-		<inertial>
-			<origin xyz="0 0 0" rpy="0 0 3.142"/>
-			<mass value="0.041"/>
-			<inertia ixx="2.967e-5"  ixy="-7.675e-15"  ixz="-4.765e-14" iyy="1.616e-5" iyz="-1.121e-16" izz="1.616e-5" />
-    	</inertial>
-	</link>
-	<joint name="base_to_right_wheel" type="continuous">
-		<parent link="chassis"/>
-		<child link="right_wheel"/>
-		<origin xyz="0.0281 -0.067 -0.01425" rpy="0 0 0" />
-		<axis xyz="0 1 0" rpy="0 0 0" />
-	</joint>
-  <gazebo reference="right_wheel">
-    <mu1 value="1.0"/>
-    <mu2 value="0.5"/>
-    <kp value="10000000.0" />
-    <kd value="1.0" />
-    <fdir1 value="1 0 0"/>
-  </gazebo>
+  <xacro:littlebot_wheel side_wheel="left">
+    <origin xyz="0.0 0 0" rpy="0 0 0"/>
+    <origin xyz="0.0281 0.067 -0.01425" rpy="0 0 0" />
+  </xacro:littlebot_wheel>
+  <xacro:littlebot_wheel side_wheel="right">
+    <origin xyz="0 0 0" rpy="0 0 3.142"/>
+    <origin xyz="0.0281 -0.067 -0.01425" rpy="0 0 0" />
+  </xacro:littlebot_wheel>
 <!-- Modelagem do sonar "link" "joint" -->
 <!-- ========================================================================== -->
@@ -237,33 +183,10 @@
     </gazebo>
   </xacro:macro>
-  <!--
-  ******************************************************************************************
-  SONAR_01 gazebo plugin
-  ******************************************************************************************
-  -->
+<!-- Call SONAR gazebo plugin xacro -->
+<!-- ***************************************************************************** -->
   <xacro:sonar reference="sonar_1" topic_name="sonar1" />
-  <!--
-  ******************************************************************************************
-  SONAR02 gazebo plugin
-  ******************************************************************************************
-  -->
   <xacro:sonar reference="sonar_2" topic_name="sonar2" />
-  <!--
-  ******************************************************************************************
-  SONAR03 gazebo plugin
-  ******************************************************************************************
-  -->
   <xacro:sonar reference="sonar_3" topic_name="sonar3" />
-  <!--
-  ******************************************************************************************
-  SONAR04 gazebo plugin
-  ******************************************************************************************
-  -->
   <xacro:sonar reference="sonar_4" topic_name="sonar4" />
-  <!--
-  ******************************************************************************************
-  SONAR05 gazebo plugin
-  ******************************************************************************************
-  -->
   <xacro:sonar reference="sonar_5" topic_name="sonar5" />
 </robot>
