Commit message: removed unnecessary comment

File: littlebot_description/urdf/littlebot_description.urdf.xacro (robot description, xacro)
@@ -35,7 +35,7 @@
     <origin xyz="0.0 0.0 0.0" rpy="0 0 0" />
   </joint>
- <!-- Modelagem da IMU MPU-6050 "link" "joint" -->
- <!-- ========================================================================== -->
- <link name="imu_link">
+  <!-- Modelagem da IMU MPU-6050 "link" "joint" -->
+  <!-- ========================================================================== -->
+  <link name="imu_link">
     <visual>
       <origin xyz="0 0 0" rpy="0 0 0" />

Commit message: split urdf , create littlebot_robot urdf file

File: littlebot_description/urdf/littlebot_description.urdf.xacro (robot description, xacro)
@@ -1,68 +1,15 @@
 <?xml version="1.0"?>
 <robot xmlns:xacro="http://ros.org/wiki/xacro"  name="littlebot">
-<!-- Included URDF XACRO Files -->
-<xacro:include filename="$(find littlebot_description)/urdf/littlebot_wheel.urdf.xacro" />
-<xacro:include filename="$(find littlebot_description)/urdf/littlebot_sonar.urdf.xacro" />
-  <!-- Modelagem base_link "link" -->
-  <link name="base_link">
-  </link>
-  <!-- Modelagem chassis "link" and "joint"-->
+  <xacro:arg name="use_sim" default="false" />
+  <xacro:arg name="prefix" default="littlebot" />
+  <!-- Included URDF XACRO Files -->
+  <xacro:include filename="$(find littlebot_description)/urdf/littlebot_wheel.urdf.xacro" />
+  <xacro:include filename="$(find littlebot_description)/urdf/littlebot_sonar.urdf.xacro" />
+  <xacro:include filename="$(find littlebot_description)/urdf/littlebot_robot.urdf.xacro" />
+  <!-- Littlebot's robot description -->
   <!-- ========================================================================== -->
-  <link name="chassis">
-    <visual>
-      <origin xyz="0 0 0" rpy="0 0 0" />
-      <geometry>
-        <mesh filename="file://$(find littlebot_description)/meshes/littlebot.dae" />
-      </geometry>
-    </visual>
-    <collision>
-      <origin xyz="0 0 0" rpy="0 0 0" />
-      <geometry>
-	      <mesh filename="file://$(find littlebot_description)/meshes/chassis.dae" />
-      </geometry>
-    </collision>
-    <inertial>
-      <origin xyz="0 0 0" rpy="0 0 0"/>
-      <mass value="0.19357368"/>
-      <inertia ixx="1.84569610e-4"  ixy="-4.09475462e-6"  ixz="-2.91063667e-5"
-                                    iyy="7.65700035e-4"   iyz="2.32776537e-8"
-                                                          izz="9.00861891e-4" />
-    </inertial>
-  </link>
-  <joint name="base_to_chassis" type="fixed">
-    <parent link="base_link"/>
-    <child link="chassis"/>
-    <origin xyz="0.0 0.0 0.0" rpy="0 0 0" />
-  </joint>
-  <!-- Modelagem da IMU MPU-6050 "link" "joint" -->
-  <!-- ========================================================================== -->
-  <link name="imu_link">
-    <visual>
-      <origin xyz="0 0 0" rpy="0 0 0" />
-      <geometry>
-        <mesh filename="file://$(find littlebot_description)/meshes/MPU_6050.dae" />
-      </geometry>
-    </visual>
-    <collision>
-      <origin xyz="0 0 0" rpy="0 0 0" />
-      <geometry>
-	      <mesh filename="file://$(find littlebot_description)/meshes/MPU_6050.dae" />
-      </geometry>
-    </collision>
-    <inertial>
-      <origin xyz="0 0 0" rpy="0 0 0"/>
-      <mass value="0.00142672"/>
-      <inertia ixx="4.54052487e-8"  ixy="1.07305074e-10"  ixz="-2.17782593e-10"
-                                    iyy="2.70451174e-8"   iyz="-4.58999382e-11"
-                                                          izz="7.14041804e-8" />
-    </inertial>
-  </link>
-  <joint name="chassis_to_imu" type="fixed">
-    <parent link="chassis"/>
-    <child link="imu_link"/>
-    <origin xyz="0.028 0.0 0.005" rpy="0 0 0" />
-  </joint>
-  <!-- Whells model "link" "joint" "transmission" "gazebo" -->
-  <!-- ========================================================================== -->
+  <!-- Body model -->
+  <xacro:littlebot_robot />
+  <!-- Whells model -->
   <xacro:littlebot_wheel side_wheel="left">
     <origin xyz="0.0 0 0" rpy="0 0 0"/>
@@ -73,6 +20,5 @@
     <origin xyz="0.0281 -0.067 -0.01425" rpy="0 0 0" />
   </xacro:littlebot_wheel>
-<!-- Modelagem do sonar "link" "joint" -->
-<!-- ========================================================================== -->
+  <!-- Modelagem do sonar -->
   <xacro:littlebot_sonar sonar_numero="1">
     <origin xyz="0 0 -0.020267" rpy="0 0 0" />
@@ -95,98 +41,98 @@
     <origin xyz="0.07879836 -0.03772198 0.02500000" rpy="0 0 -0.686455448"/>
   </xacro:littlebot_sonar>
-<!-- Plugin CONTROLER -->
-<!-- ***************************************************************************** -->
-	<gazebo>
-    <plugin name="gazebo_ros2_control" filename="libgazebo_ros2_control.so">
-      <parameters>$(find littlebot_control)/config/control.yaml</parameters>
-    </plugin>
-  </gazebo>
-	<ros2_control name="littlebot_hardware" type="system">
-    <hardware>
-      <plugin>gazebo_ros2_control/GazeboSystem</plugin>
-    </hardware>
-    <joint name="base_to_left_wheel">
-      <command_interface name="velocity">
-        <param name="min">-1</param>
-        <param name="max">1</param>
-      </command_interface>
-      <state_interface name="position"/>
-      <state_interface name="velocity"/>
-    </joint>
-    <joint name="base_to_right_wheel">
-      <command_interface name="velocity">
-        <param name="min">-1</param>
-        <param name="max">1</param>
-      </command_interface>
-      <state_interface name="position"/>
-      <state_interface name="velocity"/>
-    </joint>
-  </ros2_control>
-<!-- Plugin IMU -->
-<!-- ***************************************************************************** -->
-  <gazebo reference="imu_link">
-    <sensor name="imu_sensor" type="imu">
-      <plugin filename="libgazebo_ros_imu_sensor.so" name="imu_plugin">
-        <ros>
-          <namespace>/</namespace>
-          <remapping>~/out:=imu/data_raw</remapping>
-        </ros>
-        <initial_orientation_as_reference>false</initial_orientation_as_reference>
+  <!-- Plugin CONTROLER -->
+  <!-- ***************************************************************************** -->
+    <!-- <gazebo>
+      <plugin name="gazebo_ros2_control" filename="libgazebo_ros2_control.so">
+        <parameters>$(find littlebot_control)/config/control.yaml</parameters>
       </plugin>
-      <always_on>true</always_on>
-      <update_rate>100</update_rate>
-      <visualize>true</visualize>
-    </sensor>
-  </gazebo>
-<!-- Plugin SONAR -->
-<!-- ***************************************************************************** -->
-  <xacro:macro name="sonar" params="reference topic_name">
-    <gazebo reference="${reference}">
-      <sensor type="ray" name="TeraRanger">
-        <update_rate>50</update_rate>
-        <ray>
-          <scan>
-            <horizontal>
-              <samples>10</samples>
-              <resolution>1</resolution>
-              <min_angle>-0.14835</min_angle>
-              <max_angle>0.14835</max_angle>
-            </horizontal>
-            <vertical>
-              <samples>10</samples>
-              <resolution>1</resolution>
-              <min_angle>-0.14835</min_angle>
-              <max_angle>0.14835</max_angle>
-            </vertical>
-          </scan>
-          <range>
-            <min>0.01</min>
-            <max>2</max>
-            <resolution>0.02</resolution>
-          </range>
-          <noise>
-            <type>gaussian</type>
-            <mean>0.0</mean>
-            <stddev>0.005</stddev>
-          </noise>
-        </ray>
-        <plugin name="gazebo_ros_range_controller" filename="libgazebo_ros_ray_sensor.so">
+    </gazebo>
+    <ros2_control name="littlebot_hardware" type="system">
+      <hardware>
+        <plugin>gazebo_ros2_control/GazeboSystem</plugin>
+      </hardware>
+      <joint name="base_to_left_wheel">
+        <command_interface name="velocity">
+          <param name="min">-1</param>
+          <param name="max">1</param>
+        </command_interface>
+        <state_interface name="position"/>
+        <state_interface name="velocity"/>
+      </joint>
+      <joint name="base_to_right_wheel">
+        <command_interface name="velocity">
+          <param name="min">-1</param>
+          <param name="max">1</param>
+        </command_interface>
+        <state_interface name="position"/>
+        <state_interface name="velocity"/>
+      </joint>
+    </ros2_control> -->
+  <!-- Plugin IMU -->
+  <!-- ***************************************************************************** -->
+    <!-- <gazebo reference="imu_link">
+      <sensor name="imu_sensor" type="imu">
+        <plugin filename="libgazebo_ros_imu_sensor.so" name="imu_plugin">
           <ros>
-            <!-- <namespace>/</namespace> -->
-            <remapping>~/out:=sensor/${topic_name}</remapping>
+            <namespace>/</namespace>
+            <remapping>~/out:=imu/data_raw</remapping>
           </ros>
-          <output_type>sensor_msgs/Range</output_type>
-          <frame_name>${reference}</frame_name>
-          <radiation_type>ultrasound</radiation_type>
+          <initial_orientation_as_reference>false</initial_orientation_as_reference>
         </plugin>
+        <always_on>true</always_on>
+        <update_rate>100</update_rate>
+        <visualize>true</visualize>
       </sensor>
-    </gazebo>
-  </xacro:macro>
-<!-- Call SONAR gazebo plugin xacro -->
-<!-- ***************************************************************************** -->
-  <xacro:sonar reference="sonar_1" topic_name="sonar1" />
-  <xacro:sonar reference="sonar_2" topic_name="sonar2" />
-  <xacro:sonar reference="sonar_3" topic_name="sonar3" />
-  <xacro:sonar reference="sonar_4" topic_name="sonar4" />
-  <xacro:sonar reference="sonar_5" topic_name="sonar5" />
+    </gazebo> -->
+  <!-- Plugin SONAR -->
+  <!-- ***************************************************************************** -->
+    <!-- <xacro:macro name="sonar" params="reference topic_name">
+      <gazebo reference="${reference}">
+        <sensor type="ray" name="TeraRanger">
+          <update_rate>50</update_rate>
+          <ray>
+            <scan>
+              <horizontal>
+                <samples>10</samples>
+                <resolution>1</resolution>
+                <min_angle>-0.14835</min_angle>
+                <max_angle>0.14835</max_angle>
+              </horizontal>
+              <vertical>
+                <samples>10</samples>
+                <resolution>1</resolution>
+                <min_angle>-0.14835</min_angle>
+                <max_angle>0.14835</max_angle>
+              </vertical>
+            </scan>
+            <range>
+              <min>0.01</min>
+              <max>2</max>
+              <resolution>0.02</resolution>
+            </range>
+            <noise>
+              <type>gaussian</type>
+              <mean>0.0</mean>
+              <stddev>0.005</stddev>
+            </noise>
+          </ray> -->
+          <!-- <plugin name="gazebo_ros_range_controller" filename="libgazebo_ros_ray_sensor.so">
+            <ros>
+              <namespace>/</namespace>
+              <remapping>~/out:=sensor/${topic_name}</remapping>
+            </ros>
+            <output_type>sensor_msgs/Range</output_type>
+            <frame_name>${reference}</frame_name>
+            <radiation_type>ultrasound</radiation_type>
+          </plugin>
+        </sensor>
+      </gazebo>
+    </xacro:macro> -->
+  <!-- Call SONAR gazebo plugin xacro -->
+  <!-- ***************************************************************************** -->
+    <!-- <xacro:sonar reference="sonar_1" topic_name="sonar1" />
+    <xacro:sonar reference="sonar_2" topic_name="sonar2" />
+    <xacro:sonar reference="sonar_3" topic_name="sonar3" />
+    <xacro:sonar reference="sonar_4" topic_name="sonar4" />
+    <xacro:sonar reference="sonar_5" topic_name="sonar5" /> -->
 </robot>

File: littlebot_description/urdf/littlebot_wheel.urdf.xacro (robot description, xacro)
@@ -1,46 +1,37 @@
 <?xml version="1.0"?>
 <robot name="littlebot_wheel" xmlns:xacro="http://ros.org/wiki/xacro" >
-<xacro:macro name="littlebot_wheel" params="side_wheel *mesh_wheel_pose *joint_wheel_pose">
-  <link name="${side_wheel}_wheel">
-    <visual>
-      <xacro:insert_block name="mesh_wheel_pose"/>
-      <geometry>
-        <mesh filename="file://$(find littlebot_description)/meshes/roda.dae" />
-      </geometry>
-    </visual>
-    <collision>
-      <xacro:insert_block name="mesh_wheel_pose"/>
-      <geometry>
-        <mesh filename="file://$(find littlebot_description)/meshes/roda.dae" />
-      </geometry>
-    </collision>
-    <inertial>
-      <xacro:insert_block name="mesh_wheel_pose"/>
-      <mass value="0.041"/>
-      <inertia ixx="2.967e-5"  ixy="-7.675e-15"  ixz="-4.765e-14" iyy="1.616e-5" iyz="-1.121e-16" izz="1.616e-5" />
-    </inertial>
-  </link>
-  <joint name="base_to_${side_wheel}_wheel" type="continuous">
-    <parent link="chassis"/>
-    <child link="${side_wheel}_wheel"/>
-    <xacro:insert_block name="joint_wheel_pose"/>
-    <axis xyz="0 1 0" rpy="0 0 0" />
-  </joint>
-  <!-- <transmission name="trans_${side_wheel}_wheel">
-  <type>transmission_interface/SimpleTransmission</type>
-  <joint name="base_to_${side_wheel}_wheel">
-  <hardwareInterface>hardware_interface/VelocityJointInterface</hardwareInterface>
-  </joint>
-  <actuator name="${side_wheel}_wheel_motor">
-  <mechanicalReduction>1</mechanicalReduction>
-  </actuator>
-  </transmission> -->
-  <gazebo reference="${side_wheel}_wheel">
-    <mu1 value="1000.0"/>
-    <mu2 value="1.0"/>
-    <kp value="10000000.0" />
-    <kd value="1.0" />
-    <fdir1 value="1 0 0"/>
-  </gazebo>
-</xacro:macro>
+  <xacro:macro name="littlebot_wheel" params="side_wheel *mesh_wheel_pose *joint_wheel_pose">
+    <link name="${side_wheel}_wheel">
+      <visual>
+        <xacro:insert_block name="mesh_wheel_pose"/>
+        <geometry>
+          <mesh filename="file://$(find littlebot_description)/meshes/roda.dae" />
+        </geometry>
+      </visual>
+      <collision>
+        <xacro:insert_block name="mesh_wheel_pose"/>
+        <geometry>
+          <mesh filename="file://$(find littlebot_description)/meshes/roda.dae" />
+        </geometry>
+      </collision>
+      <inertial>
+        <xacro:insert_block name="mesh_wheel_pose"/>
+        <mass value="0.041"/>
+        <inertia ixx="2.967e-5"  ixy="-7.675e-15"  ixz="-4.765e-14" iyy="1.616e-5" iyz="-1.121e-16" izz="1.616e-5" />
+      </inertial>
+    </link>
+    <joint name="base_to_${side_wheel}_wheel" type="continuous">
+      <parent link="chassis"/>
+      <child link="${side_wheel}_wheel"/>
+      <xacro:insert_block name="joint_wheel_pose"/>
+      <axis xyz="0 1 0" rpy="0 0 0" />
+    </joint>
+    <gazebo reference="${side_wheel}_wheel">
+      <mu1 value="1000.0"/>
+      <mu2 value="1.0"/>
+      <kp value="10000000.0" />
+      <kd value="1.0" />
+      <fdir1 value="1 0 0"/>
+    </gazebo>
+  </xacro:macro>
 </robot>

Commit message: create .gazebo.xacro file

File: littlebot_description/urdf/littlebot_description.urdf.xacro (robot description, xacro)
@@ -1,4 +1,5 @@
 <?xml version="1.0"?>
 <robot xmlns:xacro="http://ros.org/wiki/xacro"  name="littlebot">
+  <!-- Default arguments -->
   <xacro:arg name="use_sim" default="false" />
   <xacro:arg name="prefix" default="littlebot" />
@@ -7,6 +8,8 @@
   <xacro:include filename="$(find littlebot_description)/urdf/littlebot_sonar.urdf.xacro" />
   <xacro:include filename="$(find littlebot_description)/urdf/littlebot_robot.urdf.xacro" />
+  <!-- Included GAZEBO XACRO Files -->
+  <xacro:include filename="$(find littlebot_description)/gazebo/littlebot.gazebo.xacro" />
   <!-- Littlebot's robot description -->
-  <!-- ========================================================================== -->
+  <!-- =========================================================== -->
   <!-- Body model -->
   <xacro:littlebot_robot />
@@ -41,98 +44,6 @@
     <origin xyz="0.07879836 -0.03772198 0.02500000" rpy="0 0 -0.686455448"/>
   </xacro:littlebot_sonar>
-  <!-- Plugin CONTROLER -->
-  <!-- ***************************************************************************** -->
-    <!-- <gazebo>
-      <plugin name="gazebo_ros2_control" filename="libgazebo_ros2_control.so">
-        <parameters>$(find littlebot_control)/config/control.yaml</parameters>
-      </plugin>
-    </gazebo>
-    <ros2_control name="littlebot_hardware" type="system">
-      <hardware>
-        <plugin>gazebo_ros2_control/GazeboSystem</plugin>
-      </hardware>
-      <joint name="base_to_left_wheel">
-        <command_interface name="velocity">
-          <param name="min">-1</param>
-          <param name="max">1</param>
-        </command_interface>
-        <state_interface name="position"/>
-        <state_interface name="velocity"/>
-      </joint>
-      <joint name="base_to_right_wheel">
-        <command_interface name="velocity">
-          <param name="min">-1</param>
-          <param name="max">1</param>
-        </command_interface>
-        <state_interface name="position"/>
-        <state_interface name="velocity"/>
-      </joint>
-    </ros2_control> -->
-  <!-- Plugin IMU -->
-  <!-- ***************************************************************************** -->
-    <!-- <gazebo reference="imu_link">
-      <sensor name="imu_sensor" type="imu">
-        <plugin filename="libgazebo_ros_imu_sensor.so" name="imu_plugin">
-          <ros>
-            <namespace>/</namespace>
-            <remapping>~/out:=imu/data_raw</remapping>
-          </ros>
-          <initial_orientation_as_reference>false</initial_orientation_as_reference>
-        </plugin>
-        <always_on>true</always_on>
-        <update_rate>100</update_rate>
-        <visualize>true</visualize>
-      </sensor>
-    </gazebo> -->
-  <!-- Plugin SONAR -->
-  <!-- ***************************************************************************** -->
-    <!-- <xacro:macro name="sonar" params="reference topic_name">
-      <gazebo reference="${reference}">
-        <sensor type="ray" name="TeraRanger">
-          <update_rate>50</update_rate>
-          <ray>
-            <scan>
-              <horizontal>
-                <samples>10</samples>
-                <resolution>1</resolution>
-                <min_angle>-0.14835</min_angle>
-                <max_angle>0.14835</max_angle>
-              </horizontal>
-              <vertical>
-                <samples>10</samples>
-                <resolution>1</resolution>
-                <min_angle>-0.14835</min_angle>
-                <max_angle>0.14835</max_angle>
-              </vertical>
-            </scan>
-            <range>
-              <min>0.01</min>
-              <max>2</max>
-              <resolution>0.02</resolution>
-            </range>
-            <noise>
-              <type>gaussian</type>
-              <mean>0.0</mean>
-              <stddev>0.005</stddev>
-            </noise>
-          </ray> -->
-          <!-- <plugin name="gazebo_ros_range_controller" filename="libgazebo_ros_ray_sensor.so">
-            <ros>
-              <namespace>/</namespace>
-              <remapping>~/out:=sensor/${topic_name}</remapping>
-            </ros>
-            <output_type>sensor_msgs/Range</output_type>
-            <frame_name>${reference}</frame_name>
-            <radiation_type>ultrasound</radiation_type>
-          </plugin>
-        </sensor>
-      </gazebo>
-    </xacro:macro> -->
-  <!-- Call SONAR gazebo plugin xacro -->
-  <!-- ***************************************************************************** -->
-    <!-- <xacro:sonar reference="sonar_1" topic_name="sonar1" />
-    <xacro:sonar reference="sonar_2" topic_name="sonar2" />
-    <xacro:sonar reference="sonar_3" topic_name="sonar3" />
-    <xacro:sonar reference="sonar_4" topic_name="sonar4" />
-    <xacro:sonar reference="sonar_5" topic_name="sonar5" /> -->
+  <!-- Load Gazebo plugins -->
+  <!-- =========================================================== -->
+  <xacro:littlebot_gazebo/>
 </robot>
