Commit message: simples forms for colision areas

File: littlebot_description/urdf/littlebot_robot.urdf.xacro (robot description, xacro)
@@ -15,7 +15,7 @@
       </visual>
       <collision>
-        <origin xyz="0 0 0" rpy="0 0 0" />
+        <origin xyz="0 0 0.018" rpy="0 0 0" />
         <geometry>
-          <mesh filename="file://$(find littlebot_description)/meshes/chassis.dae" />
+          <box size="0.21 0.11 0.05"/>
         </geometry>
       </collision>

File: littlebot_description/urdf/littlebot_wheel.urdf.xacro (robot description, xacro)
@@ -10,7 +10,9 @@
       </visual>
       <collision>
-        <xacro:insert_block name="mesh_wheel_pose"/>
+        <!-- <xacro:insert_block name="mesh_wheel_pose"/> -->
+        <origin xyz="0 0 0" rpy="1.571 0 0" />
         <geometry>
-          <mesh filename="file://$(find littlebot_description)/meshes/roda.dae" />
+          <cylinder length="0.018" radius="0.03298"/>
+          <!-- <mesh filename="file://$(find littlebot_description)/meshes/roda.dae" /> -->
         </geometry>
       </collision>

Commit message: Caster wheel added into robot model

File: littlebot_description/urdf/littlebot_robot.urdf.xacro (robot description, xacro)
@@ -3,8 +3,9 @@
   <xacro:macro name="littlebot_robot" >
     <!-- Modelagem base_link "link" -->
+    <!-- ********************************************************* -->
     <link name="base_link">
     </link>
     <!-- Modelagem chassis "link" and "joint"-->
-    <!-- ========================================================================== -->
+    <!-- ********************************************************* -->
     <link name="chassis">
       <visual>
@@ -33,6 +34,62 @@
       <origin xyz="0.0 0.0 0.0" rpy="0 0 0" />
     </joint>
+    <!-- Modelagem caster wheel-->
+    <!-- ********************************************************* -->
+    <link name="caster">
+      <visual>
+        <origin xyz="0 0 0" rpy="3.14 0 3.14" />
+        <geometry>
+          <mesh filename="file://$(find littlebot_description)/meshes/Caster_Wheel_Plate.dae" />
+        </geometry>
+      </visual>
+      <collision>
+        <origin xyz="0 0 0.0" rpy="3.14 0 3.14" />
+        <geometry>
+          <mesh filename="file://$(find littlebot_description)/meshes/Caster_Wheel_Plate.dae" />
+        </geometry>
+      </collision>
+      <inertial>
+        <origin xyz="0 0 0" rpy="3.14 0 3.14"/>
+        <mass value="0.01"/>
+        <inertia ixx="8.4e-7" ixy="-1.571e-14"  ixz="-1.601e-7"
+                              iyy="8.4e-7"      iyz="1.55e-14"
+                                                izz="1.304e-6" />
+      </inertial>
+    </link>
+    <joint name="chassis_to_caster" type="fixed">
+      <parent link="chassis"/>
+      <child link="caster"/>
+      <origin xyz="-0.0871 0.0 -0.00875" rpy="0 0 0" />
+    </joint>
+    <!-- Modelagem free wheel-->
+    <!-- ********************************************************* -->
+    <link name="free_wheel">
+      <visual>
+        <origin xyz="0 0 0" rpy="0 0 0" />
+        <geometry>
+          <mesh filename="file://$(find littlebot_description)/meshes/Wheel.dae" />
+        </geometry>
+      </visual>
+      <collision>
+        <origin xyz="0 0 0.0" rpy="0 0 0" />
+        <geometry>
+          <mesh filename="file://$(find littlebot_description)/meshes/Wheel.dae" />
+        </geometry>
+      </collision>
+      <inertial>
+        <origin xyz="0 0 0" rpy="0 0 0"/>
+        <mass value="0.007"/>
+        <inertia ixx="3.6e-7" ixy="0"         ixz="0"
+                              iyy="5.344e-7"  iyz="0"
+                                              izz="3.569e-7" />
+      </inertial>
+    </link>
+    <joint name="chassis_to_free_wheel" type="fixed">
+      <parent link="chassis"/>
+      <child link="free_wheel"/>
+      <origin xyz="-0.102 0.0 -0.0245" rpy="0 0 0" />
+    </joint>
     <!-- Modelagem da IMU MPU-6050 "link" "joint" -->
-    <!-- ========================================================================== -->
+    <!-- ********************************************************* -->
     <link name="imu_link">
       <visual>

Commit message: Add start and terminatorfinal characteres to recived message

File: littlebot_description/urdf/littlebot_robot.urdf.xacro (robot description, xacro)
@@ -85,8 +85,8 @@
       </inertial>
     </link>
-    <joint name="chassis_to_free_wheel" type="fixed">
-      <parent link="chassis"/>
+    <joint name="caster_to_free_wheel" type="fixed">
+      <parent link="caster"/>
       <child link="free_wheel"/>
-      <origin xyz="-0.102 0.0 -0.0245" rpy="0 0 0" />
+      <origin xyz="0.0 0.0 0.0" rpy="0 0 0" />
     </joint>
     <!-- Modelagem da IMU MPU-6050 "link" "joint" -->

Commit message: Body colision adjustment

File: littlebot_description/urdf/littlebot_robot.urdf.xacro (robot description, xacro)
@@ -16,7 +16,7 @@
       </visual>
       <collision>
-        <origin xyz="0 0 0.018" rpy="0 0 0" />
+        <origin xyz="0 0 0.007" rpy="0 0 0" />
         <geometry>
-          <box size="0.21 0.11 0.05"/>
+          <box size="0.21 0.11 0.01"/>
         </geometry>
       </collision>

File: littlebot_description/urdf/littlebot_wheel.urdf.xacro (robot description, xacro)
@@ -10,9 +10,7 @@
       </visual>
       <collision>
-        <!-- <xacro:insert_block name="mesh_wheel_pose"/> -->
         <origin xyz="0 0 0" rpy="1.571 0 0" />
         <geometry>
           <cylinder length="0.018" radius="0.03298"/>
-          <!-- <mesh filename="file://$(find littlebot_description)/meshes/roda.dae" /> -->
         </geometry>
       </collision>

Commit message: Fixed weheel caster position

File: littlebot_description/urdf/littlebot_robot.urdf.xacro (robot description, xacro)
@@ -66,5 +66,5 @@
     <link name="free_wheel">
       <visual>
-        <origin xyz="0 0 0" rpy="0 0 0" />
+        <origin xyz="-0.015 0 -0.015" rpy="0 0 0" />
         <geometry>
           <mesh filename="file://$(find littlebot_description)/meshes/Wheel.dae" />
@@ -72,5 +72,5 @@
       </visual>
       <collision>
-        <origin xyz="0 0 0.0" rpy="0 0 0" />
+        <origin xyz="-0.015 0 -0.015" rpy="0 0 0" />
         <geometry>
           <mesh filename="file://$(find littlebot_description)/meshes/Wheel.dae" />
@@ -78,5 +78,5 @@
       </collision>
       <inertial>
-        <origin xyz="0 0 0" rpy="0 0 0"/>
+        <origin xyz="-0.015 0 -0.015" rpy="0 0 0"/>
         <mass value="0.007"/>
         <inertia ixx="3.6e-7" ixy="0"         ixz="0"

Commit message: added base_footprint link

File: littlebot_description/urdf/littlebot_robot.urdf.xacro (robot description, xacro)
@@ -6,4 +6,12 @@
     <link name="base_link">
     </link>
+    <!-- Robot Footprint -->
+    <!-- ********************************************************* -->
+    <link name="base_footprint"/>
+    <joint name="base_joint" type="fixed">
+      <parent link="base_link"/>
+      <child link="base_footprint"/>
+      <origin xyz="0.0 0.0 -0.03074" rpy="0 0 0"/>
+    </joint>
     <!-- Modelagem chassis "link" and "joint"-->
     <!-- ********************************************************* -->
