Commit message: Fixed wheel inetial positions

File: littlebot_description/urdf/littlebot_wheel.urdf.xacro (robot description, xacro)
@@ -16,5 +16,6 @@
       </collision>
       <inertial>
-        <xacro:insert_block name="mesh_wheel_pose"/>
+        <!-- <xacro:insert_block name="mesh_wheel_pose"/> -->
+        <origin xyz="0 0 0" rpy="0 0 1.571" />
         <mass value="0.041"/>
         <inertia ixx="2.967e-5" ixy="-7.675e-15"  ixz="-4.765e-14"
