Commit message: Include wheels to ignition simulation

File: littlebot_description/urdf/littlebot_body.urdf.xacro (robot description, xacro)
@@ -1,5 +1,5 @@
 <?xml version="1.0"?>
-<robot xmlns:xacro="http://ros.org/wiki/xacro"  name="littlebot_robot">
-  <xacro:macro name="littlebot_robot" >
+<robot xmlns:xacro="http://ros.org/wiki/xacro"  name="littlebot_body">
+  <xacro:macro name="littlebot_body" >
     <!-- Modelagem base_link "link" -->
     <!-- ********************************************************* -->
@@ -8,10 +8,10 @@
     <!-- Robot Footprint -->
     <!-- ********************************************************* -->
-    <link name="base_footprint"/>
-    <joint name="base_joint" type="fixed">
+    <!-- <link name="base_footprint"/> -->
+    <!-- <joint name="base_joint" type="fixed">
       <parent link="base_link"/>
       <child link="base_footprint"/>
       <origin xyz="0.0 0.0 -0.03074" rpy="0 0 0"/>
-    </joint>
+    </joint> -->
     <!-- Modelagem chassis_link "link" and "joint"-->
     <!-- ********************************************************* -->
@@ -44,5 +44,5 @@
     <!-- Modelagem caster wheel-->
     <!-- ********************************************************* -->
-    <link name="caster">
+    <!-- <link name="caster">
       <visual>
         <origin xyz="0 0 0" rpy="3.14 0 3.14" />
@@ -70,8 +70,8 @@
       <origin xyz="-0.0871 0.0 -0.00875" rpy="0 0 0" />
       <axis xyz="0 0 1" rpy="0 0 0" />
-    </joint>
+    </joint> -->
     <!-- Modelagem free wheel-->
     <!-- ********************************************************* -->
-    <link name="free_wheel">
+    <!-- <link name="free_wheel">
       <visual>
         <origin xyz="0 0 0" rpy="0 0 0" />
@@ -99,8 +99,8 @@
       <origin xyz="-0.015 0 -0.015" rpy="0 0 0" />
       <axis xyz="0 1 0" rpy="0 0 0" />
-    </joint>
+    </joint> -->
     <!-- Modelagem da IMU MPU-6050 "link" "joint" -->
     <!-- ********************************************************* -->
-    <link name="imu_link">
+    <!-- <link name="imu_link">
       <visual>
         <origin xyz="0 0 0" rpy="0 0 0" />
@@ -127,5 +127,5 @@
       <child link="imu_link"/>
       <origin xyz="0.028 0.0 0.005" rpy="0 0 0" />
-    </joint>
+    </joint> -->
   </xacro:macro>
 </robot>

File: littlebot_description/urdf/littlebot_description.urdf.xacro (robot description, xacro)
@@ -2,12 +2,12 @@
 <robot xmlns:xacro="http://ros.org/wiki/xacro"  name="littlebot">
   <!-- Default arguments -->
-  <xacro:arg name="use_sim" default="false" />
+  <xacro:arg name="use_sim" default="true" />
   <xacro:arg name="prefix" default="littlebot" />
   <!-- Included URDF XACRO Files -->
+  <xacro:include filename="$(find littlebot_description)/urdf/littlebot_body.urdf.xacro" />
   <xacro:include filename="$(find littlebot_description)/urdf/littlebot_wheel.urdf.xacro" />
   <xacro:include filename="$(find littlebot_description)/urdf/littlebot_sonar.urdf.xacro" />
-  <xacro:include filename="$(find littlebot_description)/urdf/littlebot_body.urdf.xacro" />
   <!-- Included GAZEBO XACRO Files -->
-  <xacro:include filename="$(find littlebot_description)/gazebo/littlebot.gazebo.xacro" />
+  <!-- <xacro:include filename="$(find littlebot_description)/gazebo/littlebot.gazebo.xacro" /> -->
   <!-- Included ROS2_CONTROL XACRO Files -->
   <!-- <xacro:include filename="$(find littlebot_description)/ros2_control/littlebot.ros2_control.xacro" /> -->
@@ -15,5 +15,5 @@
   <!-- =========================================================== -->
   <!-- Body model -->
-  <xacro:littlebot_robot />
+  <xacro:littlebot_body />
   <!-- Whells models -->
   <xacro:littlebot_wheel side_wheel="left">
@@ -30,29 +30,29 @@
     <origin xyz="0.07879836 0.03772198 0.02500000" rpy="0 0 0.686455448" />
   </xacro:littlebot_sonar>
-  <xacro:littlebot_sonar sonar_numero="2">
+  <!-- <xacro:littlebot_sonar sonar_numero="2">
     <origin xyz="0 0 -0.020267" rpy="0 0 0" />
     <origin xyz="0.08880761 0.02002920 0.02500000" rpy="0 0 0.343218997"/>
-  </xacro:littlebot_sonar>
-  <xacro:littlebot_sonar sonar_numero="3">
+  </xacro:littlebot_sonar> -->
+  <!-- <xacro:littlebot_sonar sonar_numero="3">
     <origin xyz="0 0 -0.020267" rpy="0 0 0" />
     <origin xyz="0.092279 0.0 0.02500000" rpy="0 0 0" />
-  </xacro:littlebot_sonar>
-  <xacro:littlebot_sonar sonar_numero="4">
+  </xacro:littlebot_sonar> -->
+  <!-- <xacro:littlebot_sonar sonar_numero="4">
     <origin xyz="0 0 -0.020267" rpy="0 0 0" />
     <origin xyz="0.08880761 -0.02002920 0.02500000" rpy="0 0 -0.343218997"/>
-  </xacro:littlebot_sonar>
-  <xacro:littlebot_sonar sonar_numero="5">
+  </xacro:littlebot_sonar> -->
+  <!-- <xacro:littlebot_sonar sonar_numero="5">
     <origin xyz="0 0 -0.020267" rpy="0 0 0" />
     <origin xyz="0.07879836 -0.03772198 0.02500000" rpy="0 0 -0.686455448"/>
-  </xacro:littlebot_sonar>
+  </xacro:littlebot_sonar> -->
   <!-- Load Gazebo plugins -->
   <!-- =========================================================== -->
-  <xacro:if value="$(arg use_sim)">
+  <!-- <xacro:if value="$(arg use_sim)">
     <xacro:littlebot_gazebo/>
-  </xacro:if>
+  </xacro:if> -->
   <!-- Load ROS2 Control plugins -->
   <!-- =========================================================== -->
-  <xacro:unless value="$(arg use_sim)">
+  <!-- <xacro:unless value="$(arg use_sim)"> -->
     <!-- <xacro:littlebot_control/> -->
-  </xacro:unless>
+  <!-- </xacro:unless> -->
 </robot>

Commit message: Basic forms to colision tags of the free wheell

File: littlebot_description/urdf/littlebot_body.urdf.xacro (robot description, xacro)
@@ -44,5 +44,5 @@
     <!-- Modelagem caster wheel-->
     <!-- ********************************************************* -->
-    <!-- <link name="caster">
+    <link name="caster">
       <visual>
         <origin xyz="0 0 0" rpy="3.14 0 3.14" />
@@ -54,5 +54,5 @@
         <origin xyz="0 0 0.0" rpy="3.14 0 3.14" />
         <geometry>
-          <mesh filename="file://$(find littlebot_description)/meshes/Caster_Wheel_Plate.dae" />
+          <box size="0.21 0.11 0.01"/>
         </geometry>
       </collision>
@@ -70,8 +70,8 @@
       <origin xyz="-0.0871 0.0 -0.00875" rpy="0 0 0" />
       <axis xyz="0 0 1" rpy="0 0 0" />
-    </joint> -->
+    </joint>
     <!-- Modelagem free wheel-->
     <!-- ********************************************************* -->
-    <!-- <link name="free_wheel">
+    <link name="free_wheel">
       <visual>
         <origin xyz="0 0 0" rpy="0 0 0" />
@@ -83,5 +83,5 @@
         <origin xyz="0 0 0" rpy="0 0 0" />
         <geometry>
-          <mesh filename="file://$(find littlebot_description)/meshes/Wheel.dae" />
+          <box size="0.21 0.11 0.01"/>
         </geometry>
       </collision>
@@ -99,8 +99,8 @@
       <origin xyz="-0.015 0 -0.015" rpy="0 0 0" />
       <axis xyz="0 1 0" rpy="0 0 0" />
-    </joint> -->
+    </joint>
     <!-- Modelagem da IMU MPU-6050 "link" "joint" -->
     <!-- ********************************************************* -->
-    <!-- <link name="imu_link">
+    <link name="imu_link">
       <visual>
         <origin xyz="0 0 0" rpy="0 0 0" />
@@ -112,5 +112,5 @@
         <origin xyz="0 0 0" rpy="0 0 0" />
         <geometry>
-          <mesh filename="file://$(find littlebot_description)/meshes/MPU_6050.dae" />
+          <box size="0.21 0.11 0.01"/>
         </geometry>
       </collision>
@@ -127,5 +127,5 @@
       <child link="imu_link"/>
       <origin xyz="0.028 0.0 0.005" rpy="0 0 0" />
-    </joint> -->
+    </joint>
   </xacro:macro>
 </robot>

File: littlebot_description/urdf/littlebot_description.urdf.xacro (robot description, xacro)
@@ -7,5 +7,5 @@
   <xacro:include filename="$(find littlebot_description)/urdf/littlebot_body.urdf.xacro" />
   <xacro:include filename="$(find littlebot_description)/urdf/littlebot_wheel.urdf.xacro" />
-  <xacro:include filename="$(find littlebot_description)/urdf/littlebot_sonar.urdf.xacro" />
+  <!-- <xacro:include filename="$(find littlebot_description)/urdf/littlebot_sonar.urdf.xacro" /> -->
   <!-- Included GAZEBO XACRO Files -->
   <!-- <xacro:include filename="$(find littlebot_description)/gazebo/littlebot.gazebo.xacro" /> -->
@@ -26,8 +26,8 @@
   </xacro:littlebot_wheel>
   <!-- Sonar models-->
-  <xacro:littlebot_sonar sonar_numero="1">
+  <!-- <xacro:littlebot_sonar sonar_numero="1">
     <origin xyz="0 0 -0.020267" rpy="0 0 0" />
     <origin xyz="0.07879836 0.03772198 0.02500000" rpy="0 0 0.686455448" />
-  </xacro:littlebot_sonar>
+  </xacro:littlebot_sonar> -->
   <!-- <xacro:littlebot_sonar sonar_numero="2">
     <origin xyz="0 0 -0.020267" rpy="0 0 0" />
