Commit message: IMU and sonar plugins added

File: littlebot_description/gazebo/littlebot.gazebo.xacro (robot description, xacro)
@@ -30,5 +30,5 @@
     </ros2_control>
     <!-- Plugin IMU -->
-    <!-- <gazebo reference="imu_link">
+    <gazebo reference="imu_link">
       <sensor name="imu_sensor" type="imu">
         <plugin filename="libgazebo_ros_imu_sensor.so" name="imu_plugin">
@@ -43,7 +43,7 @@
         <visualize>true</visualize>
       </sensor>
-    </gazebo> -->
+    </gazebo>
     <!-- Plugin SONAR -->
-    <!-- <xacro:macro name="sonar" params="reference topic_name">
+    <xacro:macro name="sonar" params="reference topic_name">
       <gazebo reference="${reference}">
         <sensor type="ray" name="TeraRanger">
@@ -74,6 +74,5 @@
               <stddev>0.005</stddev>
             </noise>
-          </ray> -->
-<!--
+          </ray>
           <plugin name="gazebo_ros_range_controller" filename="libgazebo_ros_ray_sensor.so">
             <ros>
@@ -87,11 +86,11 @@
         </sensor>
       </gazebo>
-    </xacro:macro> -->
+    </xacro:macro>
     <!-- Call SONAR gazebo plugin xacro -->
-    <!-- <xacro:sonar reference="sonar_1" topic_name="sonar1" />
+    <xacro:sonar reference="sonar_1" topic_name="sonar1" />
     <xacro:sonar reference="sonar_2" topic_name="sonar2" />
     <xacro:sonar reference="sonar_3" topic_name="sonar3" />
     <xacro:sonar reference="sonar_4" topic_name="sonar4" />
-    <xacro:sonar reference="sonar_5" topic_name="sonar5" /> -->
+    <xacro:sonar reference="sonar_5" topic_name="sonar5" />
   </xacro:macro>
 </robot>

Commit message: Add status to joint free wheel caster joints

File: littlebot_description/gazebo/littlebot.gazebo.xacro (robot description, xacro)
@@ -27,4 +27,10 @@
         <state_interface name="position"/>
         <state_interface name="velocity"/>
+      </joint>
+      <joint name="chassis_to_caster">
+        <state_interface name="position"/>
+      </joint>
+      <joint name="caster_to_free_wheel">
+        <state_interface name="position"/>
       </joint>
     </ros2_control>

File: littlebot_description/urdf/littlebot_robot.urdf.xacro (robot description, xacro)
@@ -57,8 +57,9 @@
       </inertial>
     </link>
-    <joint name="chassis_to_caster" type="fixed">
+    <joint name="chassis_to_caster" type="continuous">
       <parent link="chassis"/>
       <child link="caster"/>
       <origin xyz="-0.0871 0.0 -0.00875" rpy="0 0 0" />
+      <axis xyz="0 0 1" rpy="0 0 0" />
     </joint>
     <!-- Modelagem free wheel-->
@@ -66,5 +67,5 @@
     <link name="free_wheel">
       <visual>
-        <origin xyz="-0.015 0 -0.015" rpy="0 0 0" />
+        <origin xyz="0 0 0" rpy="0 0 0" />
         <geometry>
           <mesh filename="file://$(find littlebot_description)/meshes/Wheel.dae" />
@@ -72,5 +73,5 @@
       </visual>
       <collision>
-        <origin xyz="-0.015 0 -0.015" rpy="0 0 0" />
+        <origin xyz="0 0 0" rpy="0 0 0" />
         <geometry>
           <mesh filename="file://$(find littlebot_description)/meshes/Wheel.dae" />
@@ -78,5 +79,5 @@
       </collision>
       <inertial>
-        <origin xyz="-0.015 0 -0.015" rpy="0 0 0"/>
+        <origin xyz="0 0 0" rpy="0 0 0"/>
         <mass value="0.007"/>
         <inertia ixx="3.6e-7" ixy="0"         ixz="0"
@@ -85,8 +86,9 @@
       </inertial>
     </link>
-    <joint name="caster_to_free_wheel" type="fixed">
+    <joint name="caster_to_free_wheel" type="continuous">
       <parent link="caster"/>
       <child link="free_wheel"/>
-      <origin xyz="0.0 0.0 0.0" rpy="0 0 0" />
+      <origin xyz="-0.015 0 -0.015" rpy="0 0 0" />
+      <axis xyz="0 1 0" rpy="0 0 0" />
     </joint>
     <!-- Modelagem da IMU MPU-6050 "link" "joint" -->

Commit message: Added base_footprint and base_link to urdf file

File: littlebot_description/gazebo/littlebot.gazebo.xacro (robot description, xacro)
@@ -28,5 +28,5 @@
         <state_interface name="velocity"/>
       </joint>
-      <joint name="chassis_to_caster">
+      <joint name="base_link_to_caster">
         <state_interface name="position"/>
       </joint>

File: littlebot_description/urdf/littlebot_robot.urdf.xacro (robot description, xacro)
@@ -2,11 +2,11 @@
 <robot xmlns:xacro="http://ros.org/wiki/xacro"  name="littlebot_robot">
   <xacro:macro name="littlebot_robot" >
-    <!-- Modelagem base_link "link" -->
+    <!-- Modelagem base_footprint "link" -->
+    <!-- ********************************************************* -->
+    <link name="base_footprint">
+    </link>
+    <!-- Modelagem base_link "link" and "joint"-->
     <!-- ********************************************************* -->
     <link name="base_link">
-    </link>
-    <!-- Modelagem chassis "link" and "joint"-->
-    <!-- ********************************************************* -->
-    <link name="chassis">
       <visual>
         <origin xyz="0 0 0" rpy="0 0 0" />
@@ -29,7 +29,7 @@
       </inertial>
     </link>
-    <joint name="base_to_chassis" type="fixed">
-      <parent link="base_link"/>
-      <child link="chassis"/>
+    <joint name="base_footprint_to_base_link" type="fixed">
+      <parent link="base_footprint"/>
+      <child link="base_link"/>
       <origin xyz="0.0 0.0 0.0" rpy="0 0 0" />
     </joint>
@@ -57,6 +57,6 @@
       </inertial>
     </link>
-    <joint name="chassis_to_caster" type="continuous">
-      <parent link="chassis"/>
+    <joint name="base_link_to_caster" type="continuous">
+      <parent link="base_link"/>
       <child link="caster"/>
       <origin xyz="-0.0871 0.0 -0.00875" rpy="0 0 0" />
@@ -115,6 +115,6 @@
       </inertial>
     </link>
-    <joint name="chassis_to_imu" type="fixed">
-      <parent link="chassis"/>
+    <joint name="base_link_to_imu" type="fixed">
+      <parent link="base_link"/>
       <child link="imu_link"/>
       <origin xyz="0.028 0.0 0.005" rpy="0 0 0" />

File: littlebot_description/urdf/littlebot_sonar.urdf.xacro (robot description, xacro)
@@ -24,5 +24,5 @@
     </link>
     <joint name="base_to_sonar_${sonar_numero}" type="fixed">
-      <parent link="chassis"/>
+      <parent link="base_link"/>
       <child link="sonar_${sonar_numero}"/>
       <xacro:insert_block name="joint_pose"/>

File: littlebot_description/urdf/littlebot_wheel.urdf.xacro (robot description, xacro)
@@ -24,5 +24,5 @@
     </link>
     <joint name="base_to_${side_wheel}_wheel" type="continuous">
-      <parent link="chassis"/>
+      <parent link="base_link"/>
       <child link="${side_wheel}_wheel"/>
       <xacro:insert_block name="joint_wheel_pose"/>

Commit message: Adjust tf frames to REP105

File: littlebot_description/gazebo/littlebot.gazebo.xacro (robot description, xacro)
@@ -28,5 +28,5 @@
         <state_interface name="velocity"/>
       </joint>
-      <joint name="base_link_to_caster">
+      <joint name="body_to_caster">
         <state_interface name="position"/>
       </joint>

File: littlebot_description/urdf/littlebot_robot.urdf.xacro (robot description, xacro)
@@ -2,11 +2,11 @@
 <robot xmlns:xacro="http://ros.org/wiki/xacro"  name="littlebot_robot">
   <xacro:macro name="littlebot_robot" >
-    <!-- Modelagem base_footprint "link" -->
-    <!-- ********************************************************* -->
-    <link name="base_footprint">
-    </link>
-    <!-- Modelagem base_link "link" and "joint"-->
+    <!-- Modelagem base_link "link" -->
     <!-- ********************************************************* -->
     <link name="base_link">
+    </link>
+    <!-- Modelagem body "link" and "joint"-->
+    <!-- ********************************************************* -->
+    <link name="body">
       <visual>
         <origin xyz="0 0 0" rpy="0 0 0" />
@@ -29,7 +29,7 @@
       </inertial>
     </link>
-    <joint name="base_footprint_to_base_link" type="fixed">
-      <parent link="base_footprint"/>
-      <child link="base_link"/>
+    <joint name="base_link_to_body" type="fixed">
+      <parent link="base_link"/>
+      <child link="body"/>
       <origin xyz="0.0 0.0 0.0" rpy="0 0 0" />
     </joint>
@@ -57,6 +57,6 @@
       </inertial>
     </link>
-    <joint name="base_link_to_caster" type="continuous">
-      <parent link="base_link"/>
+    <joint name="body_to_caster" type="continuous">
+      <parent link="body"/>
       <child link="caster"/>
       <origin xyz="-0.0871 0.0 -0.00875" rpy="0 0 0" />
@@ -115,6 +115,6 @@
       </inertial>
     </link>
-    <joint name="base_link_to_imu" type="fixed">
-      <parent link="base_link"/>
+    <joint name="body_to_imu" type="fixed">
+      <parent link="body"/>
       <child link="imu_link"/>
       <origin xyz="0.028 0.0 0.005" rpy="0 0 0" />

File: littlebot_description/urdf/littlebot_sonar.urdf.xacro (robot description, xacro)
@@ -24,5 +24,5 @@
     </link>
     <joint name="base_to_sonar_${sonar_numero}" type="fixed">
-      <parent link="base_link"/>
+      <parent link="body"/>
       <child link="sonar_${sonar_numero}"/>
       <xacro:insert_block name="joint_pose"/>

File: littlebot_description/urdf/littlebot_wheel.urdf.xacro (robot description, xacro)
@@ -24,5 +24,5 @@
     </link>
     <joint name="base_to_${side_wheel}_wheel" type="continuous">
-      <parent link="base_link"/>
+      <parent link="body"/>
       <child link="${side_wheel}_wheel"/>
       <xacro:insert_block name="joint_wheel_pose"/>

Commit message: Included base_footprint link

File: littlebot_description/gazebo/littlebot.gazebo.xacro (robot description, xacro)
@@ -28,5 +28,5 @@
         <state_interface name="velocity"/>
       </joint>
-      <joint name="body_to_caster">
+      <joint name="chassis_link_to_caster">
         <state_interface name="position"/>
       </joint>

File: littlebot_description/urdf/littlebot_robot.urdf.xacro (robot description, xacro)
@@ -6,7 +6,15 @@
     <link name="base_link">
     </link>
-    <!-- Modelagem body "link" and "joint"-->
+    <!-- Robot Footprint -->
     <!-- ********************************************************* -->
-    <link name="body">
+    <link name="base_footprint"/>
+    <joint name="base_joint" type="fixed">
+      <parent link="base_link"/>
+      <child link="base_footprint"/>
+      <origin xyz="0.0 0.0 -0.03074" rpy="0 0 0"/>
+    </joint>
+    <!-- Modelagem chassis_link "link" and "joint"-->
+    <!-- ********************************************************* -->
+    <link name="chassis_link">
       <visual>
         <origin xyz="0 0 0" rpy="0 0 0" />
@@ -29,7 +37,7 @@
       </inertial>
     </link>
-    <joint name="base_link_to_body" type="fixed">
+    <joint name="base_link_to_chassis_link" type="fixed">
       <parent link="base_link"/>
-      <child link="body"/>
+      <child link="chassis_link"/>
       <origin xyz="0.0 0.0 0.0" rpy="0 0 0" />
     </joint>
@@ -57,6 +65,6 @@
       </inertial>
     </link>
-    <joint name="body_to_caster" type="continuous">
-      <parent link="body"/>
+    <joint name="chassis_link_to_caster" type="continuous">
+      <parent link="chassis_link"/>
       <child link="caster"/>
       <origin xyz="-0.0871 0.0 -0.00875" rpy="0 0 0" />
@@ -115,6 +123,6 @@
       </inertial>
     </link>
-    <joint name="body_to_imu" type="fixed">
-      <parent link="body"/>
+    <joint name="chassis_link_to_imu" type="fixed">
+      <parent link="chassis_link"/>
       <child link="imu_link"/>
       <origin xyz="0.028 0.0 0.005" rpy="0 0 0" />

File: littlebot_description/urdf/littlebot_sonar.urdf.xacro (robot description, xacro)
@@ -24,5 +24,5 @@
     </link>
     <joint name="base_to_sonar_${sonar_numero}" type="fixed">
-      <parent link="body"/>
+      <parent link="chassis_link"/>
       <child link="sonar_${sonar_numero}"/>
       <xacro:insert_block name="joint_pose"/>

File: littlebot_description/urdf/littlebot_wheel.urdf.xacro (robot description, xacro)
@@ -24,5 +24,5 @@
     </link>
     <joint name="base_to_${side_wheel}_wheel" type="continuous">
-      <parent link="body"/>
+      <parent link="chassis_link"/>
       <child link="${side_wheel}_wheel"/>
       <xacro:insert_block name="joint_wheel_pose"/>

Commit message: update urdf to ignition differential controller

File: littlebot_description/gazebo/littlebot.gazebo.xacro (robot description, xacro)
@@ -2,11 +2,30 @@
 <robot xmlns:xacro="http://ros.org/wiki/xacro">
   <xacro:macro name="littlebot_gazebo">
+  <gazebo>
+    <plugin
+      filename="ignition-gazebo-diff-drive-system"
+      name="ignition::gazebo::systems::DiffDrive">
+      <left_joint>base_to_left_wheel</left_joint>
+      <right_joint>base_to_right_wheel</right_joint>
+      <wheel_separation>0.11</wheel_separation>
+      <wheel_radius>0.0329</wheel_radius>
+      <odom_publish_frequency>1</odom_publish_frequency>
+      <max_linear_acceleration>1</max_linear_acceleration>
+      <min_linear_acceleration>-1</min_linear_acceleration>
+      <max_angular_acceleration>2</max_angular_acceleration>
+      <min_angular_acceleration>-2</min_angular_acceleration>
+      <max_linear_velocity>0.5</max_linear_velocity>
+      <min_linear_velocity>-0.5</min_linear_velocity>
+      <max_angular_velocity>1</max_angular_velocity>
+      <min_angular_velocity>-1</min_angular_velocity>
+    </plugin>
+  </gazebo>
     <!-- Plugin CONTROLER -->
-    <gazebo>
+    <!-- <gazebo>
       <plugin name="gazebo_ros2_control" filename="libgazebo_ros2_control.so">
         <parameters>$(find littlebot_control)/config/control.yaml</parameters>
       </plugin>
-    </gazebo>
-    <ros2_control name="littlebot_hardware_sim" type="system">
+    </gazebo> -->
+    <!-- <ros2_control name="littlebot_hardware_sim" type="system">
       <hardware>
         <plugin>gazebo_ros2_control/GazeboSystem</plugin>
@@ -34,7 +53,7 @@
         <state_interface name="position"/>
       </joint>
-    </ros2_control>
+    </ros2_control> -->
     <!-- Plugin IMU -->
-    <gazebo reference="imu_link">
+    <!-- <gazebo reference="imu_link">
       <sensor name="imu_sensor" type="imu">
         <plugin filename="libgazebo_ros_imu_sensor.so" name="imu_plugin">
@@ -49,7 +68,7 @@
         <visualize>true</visualize>
       </sensor>
-    </gazebo>
+    </gazebo> -->
     <!-- Plugin SONAR -->
-    <xacro:macro name="sonar" params="reference topic_name">
+    <!-- <xacro:macro name="sonar" params="reference topic_name">
       <gazebo reference="${reference}">
         <sensor type="ray" name="TeraRanger">
@@ -92,11 +111,11 @@
         </sensor>
       </gazebo>
-    </xacro:macro>
+    </xacro:macro> -->
     <!-- Call SONAR gazebo plugin xacro -->
-    <xacro:sonar reference="sonar_1" topic_name="sonar1" />
-    <xacro:sonar reference="sonar_2" topic_name="sonar2" />
-    <xacro:sonar reference="sonar_3" topic_name="sonar3" />
-    <xacro:sonar reference="sonar_4" topic_name="sonar4" />
-    <xacro:sonar reference="sonar_5" topic_name="sonar5" />
+    <!-- <xacro:sonar reference="sonar_1" topic_name="sonar1" /> -->
+    <!-- <xacro:sonar reference="sonar_2" topic_name="sonar2" /> -->
+    <!-- <xacro:sonar reference="sonar_3" topic_name="sonar3" /> -->
+    <!-- <xacro:sonar reference="sonar_4" topic_name="sonar4" /> -->
+    <!-- <xacro:sonar reference="sonar_5" topic_name="sonar5" /> -->
   </xacro:macro>
 </robot>

File: littlebot_description/urdf/littlebot_description.urdf.xacro (robot description, xacro)
@@ -9,5 +9,5 @@
   <!-- <xacro:include filename="$(find littlebot_description)/urdf/littlebot_sonar.urdf.xacro" /> -->
   <!-- Included GAZEBO XACRO Files -->
-  <!-- <xacro:include filename="$(find littlebot_description)/gazebo/littlebot.gazebo.xacro" /> -->
+  <xacro:include filename="$(find littlebot_description)/gazebo/littlebot.gazebo.xacro" />
   <!-- Included ROS2_CONTROL XACRO Files -->
   <!-- <xacro:include filename="$(find littlebot_description)/ros2_control/littlebot.ros2_control.xacro" /> -->
@@ -48,7 +48,7 @@
   <!-- Load Gazebo plugins -->
   <!-- =========================================================== -->
-  <!-- <xacro:if value="$(arg use_sim)">
+  <xacro:if value="$(arg use_sim)">
     <xacro:littlebot_gazebo/>
-  </xacro:if> -->
+  </xacro:if>
   <!-- Load ROS2 Control plugins -->
   <!-- =========================================================== -->

Commit message: add files to launch differential controller

File: littlebot_description/gazebo/littlebot.gazebo.xacro (robot description, xacro)
@@ -2,5 +2,5 @@
 <robot xmlns:xacro="http://ros.org/wiki/xacro">
   <xacro:macro name="littlebot_gazebo">
-  <gazebo>
+  <!-- <gazebo>
     <plugin
       filename="ignition-gazebo-diff-drive-system"
@@ -19,4 +19,24 @@
       <max_angular_velocity>1</max_angular_velocity>
       <min_angular_velocity>-1</min_angular_velocity>
+    </plugin>
+  </gazebo> -->
+  <ros2_control name="IgnitionSystem" type="system">
+    <hardware>
+      <plugin>ign_ros2_control/IgnitionSystem</plugin>
+    </hardware>
+    <joint name="base_to_left_wheel">
+        <command_interface name="velocity"/>
+        <state_interface name="position"/>
+        <state_interface name="velocity"/>
+    </joint>
+    <joint name="base_to_right_wheel">
+        <command_interface name="velocity"/>
+        <state_interface name="position"/>
+        <state_interface name="velocity"/>
+    </joint>
+  </ros2_control>
+  <gazebo>
+    <plugin filename="ign_ros2_control-system" name="ign_ros2_control::IgnitionROS2ControlPlugin">
+      <parameters>$(find littlebot_control)/config/control.yaml</parameters>
     </plugin>
   </gazebo>

Commit message: fix rviz ros2 control joint visualization

File: littlebot_description/gazebo/littlebot.gazebo.xacro (robot description, xacro)
@@ -34,4 +34,10 @@
         <state_interface name="position"/>
         <state_interface name="velocity"/>
+    </joint>
+    <joint name="chassis_link_to_caster">
+        <state_interface name="position"/>
+    </joint>
+    <joint name="caster_to_free_wheel">
+        <state_interface name="position"/>
     </joint>
   </ros2_control>

Commit message: Delete unecessary comments

File: littlebot_description/gazebo/littlebot.gazebo.xacro (robot description, xacro)
@@ -47,54 +47,20 @@
     </plugin>
   </gazebo>
-    <!-- Plugin CONTROLER -->
-    <!-- <gazebo>
-      <plugin name="gazebo_ros2_control" filename="libgazebo_ros2_control.so">
-        <parameters>$(find littlebot_control)/config/control.yaml</parameters>
-      </plugin>
-    </gazebo> -->
-    <!-- <ros2_control name="littlebot_hardware_sim" type="system">
-      <hardware>
-        <plugin>gazebo_ros2_control/GazeboSystem</plugin>
-      </hardware>
-      <joint name="base_to_left_wheel">
-        <command_interface name="velocity">
-          <param name="min">-1</param>
-          <param name="max">1</param>
-        </command_interface>
-        <state_interface name="position"/>
-        <state_interface name="velocity"/>
-      </joint>
-      <joint name="base_to_right_wheel">
-        <command_interface name="velocity">
-          <param name="min">-1</param>
-          <param name="max">1</param>
-        </command_interface>
-        <state_interface name="position"/>
-        <state_interface name="velocity"/>
-      </joint>
-      <joint name="chassis_link_to_caster">
-        <state_interface name="position"/>
-      </joint>
-      <joint name="caster_to_free_wheel">
-        <state_interface name="position"/>
-      </joint>
-    </ros2_control> -->
-       <gazebo>
-      <plugin filename="ignition-gazebo-sensors-system" name="ignition::gazebo::systems::Sensors">
-            <render_engine>ogre2</render_engine>
-        </plugin>
-      <plugin filename="ignition-gazebo-imu-system" name="ignition::gazebo::systems::Imu">
-        </plugin>
-    </gazebo>
-    <!-- Plugin IMU -->
-    <gazebo reference="imu_link">
-      <sensor name="imu_sensor" type="imu">
-        <always_on>1</always_on>
-        <update_rate>100</update_rate>
-        <visualize>true</visualize>
-        <ignition_frame_id>imu_link</ignition_frame_id>
-        <topic>imu</topic>
-      </sensor>
-    </gazebo>
+  <!-- Plugin IMU -->
+  <gazebo>
+    <plugin filename="ignition-gazebo-sensors-system" name="ignition::gazebo::systems::Sensors">
+          <render_engine>ogre2</render_engine>
+    </plugin>
+    <plugin filename="ignition-gazebo-imu-system" name="ignition::gazebo::systems::Imu"/>
+  </gazebo>
+  <gazebo reference="imu_link">
+    <sensor name="imu_sensor" type="imu">
+      <always_on>1</always_on>
+      <update_rate>100</update_rate>
+      <visualize>true</visualize>
+      <ignition_frame_id>imu_link</ignition_frame_id>
+      <topic>imu</topic>
+    </sensor>
+  </gazebo>
     <!-- Plugin SONAR -->
     <!-- <xacro:macro name="sonar" params="reference topic_name">
